File: ch32v003f4u6_with_wsleds/ch32v003f4u6_with_wsled.kicad_pcb (KiCad board)
At the start: 2 copper layers, 40.6 x 44.5 mm, 30 parts, among them J2 PGM, J4 USB_C_Receptacle_USB2.0, J5 HOLE, J6 HOLE, U1 CH32V003F4U6, U2 3.3vReg

Commit message: Update with new art from Astronautilus.
Parts:
- turned U1 to -45 degrees
Other:
- board text added: "To Change A: * Fixed rotation of processor."
- board text added: "rev A"
