File: ch32v003-oled-64x48-rb0066E2801a/ch32v003-oled-64x48-rb0066E2801a.kicad_sch (KiCad schematic)
At the start: 20 parts, among them J1 USB_C_Receptacle_USB2.0, J2 PGM, U1 CH32V003F4U6, U2 3.3vReg, U3 25WQ32, U4 OLED-RB0066E2801A-64x48-FULL

Commit message: Forgot to include the build files.
Parts:
- added D1, D2: LED, LED_SMD:LED_0402_1005Metric, symbol Device:LED
- added J3: APPLE, artwork:apple, symbol artwork:artwork
- added R4, R5: 10, Resistor_SMD:R_0402_1005Metric, symbol Device:R
- J2: symbol Connector_Generic:Conn_01x03 -> Connector_Generic:Conn_01x02
Connections:
- net FIOB: now also R4.2, R5.2
- net GND: now also J2.1 (Pin_1), D1.1 (K), D2.1 (K); no longer J2.2 (Pin_2)
- net PGM: now also J2.2 (Pin_2); no longer J2.3 (Pin_3)
- net VDD: no longer J2.1 (Pin_1)
- net at U1.1 (PD7/NRST/T2CH4/OPP1/UCK): no longer R1.2
- net at U1.18 (PD4/A7/UCK/T2CH1ETR/OPO/T1CH4ETR): now also R1.2
- new net: D2.2 (A), R5.1
- new net: D1.2 (A), R4.1

Commit message: Bump versions.
Other:
- note removed: "IRE: 741+286mV White, 286mV Black, 0V Sync"
- moved on the sheet: U2
Changed lines of the file:
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@@
     (stroke (width 0) (type default) (color 0 0 0 0))
-  )
-  (text "IRE: 741+286mV White, 286mV Black, 0V Sync" (at 130.81 85.09 0)
-    (effects (font (size 1.27 1.27)) (justify left bottom))
   )
   (text "Analog TRRS" (at 71.12 146.05 0)
@@
     )
   )
-  (symbol (lib_id "power:VDD") (at 133.35 110.49 270) (unit 1)
-    (in_bom yes) (on_board yes)
-    (property "Reference" "#PWR018" (id 0) (at 129.54 110.49 0)
-      (effects (font (size 1.27 1.27)) hide)
-    )
-    (property "Value" "VDD" (id 1) (at 137.16 110.49 90)
-      (effects (font (size 1.27 1.27)) (justify left))
-    )
-    (property "Footprint" "" (id 2) (at 133.35 110.49 0)
-      (effects (font (size 1.27 1.27)) hide)
-    )
-    (property "Datasheet" "" (id 3) (at 133.35 110.49 0)
+  (symbol (lib_id "power:VDD") (at 139.7 113.03 270) (unit 1)
+    (in_bom yes) (on_board yes)
+    (property "Reference" "#PWR018" (id 0) (at 135.89 113.03 0)
+      (effects (font (size 1.27 1.27)) hide)
+    )
+    (property "Value" "VDD" (id 1) (at 143.51 113.03 90)
+      (effects (font (size 1.27 1.27)) (justify left))
+    )
+    (property "Footprint" "" (id 2) (at 139.7 113.03 0)
+      (effects (font (size 1.27 1.27)) hide)
+    )
+    (property "Datasheet" "" (id 3) (at 139.7 113.03 0)
       (effects (font (size 1.27 1.27)) hide)
     )
@@
     (pin "1")
   )
-  (symbol (lib_id "power:+5V") (at 113.03 110.49 90) (unit 1)
-    (in_bom yes) (on_board yes)
-    (property "Reference" "#PWR013" (id 0) (at 116.84 110.49 0)
-      (effects (font (size 1.27 1.27)) hide)
-    )
-    (property "Value" "+5V" (id 1) (at 105.41 110.49 90)
-      (effects (font (size 1.27 1.27)) (justify right))
-    )
-    (property "Footprint" "" (id 2) (at 113.03 110.49 0)
-      (effects (font (size 1.27 1.27)) hide)
-    )
-    (property "Datasheet" "" (id 3) (at 113.03 110.49 0)
+  (symbol (lib_id "power:+5V") (at 119.38 113.03 90) (unit 1)
+    (in_bom yes) (on_board yes)
+    (property "Reference" "#PWR013" (id 0) (at 123.19 113.03 0)
+      (effects (font (size 1.27 1.27)) hide)
+    )
+    (property "Value" "+5V" (id 1) (at 111.76 113.03 90)
+      (effects (font (size 1.27 1.27)) (justify right))
+    )
+    (property "Footprint" "" (id 2) (at 119.38 113.03 0)
+      (effects (font (size 1.27 1.27)) hide)
+    )
+    (property "Datasheet" "" (id 3) (at 119.38 113.03 0)
       (effects (font (size 1.27 1.27)) hide)
     )
@@
     (pin "1")
   )
-  (symbol (lib_id "Regulator_Linear:NCP115AMX120TCG") (at 123.19 113.03 0) (unit 1)
-    (in_bom yes) (on_board yes) (fields_autoplaced)
-    (property "Reference" "U2" (id 0) (at 123.19 104.2502 0))
-    (property "Value" "3.3vReg" (id 1) (at 123.19 106.7871 0))
-    (property "Footprint" "cnhardware:xdfn-reg" (id 2) (at 123.19 113.03 0)
-      (effects (font (size 1.27 1.27)) hide)
-    )
-    (property "Datasheet" "https://www.onsemi.com/pub/Collateral/NCP115-D.PDF" (id 3) (at 123.19 113.03 0)
-      (effects (font (size 1.27 1.27)) hide)
-    )
-    (property "LCSC" "C379350" (id 4) (at 123.19 113.03 0)
+  (symbol (lib_id "Regulator_Linear:NCP115AMX120TCG") (at 129.54 115.57 0) (unit 1)
+    (in_bom yes) (on_board yes) (fields_autoplaced)
+    (property "Reference" "U2" (id 0) (at 129.54 106.7902 0))
+    (property "Value" "3.3vReg" (id 1) (at 129.54 109.3271 0))
+    (property "Footprint" "cnhardware:xdfn-reg" (id 2) (at 129.54 115.57 0)
+      (effects (font (size 1.27 1.27)) hide)
+    )
+    (property "Datasheet" "https://www.onsemi.com/pub/Collateral/NCP115-D.PDF" (id 3) (at 129.54 115.57 0)
+      (effects (font (size 1.27 1.27)) hide)
+    )
+    (property "LCSC" "C379350" (id 4) (at 129.54 115.57 0)
       (effects (font (size 1.27 1.27)) hide)
     )
@@
     (pin "1")
   )
-  (symbol (lib_id "power:GND") (at 123.19 120.65 0) (unit 1)
-    (in_bom yes) (on_board yes) (fields_autoplaced)
-    (property "Reference" "#PWR015" (id 0) (at 123.19 127 0)
-      (effects (font (size 1.27 1.27)) hide)
-    )
-    (property "Value" "GND" (id 1) (at 123.19 125.73 0))
-    (property "Footprint" "" (id 2) (at 123.19 120.65 0)
-      (effects (font (size 1.27 1.27)) hide)
-    )
-    (property "Datasheet" "" (id 3) (at 123.19 120.65 0)
+  (symbol (lib_id "power:GND") (at 129.54 123.19 0) (unit 1)
+    (in_bom yes) (on_board yes) (fields_autoplaced)
+    (property "Reference" "#PWR015" (id 0) (at 129.54 129.54 0)
+      (effects (font (size 1.27 1.27)) hide)
+    )
+    (property "Value" "GND" (id 1) (at 129.54 128.27 0))
+    (property "Footprint" "" (id 2) (at 129.54 123.19 0)
+      (effects (font (size 1.27 1.27)) hide)
+    )
+    (property "Datasheet" "" (id 3) (at 129.54 123.19 0)
       (effects (font (size 1.27 1.27)) hide)
     )
@@
     (pin "1")
   )
-  (symbol (lib_id "power:+5V") (at 113.03 115.57 90) (unit 1)
-    (in_bom yes) (on_board yes)
-    (property "Reference" "#PWR014" (id 0) (at 116.84 115.57 0)
-      (effects (font (size 1.27 1.27)) hide)
-    )
-    (property "Value" "+5V" (id 1) (at 105.41 115.57 90)
-      (effects (font (size 1.27 1.27)) (justify right))
-    )
-    (property "Footprint" "" (id 2) (at 113.03 115.57 0)
-      (effects (font (size 1.27 1.27)) hide)
-    )
-    (property "Datasheet" "" (id 3) (at 113.03 115.57 0)
-      (effects (font (size 1.27 1.27)) hide)
-    )
+  (symbol (lib_id "power:+5V") (at 119.38 118.11 90) (unit 1)
+    (in_bom yes) (on_board yes)
+    (property "Reference" "#PWR014" (id 0) (at 123.19 118.11 0)
+      (effects (font (size 1.27 1.27)) hide)
+    )
+    (property "Value" "+5V" (id 1) (at 111.76 118.11 90)
+      (effects (font (size 1.27 1.27)) (justify right))
+    )
+    (property "Footprint" "" (id 2) (at 119.38 118.11 0)
+      (effects (font (size 1.27 1.27)) hide)
+    )
+    (property "Datasheet" "" (id 3) (at 119.38 118.11 0)
+      (effects (font (size 1.27 1.27)) hide)
+    )
