File: ch32v003/tinybadapple/tinybadapple.kicad_sch (KiCad schematic)
At the start: 9 parts, among them J1 USB_C_Receptacle_USB2.0, U1 RS3236-3.3YUTDN4, U2 ZD25WQ16BUIGR, U3 CH32V003F4U6

Commit message: Bump versions.
Parts:
- removed C1, C2, C?: 10u, Capacitor_SMD:C_0402_1005Metric, symbol Device:C
- removed U1: RS3236-3.3YUTDN4, cnhardware:xdfn-reg, symbol Regulator_Linear:NCP115AMX250TCG
- added C3, C4: 4.7u, Resistor_SMD:R_0402_1005Metric, symbol Device:C
- added J2: APPLE, artwork:apple, symbol artwork:artwork
- added R3, R4, R5, R6: 1.5k, Resistor_SMD:R_0402_1005Metric, symbol Device:R
- added U1: 3.3vReg, cnhardware:xdfn-reg, symbol Regulator_Linear:NCP115AMX120TCG
- R1, R2: LCSC C105872 -> C25905
- U2: value ZD25WQ16BUIGR -> 25WQ32; footprint Package_SON:SON-8-1EP_3x2mm_P0.5mm_EP1.4x1.6mm -> cnhardware:USON8-LINE(2x3); LCSC C2983691 -> C5258281
Connections:
- net GND: now also J1.A8 (SBU1), C3.1, C4.1, U1.2 (GND), U1.5 (GND)
- net VDD: now also C3.2, U1.1 (OUT)
- net D+: now reaches J1.A6 (D+)
- net D+: now also J1.B6 (D+), U3.5 (PD0/T1CH1N/OPN1/SDA/UTX)
- net D-: now reaches J1.A7 (D-)
- net D-: now also J1.B7 (D-), U3.2 (PA1/OSCI/A1/T1CH2/OPN0)
- net SBU2: now reaches J1.B8 (SBU2)
- net SBU2: now also R3.2, R4.2, R5.2, R6.2
- net FIOB: now reaches U3.10 (PC3/T1CH3/T1CHIN/UCTS)
- net FIOB: now also U2.7 (IO3)
- net SCK: now reaches U3.11 (PC4/A2/T1CH4/MCO/T1CH1CH2N)
- net SCK: now also U2.6 (CLK)
- net at U3.13 (PC6/MOSI/T1CH1CH3/UCTS/SDA): now also R5.1
- net SS: now reaches U3.14 (PC7/MISO/T1CH2/T2CH2/URTS)
- net SS: now also U2.1 (~{CS})
- net SWIO: now reaches U3.15 (PD1/SWIO/AETR/T1CH3/SCL/URX)
- net at U3.16 (PD2/A3/T1CH1/T2CH3/T1CH2N): now also R6.1
- net at U3.17 (PD3/A4/T2CH2/AETR/UCTS/T1CH4): now also R4.1
- net at U3.19 (PD5/A5/UTX/T2CH4/URX): now also U3.20 (PD6/A7/URX/T2CH3/UTX), R3.1
- net MOSI: now reaches U3.7 (PC0/T2CH3/UTX/NSS/T1CH3)
- net MOSI: now also U2.5 (DI(IO0))
- net MISO: now reaches U3.8 (PC1/SDA/NSS/T2CH4/T2CH1ETR/T1BKIN/URX)
- net MISO: now also U2.2 (DO(IO1))
- net FIOA: now reaches U3.9 (PC2/SCL/URTS/T1BKIN/AETR/T2CH2/T1ETR)
- net FIOA: now also U2.3 (IO2)
- net VBUS renamed +5V
- net +5V: now also C4.2, U1.3 (EN), U1.4 (IN)
Other:
- note added: "How to generate NTSC?"
- note added: "IRE: 741+286mV White, 286mV Black, 0V Sync"
- note removed: "Can this work with an 8mbit prom? There be a tiny one."

Commit message: As ordered.
Parts:
- added J3, J4, J5, J6: ~, TestPoint:TestPoint_Pad_1.0x1.0mm, symbol Connector:Conn_01x01_Female
Connections:
- net D-: now also U3.1 (PD7/NRST/T2CH4/OPP1/UCK); no longer U3.2 (PA1/OSCI/A1/T1CH2/OPN0)
- net SWIO: now also J6.1 (Pin_1)
- net at U3.12 (PC5/SCK/T1ETR/T2CH1ETR/SCL/UCK/T1CH3): now also J5.1 (Pin_1)
- net at U3.3 (PA2/OSCO/A0/T1CH2N/OPP0/AETR2): now also J4.1 (Pin_1)
- new net: J3.1 (Pin_1), U3.2 (PA1/OSCI/A1/T1CH2/OPN0)
Changed lines of the file:
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@@
+    (stroke (width 0) (type default) (color 0 0 0 0))
+  )
+  (wire (pts (xy 134.62 67.31) (xy 106.68 67.31))
     (stroke (width 0) (type default) (color 0 0 0 0))
   )
@@
     (stroke (width 0) (type default) (color 0 0 0 0))
   )
+  (wire (pts (xy 106.68 67.31) (xy 106.68 74.93))
+    (stroke (width 0) (type default) (color 0 0 0 0))
+  )
   (wire (pts (xy 78.74 68.58) (xy 80.01 68.58))
     (stroke (width 0) (type default) (color 0 0 0 0))
   )
+  (wire (pts (xy 114.3 69.85) (xy 134.62 69.85))
+    (stroke (width 0) (type default) (color 0 0 0 0))
+  )
   (wire (pts (xy 232.41 67.31) (xy 232.41 64.77))
     (stroke (width 0) (type default) (color 0 0 0 0))
@@
   )
   (wire (pts (xy 228.6 67.31) (xy 232.41 67.31))
+    (stroke (width 0) (type default) (color 0 0 0 0))
+  )
+  (wire (pts (xy 114.3 74.93) (xy 114.3 69.85))
     (stroke (width 0) (type default) (color 0 0 0 0))
   )
@@
     )
   )
+  (global_label "SWIO" (shape input) (at 118.11 97.79 0) (fields_autoplaced)
+    (effects (font (size 1.27 1.27)) (justify left))
+    (property "Intersheet References" "${INTERSHEET_REFS}" (id 0) (at 125.1193 97.7106 0)
+      (effects (font (size 1.27 1.27)) (justify left) hide)
+    )
+  )
   (global_label "D-" (shape input) (at 80.01 74.93 0) (fields_autoplaced)
     (effects (font (size 1.27 1.27)) (justify left))
@@
     )
   )
-  (global_label "D-" (shape input) (at 134.62 67.31 180) (fields_autoplaced)
-    (effects (font (size 1.27 1.27)) (justify right))
-    (property "Intersheet References" "${INTERSHEET_REFS}" (id 0) (at 129.3645 67.2306 0)
-      (effects (font (size 1.27 1.27)) (justify right) hide)
-    )
-  )
   (global_label "FIOA" (shape input) (at 228.6 34.29 0) (fields_autoplaced)
     (effects (font (size 1.27 1.27)) (justify left))
@@
     )
   )
+  (global_label "D-" (shape input) (at 134.62 64.77 180) (fields_autoplaced)
+    (effects (font (size 1.27 1.27)) (justify right))
+    (property "Intersheet References" "${INTERSHEET_REFS}" (id 0) (at 129.3645 64.6906 0)
+      (effects (font (size 1.27 1.27)) (justify right) hide)
+    )
+  )
   (global_label "MOSI" (shape input) (at 134.62 80.01 180) (fields_autoplaced)
     (effects (font (size 1.27 1.27)) (justify right))
@@
     (pin "1")
     (pin "2")
+  )
+  (symbol (lib_id "Connector:Conn_01x01_Female") (at 113.03 97.79 180) (unit 1)
+    (in_bom yes) (on_board yes) (fields_autoplaced)
+    (property "Reference" "J6" (id 0) (at 113.665 93.633 0))
+    (property "Value" "~" (id 1) (at 113.665 96.1699 0))
+    (property "Footprint" "TestPoint:TestPoint_Pad_1.0x1.0mm" (id 2) (at 113.03 97.79 0)
+      (effects (font (size 1.27 1.27)) hide)
+    )
+    (property "Datasheet" "~" (id 3) (at 113.03 97.79 0)
+      (effects (font (size 1.27 1.27)) hide)
+    )
+    (pin "1")
   )
   (symbol (lib_id "Device:R") (at 245.11 67.31 90) (unit 1)
@@
     )
     (property "Datasheet" "" (id 3) (at 267.97 27.94 0)
+      (effects (font (size 1.27 1.27)) hide)
+    )
+    (pin "1")
+  )
+  (symbol (lib_id "Connector:Conn_01x01_Female") (at 114.3 80.01 270) (unit 1)
+    (in_bom yes) (on_board yes) (fields_autoplaced)
+    (property "Reference" "J4" (id 0) (at 115.5192 78.5403 90)
+      (effects (font (size 1.27 1.27)) (justify left))
+    )
+    (property "Value" "~" (id 1) (at 115.5192 81.0772 90)
+      (effects (font (size 1.27 1.27)) (justify left))
+    )
+    (property "Footprint" "TestPoint:TestPoint_Pad_1.0x1.0mm" (id 2) (at 114.3 80.01 0)
+      (effects (font (size 1.27 1.27)) hide)
+    )
+    (property "Datasheet" "~" (id 3) (at 114.3 80.01 0)
       (effects (font (size 1.27 1.27)) hide)
     )
@@
     (pin "1")
   )
+  (symbol (lib_id "Connector:Conn_01x01_Female") (at 106.68 80.01 270) (unit 1)
+    (in_bom yes) (on_board yes) (fields_autoplaced)
+    (property "Reference" "J3" (id 0) (at 107.8992 78.5403 90)
+      (effects (font (size 1.27 1.27)) (justify left))
+    )
+    (property "Value" "~" (id 1) (at 107.8992 81.0772 90)
+      (effects (font (size 1.27 1.27)) (justify left))
+    )
+    (property "Footprint" "TestPoint:TestPoint_Pad_1.0x1.0mm" (id 2) (at 106.68 80.01 0)
+      (effects (font (size 1.27 1.27)) hide)
+    )
+    (property "Datasheet" "~" (id 3) (at 106.68 80.01 0)
+      (effects (font (size 1.27 1.27)) hide)
+    )
+    (pin "1")
+  )
   (symbol (lib_id "power:GND") (at 267.97 35.56 0) (unit 1)
     (in_bom yes) (on_board yes) (fields_autoplaced)
@@
     )
     (property "Datasheet" "" (id 3) (at 256.54 27.94 0)
+      (effects (font (size 1.27 1.27)) hide)
+    )
+    (pin "1")
+  )
+  (symbol (lib_id "Connector:Conn_01x01_Female") (at 233.68 85.09 0) (unit 1)
+    (in_bom yes) (on_board yes) (fields_autoplaced)
+    (property "Reference" "J5" (id 0) (at 234.3912 84.2553 0)
+      (effects (font (size 1.27 1.27)) (justify left))
+    )
+    (property "Value" "~" (id 1) (at 234.3912 86.7922 0)
+      (effects (font (size 1.27 1.27)) (justify left))
+    )
+    (property "Footprint" "TestPoint:TestPoint_Pad_1.0x1.0mm" (id 2) (at 233.68 85.09 0)
+      (effects (font (size 1.27 1.27)) hide)
+    )
+    (property "Datasheet" "~" (id 3) (at 233.68 85.09 0)
       (effects (font (size 1.27 1.27)) hide)
     )
@@
       (reference "J2") (unit 1) (value "APPLE") (footprint "artwork:apple")
     )
+    (path "/c64a3406-1a36-4915-a3e4-838238f67d3b"
+      (reference "J3") (unit 1) (value "~") (footprint "TestPoint:TestPoint_Pad_1.0x1.0mm")
+    )
+    (path "/6da30ab9-72c8-4572-aedc-2aae74193b76"
+      (reference "J4") (unit 1) (value "~") (footprint "TestPoint:TestPoint_Pad_1.0x1.0mm")
+    )
+    (path "/e551905b-d1db-4035-bbf0-a8a4b92c89ed"
+      (reference "J5") (unit 1) (value "~") (footprint "TestPoint:TestPoint_Pad_1.0x1.0mm")
+    )
+    (path "/33b111ed-515c-4424-9087-dad7b2e358c8"
+      (reference "J6") (unit 1) (value "~") (footprint "TestPoint:TestPoint_Pad_1.0x1.0mm")
+    )
     (path "/674d720e-b431-4d5b-839c-b1b425002728"

Commit message: Update bad apple with tighter constraints on USB.
Parts:
- removed J5: ~, TestPoint:TestPoint_Pad_1.0x1.0mm, symbol Connector:Conn_01x01_Female
- J1: footprint Connector_USB:USB_C_Receptacle_HRO_TYPE-C-31-M-12 -> cnhardware:USB_C_MOD_Receptacle_HRO_TYPE-C-31-M-12
Connections:
- net D-: now also R4.2, U3.18 (PD4/A7/UCK/T2CH1ETR/OPO/T1CH4ETR); no longer U3.1 (PD7/NRST/T2CH4/OPP1/UCK)
- net SBU2: now also U3.16 (PD2/A3/T1CH1/T2CH3/T1CH2N); no longer R4.2
- net at R4.1: now also U3.19 (PD5/A5/UTX/T2CH4/URX); no longer U3.17 (PD3/A4/T2CH2/AETR/UCTS/T1CH4)
- net at R3.1, U3.20 (PD6/A7/URX/T2CH3/UTX): no longer U3.19 (PD5/A5/UTX/T2CH4/URX)
- net at R6.1: now also U3.17 (PD3/A4/T2CH2/AETR/UCTS/T1CH4); no longer U3.16 (PD2/A3/T1CH1/T2CH3/T1CH2N)
Other:
- moved on the sheet: R3
