File: esp32s2-funprog2/esp32s2-funprog2.kicad_sch (KiCad schematic)
At the start: 59 parts, among them J1 OPGM, J2 PGM, J3 USB_C_Receptacle_USB2.0, J4 MOUNT, J5 MOUNT, Q1 SE4625-PandN, Q2 SE4625-PandN, Q3 AP2302B, SW1 TS-1187A-B-A-B, U1 ESP32-S2, U2 AP1117-33, Y1 40MHz

Commit message: Tweaking design
Other:
- note removed: "TODO: Add 5705 Monitoring"
- moved on the sheet: D2, U2
Changed lines of the file:
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@@
     (stroke (width 0) (type default))
   )
-  (text "UNTESTED" (at 16.51 22.86 0)
-    (effects (font (size 5 5)) (justify left bottom))
-  )
-  (text "TODO: Add 5705 Monitoring" (at 82.55 147.32 0)
+  (text "UNTESTED" (at 177.8 172.72 0)
     (effects (font (size 5 5)) (justify left bottom))
   )
@@
     )
   )
-  (global_label "VBUS" (shape input) (at 171.45 77.47 180) (fields_autoplaced)
+  (global_label "VBUS" (shape input) (at 191.77 110.49 180) (fields_autoplaced)
     (effects (font (size 1.27 1.27)) (justify right))
-    (property "Intersheetrefs" "${INTERSHEET_REFS}" (at 164.1383 77.5494 0)
+    (property "Intersheetrefs" "${INTERSHEET_REFS}" (at 184.4583 110.5694 0)
       (effects (font (size 1.27 1.27)) (justify right) hide)
     )
@@
     )
   )
-  (symbol (lib_id "Regulator_Linear:AP1117-33") (at 179.07 77.47 0) (unit 1)
+  (symbol (lib_id "Regulator_Linear:AP1117-33") (at 199.39 110.49 0) (unit 1)
     (in_bom yes) (on_board yes) (dnp no) (fields_autoplaced)
-    (property "Reference" "U2" (at 179.07 69.85 0)
+    (property "Reference" "U2" (at 199.39 102.87 0)
       (effects (font (size 1.27 1.27)))
     )
-    (property "Value" "AP1117-33" (at 179.07 72.39 0)
+    (property "Value" "AP1117-33" (at 199.39 105.41 0)
       (effects (font (size 1.27 1.27)))
     )
-    (property "Footprint" "Package_TO_SOT_SMD:SOT-223-3_TabPin2" (at 179.07 72.39 0)
+    (property "Footprint" "Package_TO_SOT_SMD:SOT-223-3_TabPin2" (at 199.39 105.41 0)
       (effects (font (size 1.27 1.27)) hide)
     )
-    (property "Datasheet" "http://www.diodes.com/datasheets/AP1117.pdf" (at 181.61 83.82 0)
+    (property "Datasheet" "http://www.diodes.com/datasheets/AP1117.pdf" (at 201.93 116.84 0)
       (effects (font (size 1.27 1.27)) hide)
     )
-    (property "LCSC" "C6186" (at 179.07 77.47 0)
+    (property "LCSC" "C6186" (at 199.39 110.49 0)
       (effects (font (size 1.27 1.27)) hide)
     )
@@
     )
   )
-  (symbol (lib_id "power:GND") (at 179.07 85.09 0) (unit 1)
+  (symbol (lib_id "power:GND") (at 199.39 118.11 0) (unit 1)
     (in_bom yes) (on_board yes) (dnp no)
-    (property "Reference" "#PWR0129" (at 179.07 91.44 0)
+    (property "Reference" "#PWR0129" (at 199.39 124.46 0)
       (effects (font (size 1.27 1.27)) hide)
     )
-    (property "Value" "GND" (at 181.61 87.63 0)
+    (property "Value" "GND" (at 201.93 120.65 0)
       (effects (font (size 1.27 1.27)))
     )
-    (property "Footprint" "" (at 179.07 85.09 0)
+    (property "Footprint" "" (at 199.39 118.11 0)
       (effects (font (size 1.27 1.27)) hide)
     )
-    (property "Datasheet" "" (at 179.07 85.09 0)
+    (property "Datasheet" "" (at 199.39 118.11 0)
       (effects (font (size 1.27 1.27)) hide)
     )
@@
     )
   )
-  (symbol (lib_id "power:VDD") (at 186.69 77.47 270) (unit 1)
+  (symbol (lib_id "power:VDD") (at 207.01 110.49 270) (unit 1)
     (in_bom yes) (on_board yes) (dnp no) (fields_autoplaced)
-    (property "Reference" "#PWR0130" (at 182.88 77.47 0)
+    (property "Reference" "#PWR0130" (at 203.2 110.49 0)
       (effects (font (size 1.27 1.27)) hide)
     )
-    (property "Value" "VDD" (at 190.5 77.4699 90)
+    (property "Value" "VDD" (at 210.82 110.4899 90)
       (effects (font (size 1.27 1.27)) (justify left))
     )
-    (property "Footprint" "" (at 186.69 77.47 0)
+    (property "Footprint" "" (at 207.01 110.49 0)
       (effects (font (size 1.27 1.27)) hide)
     )
-    (property "Datasheet" "" (at 186.69 77.47 0)
+    (property "Datasheet" "" (at 207.01 110.49 0)
       (effects (font (size 1.27 1.27)) hide)
     )
@@
     )
   )
-  (symbol (lib_id "Device:LED_RAGB") (at 186.69 130.81 0) (unit 1)
+  (symbol (lib_id "Device:LED_RAGB") (at 185.42 156.21 0) (unit 1)
     (in_bom yes) (on_board yes) (dnp no) (fields_autoplaced)
-    (property "Reference" "D2" (at 186.69 118.11 0)
+    (property "Reference" "D2" (at 185.42 143.51 0)
       (effects (font (size 1.27 1.27)))
     )
-    (property "Value" "LED_RAGB" (at 186.69 120.65 0)
+    (property "Value" "LED_RAGB" (at 185.42 146.05 0)
       (effects (font (size 1.27 1.27)))
     )
-    (property "Footprint" "LED_SMD:LED_WS2812B-2020_PLCC4_2.0x2.0mm" (at 186.69 132.08 0)
+    (property "Footprint" "LED_SMD:LED_WS2812B-2020_PLCC4_2.0x2.0mm" (at 185.42 157.48 0)
       (effects (font (size 1.27 1.27)) hide)
     )
-    (property "Datasheet" "~" (at 186.69 132.08 0)
+    (property "Datasheet" "~" (at 185.42 157.48 0)
       (effects (font (size 1.27 1.27)) hide)
     )
-    (property "LCSC" "C965840" (at 186.69 130.81 0)
+    (property "LCSC" "C965840" (at 185.42 156.21 0)
       (effects (font (size 1.27 1.27)) hide)
     )
@@
     )
   )
-  (symbol (lib_id "power:VDD") (at 191.77 130.81 270) (unit 1)
+  (symbol (lib_id "power:VDD") (at 190.5 156.21 270) (unit 1)
     (in_bom yes) (on_board yes) (dnp no) (fields_autoplaced)
-    (property "Reference" "#PWR07" (at 187.96 130.81 0)
+    (property "Reference" "#PWR07" (at 186.69 156.21 0)
       (effects (font (size 1.27 1.27)) hide)
     )
-    (property "Value" "VDD" (at 195.58 130.81 90)
+    (property "Value" "VDD" (at 194.31 156.21 90)
       (effects (font (size 1.27 1.27)) (justify left))
     )
-    (property "Footprint" "" (at 191.77 130.81 0)
+    (property "Footprint" "" (at 190.5 156.21 0)
       (effects (font (size 1.27 1.27)) hide)
     )
-    (property "Datasheet" "" (at 191.77 130.81 0)
+    (property "Datasheet" "" (at 190.5 156.21 0)
       (effects (font (size 1.27 1.27)) hide)
     )

Commit message: Update funprog
Parts:
- added C20: 10p, Capacitor_SMD:C_0402_1005Metric, symbol Device:C
- added C21: 330p, Capacitor_SMD:C_0402_1005Metric, symbol Device:C
- added R16: 49.9, Resistor_SMD:R_0402_1005Metric, symbol Device:R
- added R17, R18: 100k, Resistor_SMD:R_0402_1005Metric, symbol Device:R
- added R19: 20m, Resistor_SMD:R_1206_3216Metric, symbol Device:R
- added R20: 10k, Resistor_SMD:R_0402_1005Metric, symbol Device:R
- added R21: 200m, Resistor_SMD:R_1206_3216Metric, symbol Device:R
- added R22: 2, Resistor_SMD:R_1206_3216Metric, symbol Device:R
- added R23: 20, Resistor_SMD:R_1206_3216Metric, symbol Device:R
- added U3: LM321, Package_TO_SOT_SMD:SOT-23-5, symbol Amplifier_Operational:LM321
- added U4: ZDT6790TA, Package_TO_SOT_SMD:SOT-223-8, symbol cnhardware:ZDT6790-COMPLEMENTARY-BJT
- added U5: INA199A2DCKR, Package_TO_SOT_SMD:SOT-363_SC-70-6, symbol Amplifier_Current:INA199xxDCK
Connections:
- net DAC1: now also C21.1, U3.1 (+)
- net GND: now also C21.2, R18.1, U3.2 (V-), U4.7 (CP), U4.8 (CP), U5.2 (GND)
- new net: U4.1 (EP), U4.3 (EN), U5.4 (+)
- new net: R16.2, U4.2 (BP), U4.4 (BN)
- new net: C20.2, R17.1, R18.2, U3.3 (-)
- new net: R16.1, U3.4
- new net +VSW: U3.5 (V+), U4.5 (CN), U4.6 (CN)
- new net OVMON: C20.1, R17.2, R19.1, R21.1, R22.1, R23.1, U5.5 (-)
Other:
- note added: "100 v/v -> .250mA * .020 = 5mV * 100 = 500mV"
- note added: "Class B Push-Pull follower"
- note added: "INA199A1 = 50v/v gain Max Current: 200mA For 0.5V swing, 20mOhm How to switch between current sense resistors?"
- note added: "VSW = 12V or 5V TODO: PSU TODO: Make VREF be 0.66ish V"
- moved on the sheet: A1, C1, C10, C11, C12, C13, C14, C15, C2, C3, C4, C5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

Commit message: Update with some progress on funprog2
Parts:
- added C22: 10u25v, Capacitor_SMD:C_0603_1608Metric, symbol Device:C
- added C23, C24, C25: 100n, Capacitor_SMD:C_0402_1005Metric, symbol Device:C
- added D3, D5, D6, D7: 1N5819WS, Diode_SMD:D_SOD-323, symbol Device:D
- added Q4, Q5: SE4625-PandN, cnhardware:DFN-6-2x2-SplitPad, symbol SE4625-PandN:SE4625-PandN
- added R24, R33, R34, R35, R36: 100k, Resistor_SMD:R_0402_1005Metric, symbol Device:R
- added R25, R37, R38, R39, R40: 4.7k, Resistor_SMD:R_0402_1005Metric, symbol Device:R
- added R26, R29: 5.1k, Resistor_SMD:R_0402_1005Metric, symbol Device:R
- added R27: 47k, Resistor_SMD:R_0402_1005Metric, symbol Device:R
- added R28, R32: 10k, Resistor_SMD:R_0402_1005Metric, symbol Device:R
- added R30, R31: 1k, Resistor_SMD:R_0402_1005Metric, symbol Device:R
- added U10, U11: DUAL-P-FET, Package_TO_SOT_SMD:SOT-23-6, symbol cnhardware:AP2625GY-VB-DUAL-P-FET
- added U6: MT3608, Package_TO_SOT_SMD:SOT-23-6, symbol Regulator_Switching:MT3608
- added U7, U8, U9: INA199A1DCKR, Package_TO_SOT_SMD:SOT-363_SC-70-6, symbol Amplifier_Current:INA199xxDCK
- D1: value D -> 1N5819WS; footprint Diode_SMD:D_SMA -> Diode_SMD:D_SOD-323; LCSC C8678 -> C191023
- R18: value 100k -> 1M; LCSC C25741 -> C26083
- R19: value 20m -> 33m; LCSC C7420010 -> C705566
- R20: value 10k -> 1k; LCSC C25744 -> C102748
- R21: value 200m -> 330m; LCSC C2911295 -> C341598
- R22: value 2 -> 3.3; LCSC C2936596 -> C140028
- R23: value 20 -> 33; LCSC C25362 -> C137308
- R7: value 10k -> 5.1k; LCSC C144807 -> C25905
- U5: value INA199A2DCKR -> INA199A1DCKR; LCSC C131913 -> C59135
Connections:
- net +VSW: now also D1.1 (K), C22.2, C23.1, C24.1, R24.2
- net 5VSW: now also Q4.3 (D2), Q4.8 (D2)
- net DAC1: no longer J1.4 (Pin_4)
- net GND: now also C22.1, C23.2, C24.2, C25.2, Q4.1 (S1), Q5.1 (S1), R25.1, R28.1, R32.1, U6.2 (GND), U7.2 (GND), U8.2 (GND), U9.2 (GND)
- net MIDBUS: no longer D1.1 (K), Q2.4 (S2)
- net MULTI2: no longer U1.7 (GPIO2)
- net OVMON: now also C20.2, R17.1, R18.2, U3.3 (-); no longer C20.1, R17.2, R19.1, R21.1, R22.1, R23.1, U5.5 (-)
- net VBUS: now also L2.1, Q4.4 (S2), Q4.5 (G2), Q4.6 (D1), Q4.7 (D1), R29.1, R29.2, U6.5 (IN); no longer L2.2
- net VCCCTL5: now also Q4.2 (G1); no longer Q2.2 (G1)
- net VDD: no longer U1.27 (VDD3P3_RTC_IO)
- net VSW: no longer U1.15 (GPIO10)
- net at C16.1, C17.1, L3.2: no longer D1.2 (A)
- net at C16.2, C17.2, Q3.2 (D): no longer L2.1
- net DYNRAIL: now reaches U4.1 (EP), U4.3 (EN), U5.4 (+)
- net DYNRAIL: now also R19.2, R21.2, R22.2, R23.2, Q5.4 (S2), Q5.5 (G2), Q5.6 (D1), Q5.7 (D1), R26.1, R26.2, U7.4 (+), U8.4 (+), U9.4 (+)
- net at U1.41 (GPIO37): now also R31.2
- net at U1.42 (GPIO38): now also R30.2
- net at U1.43 (MTCK): now also R20.2
- net at R20.1: now also D2.1 (RK)
- net VREF06: now reaches U5.1 (REF)
- net VREF06: now also R27.1, R28.2, U7.1 (REF), U8.1 (REF), U9.1 (REF)
- net +3.3VA: now reaches U5.3 (V+)
- net +3.3VA: now also U1.27 (VDD3P3_RTC_IO), R27.2, U7.3 (V+), U8.3 (V+), U9.3 (V+)
- net IMN0: now reaches U5.6
- net DYNVSW: now reaches Q2.3 (D2), Q2.8 (D2)
- net at D2.3 (GK): now also R30.1
- net at D2.4 (BK): now also R31.1
- new net: D5.1 (K), R19.1, R35.2, U10.5 (S1), U5.5 (-)
- new net: D6.1 (K), R22.1, R34.2, U11.5 (S1), U8.5 (-)
- new net: D6.2 (A), R34.1, R39.2, U11.1 (G1)
- new net: D7.1 (K), R23.1, R33.1, U11.2 (S2), U9.5 (-)
- new net: D7.2 (A), R33.2, R40.2, U11.3 (G2)
- new net: D1.2 (A), L2.2, U6.1 (SW)
- new net: R24.1, R25.2, U6.3 (FB)
- new net: D5.2 (A), R35.1, R38.2, U10.1 (G1)
- new net: D3.2 (A), R36.2, R37.2, U10.3 (G2)
- new net: D3.1 (K), R21.1, R36.1, U10.2 (S2), U7.5 (-)
- new net BOOSTEN: U6.4 (EN)
- new net DYNCTL: Q2.2 (G1), R32.2
- new net IMN1: U7.6
- new net IMN2: U8.6
- new net IMN3: U9.6
- new net MODE_0: R38.1
- new net MODE_1: R37.1
- new net MODE_2: R39.1
- new net MODE_3: R40.1
- new net OVOUT: C20.1, C25.1, R17.2, U10.4 (D2), U10.6 (D1), U11.4 (D2), U11.6 (D1)
Other:
- note added: "50 v/v -> 300mA * .033 = 10mV * 50 = 500mV"
- note added: "Optional Boost Disable = 4.5v Enable = 13.3v Imax = 300mA"
- note added: "P-N network for all MODE control * Need negative rail to push against."
- note added: "VREF = 0.58v"
- note removed: "100 v/v -> .250mA * .020 = 5mV * 100 = 500mV"
- note removed: "INA199A1 = 50v/v gain Max Current: 200mA For 0.5V swing, 20mOhm How to switch between current sense resistors?"
- note removed: "VSW = 12V or 5V TODO: PSU TODO: Make VREF be 0.66ish V"
- moved on the sheet: A1, C1, C16, C17, C18, C19, C2, C20, C21, C3, C4, C7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
