File: ch32v003/ch32v003_rbo12864h-wfi/ch32v003_rbo12864h-wfi.kicad_sch (KiCad schematic)
At the start: 17 parts, among them J1 RBO12864H, J2 LED, J3 USB_C_Receptacle_USB2.0, J5 PGM, U1 XC6206P332MR-G, U2 CH32V003F4U6

Commit message: Update order for microlcd - 3digit
Parts:
- C3: LCSC C368809 -> C23733

Commit message: Add note!
Connections:
- no-connect marks 0 -> 2
Other:
- note added: "Default USB configuration for rv003usb. Reference only for LOW SPEED only."
- note added: "R2 only for current measurement not needed. VDD connected to PC7 for power control. (This could be tied to VCC)"
- note added: "Tested OK 2024-10-16 C. Lohr"
- note added: "VDD"
- moved on the sheet: C2, C4, C5, J1, J2, J5, R2, R6
