File: esp32s2-funprog3/esp32s2-funprog.kicad_sch (KiCad schematic)
At the start: 97 parts, among them J1 OPGM, J2 PGM, J3 USB_C_Receptacle_USB2.0, J4 MOUNT, J5 MOUNT, Q1 SE4625-PandN, Q2 SE4625-PandN, Q3 DWL336C, Q4 2N7002, Q6 2N7002KDW, Q7 MOT2302, SW1 TS-1187A-B-A-B, U1 ESP32-S2, U10 LM321, U11 ZDT6790TA, U12 COS4514, U14 AT8837, U15 AT8837, U16 AT8837, U2 XC6206P332, U3 MT3608, U4 XC6206P332, U5 COSNE5532, U6 XC6206P332, U8 HP3000, U9 AT8837, Y1 40MHz

Commit message: Bump for the rev3
Connections:
- net at R15.1: now also U1.50 (GPIO45); no longer U1.47 (MTMS)
- net at R13.1: now also U1.47 (MTMS); no longer U1.50 (GPIO45)
