File: ch32x035/OLED_TRANSPARENT_128x128/OLED_TRANSPARENT_128x128.kicad_sch (KiCad schematic)
At the start: 18 parts, among them J1 OLED, J2 USB_C_Receptacle_USB2.0, U2 CH32V003F4U6, U3 XC6206P332MR-G

Commit message: Move project around
Parts:
- removed C1, C7: 1u, Resistor_SMD:R_0402_1005Metric, symbol Device:C
- removed R5: 1.5k, Resistor_SMD:R_0402_1005Metric, symbol Device:R
- removed U2: CH32V003F4U6, Package_DFN_QFN:QFN-20-1EP_3x3mm_P0.4mm_EP1.65x1.65mm, symbol CH32V003F4U6:CH32V003F4U6
- added U1: ~, Package_DFN_QFN:QFN-28-1EP_4x4mm_P0.4mm_EP2.6x2.6mm, symbol cnhardware:CH32X035G8U6
- C3: footprint Resistor_SMD:R_0402_1005Metric -> Capacitor_SMD:C_0805_2012Metric; LCSC C23733 -> C1779
- C5, C6: value 1u -> 4.7u; footprint Resistor_SMD:R_0402_1005Metric -> Capacitor_SMD:C_0805_2012Metric; LCSC C52923 -> C1779
- R1: LCSC C25867 -> C26083
Connections:
- net +5V: now also U1.2 (VDD)
- net CS: now also U1.7 (PA2/TX2/T2C3/O2O1/T2ET_/A2)
- net D+: now also U1.27 (PC17/UDP/RTS1/TX2_/I2C_/RX4_/T1ET/PC10)
- net D-: now also U1.26 (PC16/UDM/T1C4/TX4_/I21C_/RX4_/CTS1/PC11)
- net DC: now also U1.9 (PA4/CS/O2O0/T3C2_/A4)
- net GND: now also C5.1, C6.1, R1.1, U1.29
- net RST: now also U1.8 (PA3/T2C4/O1O0/T3C1_/RX2/A3)
- net SCL: now also U1.10 (PA5/SCK/TX4_/O2N0/A2)
- net SDA: now also U1.11 (PA6/MISO/T3C1/T1BK_/O1N0/A6), U1.12 (PA7/MOSI/T3C2/T1C1N_/TX1_/O2P0/A7)
- net VDD: now also C4.1
- net VCOMH: now reaches J1.10 (Pin_10)
- net VCOMH: now also C5.2
- net VPP: now reaches J1.11 (Pin_11)
- net VPP: now also C6.2
- new net DCK: U1.24 (PC19/DCK/T2C1_/T3C1_/I2C_/RX3/C1P0)
- new net DIO: U1.25 (PC18/DIO/TX3_/T2C1N_/T3C2_/I2C_/T1ET_)
Other:
- note removed: "BS1: 1: I2C / 0: SPI"
- note removed: "Do not use PC2/PC3"
- moved on the sheet: C4, TP1, TP2, TP3

Commit message: Bump design
Parts:
- removed TP1: GND, TestPoint:TestPoint_Pad_D1.0mm, symbol Connector:TestPoint
- removed TP2: SWIO, TestPoint:TestPoint_Pad_D1.0mm, symbol Connector:TestPoint
- removed TP3: VDD, TestPoint:TestPoint_Pad_D1.0mm, symbol Connector:TestPoint
- added D1: 1N5819WS, Diode_SMD:D_SOD-323, symbol Device:D_Schottky
- added J3: PGM, Connector_PinHeader_2.54mm:PinHeader_1x04_P2.54mm_Vertical, symbol Connector_Generic:Conn_01x04
- added L1: 4.7uH 500mA, Inductor_SMD:L_0805_2012Metric, symbol Device:L
- added Q1: AO3400A, Package_TO_SOT_SMD:SOT-23, symbol Device:Q_NMOS_GSD
- added R2, R7: 5.1k, Resistor_SMD:R_0402_1005Metric, symbol Device:R
- added R5: 1M, Resistor_SMD:R_0402_1005Metric, symbol Device:R
- added R6: NP, Resistor_SMD:R_0402_1005Metric, symbol Device:R
- added SW1: Download, Button_Switch_SMD:SW_SPST_TL3342, symbol Switch:SW_SPST
- J1: footprint Connector_FFC-FPC:Hirose_FH26-15S-0.3SHW_2Rows-15Pins-1MP_P0.60mm_Horizontal -> cnhardware:FPC_BOTTOM_P0.5mm_FLIP_JUSHUO; LCSC (none) -> C561387
- R1: value 1.5k -> 1M
Connections:
- net +5V: now also J3.1 (Pin_1), L1.1; no longer U1.2 (VDD)
- net CS: now also U1.15 (PB4/T2C4_/T3C1_/T2BK_/RX3/O1P2); no longer U1.7 (PA2/TX2/T2C3/O2O1/T2ET_/A2)
- net D+: now also R7.2
- net DC: now also U1.13 (PB0/TX4/T1C2N_/O1PO/A8); no longer U1.9 (PA4/CS/O2O0/T3C2_/A4)
- net DCK: now also J3.2 (Pin_2)
- net DIO: now also J3.3 (Pin_3)
- net GND: now also J1.13 (Pin_13), J1.14 (Pin_14), R4.1, J3.4 (Pin_4), Q1.2 (S), R2.2, R6.1; no longer R4.2
- net RST: now also U1.14 (PB3/TX3/T2C3_/T2C3N_/O2P1); no longer U1.8 (PA3/T2C4/O1O0/T3C1_/RX2/A3)
- net VDD: now also U1.2 (VDD), SW1.1 (A)
- net VPP: now also D1.1 (K), R5.2
- net CC2: now reaches J2.B5 (CC2)
- net CC2: now also U1.1 (PC15/CC2/T2C3_/T1ET_), R2.1; no longer R4.1
- net VPPMON: now reaches U1.16 (PB1/T1C3N_/RX4/O2N1/A9/PB5/O101/T3C2_/T1BK)
- net VPPMON: now also R5.1, R6.2
- net VSW: now reaches U1.20 (PB9/T1C1/MCO/TX4_)
- net VSW: now also R4.2, Q1.1 (G)
- net CC1: now reaches U1.28 (PC14/CC/T1C3_/T2C2_)
- net CC1: now also J2.A5 (CC1), R3.1
- new net: D1.2 (A), L1.2, Q1.3 (D)
- new net: R7.1, SW1.2 (B)
Other:
- note added: "UNTESTED"
