File: ch32v003/aluminium-beads/aluminium-beads.kicad_pcb (KiCad board)
At the start: 2 copper layers, 35 x 50 mm, 41 parts, among them J1 GND, J2 SWIO, J3 5V, J4 5V, J5 GND, J6 GND, J7 5V, J8 GND, J9 GND, Q1 Q_NMOS_GSD, Q2 Q_NMOS_GSD, Q3 Q_NMOS_GSD, Q4 Q_NMOS_GSD, U2 CH32V003FxPx

Commit message: Bump
Parts:
- D6: value LED -> LED_1W_3W
Routing:
- net GND: track 322.0 -> 328.4 mm
- net Net-(D7-A): track 5.22 -> 5.94 mm
- net +5V: track 171.9 -> 171.3 mm
- net Net-(D3-A): track 4.88 -> 5.39 mm
