File: ch32v003/0.47incholed-wak/0.47incholed-wak.kicad_pcb (KiCad board)
At the start: 2 copper layers, 11.5 x 9.9 mm, 17 parts, among them J2 USB_C_Receptacle_USB2.0, U2 CH32V003F4U6, U3 3.3vReg

Commit message: Note as printed.
Other:
- board text added: "Tested OK. 11/11/1024"
Changed lines of the file:
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@@
 		)
 		(property "Footprint" "Resistor_SMD:R_0402_1005Metric"
-			(at 0 0 360)
+			(at 0 0 0)
 			(layer "F.Fab")
 			(hide yes)
@@
 		)
 		(property "Datasheet" ""
-			(at 0 0 360)
+			(at 0 0 0)
 			(layer "F.Fab")
 			(hide yes)
@@
 		)
 		(property "Description" ""
-			(at 0 0 360)
+			(at 0 0 0)
 			(layer "F.Fab")
 			(hide yes)
@@
 		)
 	)
+	(gr_text "Tested OK. 11/11/1024"
+		(at 155.69 74.83 0)
+		(layer "Cmts.User")
+		(effects
+			(font
+				(size 1 1)
+				(thickness 0.15)
+			)
+			(justify left bottom)
+		)
+	)
