File: ch32v003/0.47SAOB/0.47SAOB.kicad_pcb (KiCad board)
At the start: 2 copper layers, 11 x 23.2 mm, 11 parts, among them J1 SAO, SW1 TS-1187A-B-A-B, SW2 TS-1187A-B-A-B, U2 CH32V003F4U6

Commit message: General updates for order
Parts:
- added R1: 3.3k, Resistor_SMD:R_0402_1005Metric, F.Cu at (192.1, 78.8)
- moved J1 0.26 mm to (195.8, 83.8), turned to -100 degrees
Routing:
- net GND: track 38.5 -> 34.8 mm, vias 19 -> 21
- net VDD: track 18.0 -> 16.1 mm
Other:
- board text added: "0.47SAOB cnhardware revA"
- board text removed: "0.47SAOB cnhardware"
