File: ch32v006/badapple006-128-96-gpio/badapple006.kicad_pcb (KiCad board)
At the start: 2 copper layers, 32 x 30 mm, 33 parts, among them J10 OLEDGPIO, J11 PGM, J2 USB_C_Receptacle_USB2.0, J6 RFO, J7 RFA, J8 APPLE, J9 RB132-2896GSWHG_01, U1 CH32V006F8U6, U2 XC6206P332, Y1 24MHz

Commit message: General updates for order
Parts:
- moved R4 0.31 mm to (100.4, 95.4), turned to 150 degrees
Routing:
- net O_D/#C: track 37.7 -> 38.3 mm
- net GND: vias 48 -> 53
Other:
- board text added: "badapple006-128-96-gpio rev -"
