File: ch32v006/badapple006-flip/badapple006.kicad_sch (KiCad schematic)
At the start: 25 parts, among them J1 OLED, J2 USB_C_Receptacle_USB2.0, J3 PG, J4 3v3, J5 GND, J6 RFO, J7 RFA, J8 APPLE, U1 CH32V006F8U6, U2 XC6206P332, Y1 24MHz

Commit message: Bump
Parts:
- added J10: OVDD, TestPoint:TestPoint_Pad_D1.0mm, symbol Connector_Generic:Conn_01x01
- added J9: RFO2, TestPoint:TestPoint_Pad_D1.0mm, symbol Connector_Generic:Conn_01x01
- C1, C5: footprint Capacitor_SMD:C_0402_1005Metric -> Capacitor_SMD:C_0603_1608Metric; LCSC C72203 -> C23630
- C2, C6: value 4.7u16v -> 2.2u16v; LCSC C77045 -> C23630
- C4: value 4.7u16v -> 2.2u16v; footprint Capacitor_SMD:C_0402_1005Metric -> Capacitor_SMD:C_0603_1608Metric; LCSC C72203 -> C23630
- J3, J4, J5, J6, J7, J8: now left out of the parts list
Connections:
- net OVDD: now also U1.10 (PC3/T1/T2), J10.1 (Pin_1); no longer U1.11 (PC4/T1C1_/T1/MCO/A2)
- net RES: now also U1.7 (PC0/T1C1N_/T1/T2/TX_/MOSI_); no longer U1.10 (PC3/T1/T2)
- net RFO2: now reaches U1.12 (PC5/T1C2_/T1/T2/TX_/SCK)
- net RFO2: now also U1.11 (PC4/T1C1_/T1/MCO/A2), U1.13 (PC6/T1C3_/T1/RX_/MOSI), J9.1 (Pin_1)

Commit message: Mild tweaks
Parts:
- added D1, D2: LED, LED_SMD:LED_0603_1608Metric, symbol Device:LED
- added R5: J, Resistor_SMD:R_0402_1005Metric, symbol Device:R
Connections:
- net VBUS: now also R5.1
- net REDCOLOR: now reaches U1.1 (PD7/RST/R2C4/OPP1/PA4/U2TX_/OPN2)
- net REDCOLOR: now also D1.1 (K)
- new net: D1.2 (A), D2.1 (K)
- new net: D2.2 (A), R5.2

Commit message: Bump update
Connections:
- net SBU: now reaches U1.16 (PD2/T1/T2/U2TX_/A3)
- net SBU: now also J2.A8 (SBU1), J2.B8 (SBU2)
Changed lines of the file:
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@@
+	(wire
+		(pts
+			(xy 107.95 129.54) (xy 107.95 132.08)
+		)
+		(stroke
+			(width 0)
+			(type default)
+		)
+	)
 	(wire
 		(pts
@@
 		)
 	)
+	(global_label "SBU"
+		(shape input)
+		(at 129.54 97.79 0)
+		(fields_autoplaced yes)
+		(effects
+			(font
+				(size 1.27 1.27)
+			)
+			(justify left)
+		)
+		(property "Intersheetrefs" "${INTERSHEET_REFS}"
+			(at 136.3352 97.79 0)
+			(effects
+				(font
+					(size 1.27 1.27)
+				)
+				(justify left)
+				(hide yes)
+			)
+		)
+	)
 	(global_label "RFO"
 		(shape input)
@@
 		)
 	)
+	(global_label "SBU"
+		(shape input)
+		(at 163.83 45.72 0)
+		(fields_autoplaced yes)
+		(effects
+			(font
+				(size 1.27 1.27)
+			)
+			(justify left)
+		)
+		(property "Intersheetrefs" "${INTERSHEET_REFS}"
+			(at 170.6252 45.72 0)
+			(effects
+				(font
+					(size 1.27 1.27)
+				)
+				(justify left)
+				(hide yes)
+			)
+		)
+	)
 	(global_label "D+"
 		(shape input)
@@
 			(effects
 				(font
+					(size 1.27 1.27)
+				)
+				(justify left)
+				(hide yes)
+			)
+		)
+	)
+	(global_label "SBU"
+		(shape input)
+		(at 107.95 132.08 0)
+		(fields_autoplaced yes)
+		(effects
+			(font
+				(size 1.27 1.27)
+			)
+			(justify left)
+		)
+		(property "Intersheetrefs" "${INTERSHEET_REFS}"
+			(at 114.7452 132.08 0)
+			(effects
+				(font

Commit message: Fix BOM
Parts:
- J10, J3, J4, J5, J6, J7, J8, J9: now not fitted
- R5: value J -> 30; LCSC (none) -> C1091
- U1: LCSC (none) -> C42431288
Changed lines of the file:
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@@
 		(in_bom no)
 		(on_board yes)
-		(dnp no)
+		(dnp yes)
 		(fields_autoplaced yes)
 		(property "Reference" "J7"
@@
 		(in_bom no)
 		(on_board yes)
-		(dnp no)
+		(dnp yes)
 		(fields_autoplaced yes)
 		(property "Reference" "J6"
@@
 		(in_bom no)
 		(on_board yes)
-		(dnp no)
+		(dnp yes)
 		(fields_autoplaced yes)
 		(property "Reference" "J9"
@@
 		(in_bom no)
 		(on_board yes)
-		(dnp no)
+		(dnp yes)
 		(fields_autoplaced yes)
 		(property "Reference" "J4"
@@
 		(in_bom no)
 		(on_board yes)
-		(dnp no)
+		(dnp yes)
 		(fields_autoplaced yes)
 		(property "Reference" "J5"
@@
 		(in_bom no)
 		(on_board yes)
-		(dnp no)
+		(dnp yes)
 		(fields_autoplaced yes)
 		(property "Reference" "J8"
@@
 		(in_bom no)
 		(on_board yes)
-		(dnp no)
+		(dnp yes)
 		(fields_autoplaced yes)
 		(property "Reference" "J3"
@@
 			)
 		)
-		(property "Value" "J"
+		(property "Value" "30"
 			(at 64.77 73.66 0)
 			(effects
@@
 			)
 		)
-		(property "LCSC" ""
+		(property "LCSC" "C1091"
 			(at 62.23 72.39 0)
 			(effects
@@
 			)
 		)
+		(property "LCSC" "C42431288"
+			(at 128.27 46.99 0)
+			(effects
+				(font
+					(size 1.27 1.27)
+				)
+				(hide yes)
+			)
+		)
 		(pin "6"
 		)
@@
 		(in_bom no)
 		(on_board yes)
-		(dnp no)
+		(dnp yes)
 		(fields_autoplaced yes)
 		(property "Reference" "J10"

Commit message: Bump design
Parts:
- added J11: SDA, TestPoint:TestPoint_Pad_D1.0mm, symbol Connector_Generic:Conn_01x01
- J10: value OVDD -> SCL
Connections:
- net SCL: now also J10.1 (Pin_1)
- net SDA: now also J11.1 (Pin_1)
- net VDD: now also C5.1, J1.7 (Pin_7)
- removed net OVDD: C5.1, J1.7 (Pin_7), J10.1 (Pin_1), U1.10 (PC3/T1/T2)
Changed lines of the file:
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@@
 	(global_label "SCL"
 		(shape input)
+		(at 246.38 53.34 180)
+		(fields_autoplaced yes)
+		(effects
+			(font
+				(size 1.27 1.27)
+			)
+			(justify right)
+		)
+		(property "Intersheetrefs" "${INTERSHEET_REFS}"
+			(at 239.8872 53.34 0)
+			(effects
+				(font
+					(size 1.27 1.27)
+				)
+				(justify right)
+				(hide yes)
+			)
+		)
+	)
+	(global_label "SCL"
+		(shape input)
 		(at 220.98 41.91 180)
 		(fields_autoplaced yes)
@@
 		)
 	)
+	(global_label "SDA"
+		(shape input)
+		(at 246.38 59.69 180)
+		(fields_autoplaced yes)
+		(effects
+			(font
+				(size 1.27 1.27)
+			)
+			(justify right)
+		)
+		(property "Intersheetrefs" "${INTERSHEET_REFS}"
+			(at 239.8267 59.69 0)
+			(effects
+				(font
+					(size 1.27 1.27)
+				)
+				(justify right)
+				(hide yes)
+			)
+		)
+	)
 	(global_label "D+"
 		(shape input)
@@
 	(global_label "OVDD"
 		(shape input)
-		(at 92.71 58.42 180)
-		(fields_autoplaced yes)
-		(effects
-			(font
-				(size 1.27 1.27)
-			)
-			(justify right)
-		)
-		(property "Intersheetrefs" "${INTERSHEET_REFS}"
-			(at 84.7657 58.42 0)
-			(effects
-				(font
-					(size 1.27 1.27)
-				)
-				(justify right)
-				(hide yes)
-			)
-		)
-	)
-	(global_label "OVDD"
-		(shape input)
 		(at 172.72 78.74 180)
 		(fields_autoplaced yes)
@@
 	)
 	(symbol
+		(lib_id "power:VDD")
+		(at 172.72 78.74 270)
+		(unit 1)
+		(exclude_from_sim no)
+		(in_bom yes)
+		(on_board yes)
+		(dnp no)
+		(fields_autoplaced yes)
+		(property "Reference" "#PWR028"
+			(at 168.91 78.74 0)
+			(effects
+				(font
+					(size 1.27 1.27)
+				)
+				(hide yes)
+			)
+		)
+		(property "Value" "VDD"
+			(at 176.53 78.7399 90)
+			(effects
+				(font
+					(size 1.27 1.27)
+				)
+				(justify left)
+			)
+		)
+		(property "Footprint" ""
+			(at 172.72 78.74 0)
+			(effects
+				(font
+					(size 1.27 1.27)
+				)
+				(hide yes)
+			)
+		)
+		(property "Datasheet" ""
+			(at 172.72 78.74 0)
+			(effects
+				(font
+					(size 1.27 1.27)
+				)
+				(hide yes)
+			)
+		)
+		(property "Description" ""
+			(at 172.72 78.74 0)
+			(effects
+				(font
+					(size 1.27 1.27)
+				)
+				(hide yes)
+			)
+		)
+		(pin "1"
+		)
+		(instances
+			(project "badapple006"
+				(path "/88f86251-37ea-456e-9a8e-c00115fc8776"
+					(reference "#PWR028")
+					(unit 1)
+				)
+			)
+		)
+	)
+	(symbol
 		(lib_id "power:GND")
 		(at 92.71 139.7 0)
@@
 		(dnp no)
 		(property "Reference" "C7"
-			(at 73.66 50.8 0)
+			(at 71.628 49.784 0)
 			(effects
 				(font
@@
 		)
 		(property "Value" "100n"
-			(at 73.66 53.34 0)
+			(at 68.58 46.736 0)
 			(effects
 				(font
@@
 	)
 	(symbol
+		(lib_id "Connector_Generic:Conn_01x01")
+		(at 251.46 53.34 0)
+		(unit 1)
+		(exclude_from_sim no)
+		(in_bom no)
+		(on_board yes)
+		(dnp yes)
+		(fields_autoplaced yes)
+		(property "Reference" "J10"
+			(at 254 52.07 0)
+			(effects
+				(font
+					(size 1.27 1.27)
+				)
+				(justify left)
+			)
+		)
+		(property "Value" "SCL"
+			(at 254 54.61 0)
+			(effects
+				(font
+					(size 1.27 1.27)
+				)
+				(justify left)
+			)
+		)
+		(property "Footprint" "TestPoint:TestPoint_Pad_D1.0mm"
+			(at 251.46 53.34 0)
+			(effects
+				(font
+					(size 1.27 1.27)
+				)
+				(hide yes)
+			)
+		)
+		(property "Datasheet" "~"
+			(at 251.46 53.34 0)
+			(effects
+				(font
+					(size 1.27 1.27)
+				)
+				(hide yes)
+			)
+		)
+		(property "Description" ""
+			(at 251.46 53.34 0)
+			(effects
+				(font
+					(size 1.27 1.27)
+				)
+				(hide yes)
+			)
+		)
+		(pin "1"
+		)
+		(instances
+			(project "badapple006"
+				(path "/88f86251-37ea-456e-9a8e-c00115fc8776"
+					(reference "J10")
+					(unit 1)
+				)
+			)
+		)
+	)
+	(symbol
+		(lib_id "Connector_Generic:Conn_01x01")
+		(at 251.46 59.69 0)
+		(unit 1)
+		(exclude_from_sim no)
+		(in_bom no)
+		(on_board yes)
+		(dnp yes)
+		(fields_autoplaced yes)
+		(property "Reference" "J11"
+			(at 254 58.42 0)
+			(effects
+				(font
+					(size 1.27 1.27)
+				)
+				(justify left)
+			)
+		)
+		(property "Value" "SDA"
+			(at 254 60.96 0)
+			(effects
+				(font
+					(size 1.27 1.27)
+				)
+				(justify left)
+			)
+		)
+		(property "Footprint" "TestPoint:TestPoint_Pad_D1.0mm"
+			(at 251.46 59.69 0)
+			(effects
+				(font
+					(size 1.27 1.27)
+				)
+				(hide yes)
+			)
+		)
+		(property "Datasheet" "~"
+			(at 251.46 59.69 0)
+			(effects
+				(font
+					(size 1.27 1.27)
+				)
+				(hide yes)
+			)
+		)
+		(property "Description" ""
+			(at 251.46 59.69 0)
+			(effects
+				(font
+					(size 1.27 1.27)
+				)
+				(hide yes)
+			)
+		)
+		(pin "1"
+		)
+		(instances
+			(project "badapple006"
+				(path "/88f86251-37ea-456e-9a8e-c00115fc8776"
+					(reference "J11")
+					(unit 1)
+				)
+			)
+		)
+	)
+	(symbol
 		(lib_id "Device:R")
 		(at 62.23 72.39 0)
@@
 		(dnp no)
 		(property "Reference" "C4"
-			(at 82.55 50.8 0)
+			(at 80.518 49.784 0)
 			(effects
 				(font
@@
 		)
 		(property "Value" "2.2u16v"
-			(at 82.55 53.34 0)
+			(at 76.2 46.736 0)
 			(effects
 				(font
@@
 					(unit 1)
 				)
-			)
-		)
-	)
-	(symbol
-		(lib_id "Connector_Generic:Conn_01x01")
-		(at 177.8 78.74 0)
-		(unit 1)
-		(exclude_from_sim no)
-		(in_bom no)
-		(on_board yes)
-		(dnp yes)
-		(fields_autoplaced yes)
-		(property "Reference" "J10"
-			(at 180.34 77.47 0)
-			(effects
-				(font
-					(size 1.27 1.27)
-				)
-				(justify left)
-			)
-		)
-		(property "Value" "OVDD"
-			(at 180.34 80.01 0)
-			(effects
-				(font
-					(size 1.27 1.27)
-				)
-				(justify left)
-			)
-		)
-		(property "Footprint" "TestPoint:TestPoint_Pad_D1.0mm"
-			(at 177.8 78.74 0)
-			(effects
-				(font
-					(size 1.27 1.27)
-				)
-				(hide yes)
-			)
-		)
-		(property "Datasheet" "~"
-			(at 177.8 78.74 0)
-			(effects
-				(font
-					(size 1.27 1.27)
-				)
-				(hide yes)
-			)
-		)
-		(property "Description" ""
-			(at 177.8 78.74 0)
-			(effects
-				(font
-					(size 1.27 1.27)
-				)
-				(hide yes)
-			)
-		)
-		(pin "1"
-		)
-		(instances
-			(project "badapple006"
-				(path "/88f86251-37ea-456e-9a8e-c00115fc8776"
-					(reference "J10")
-					(unit 1)
-				)

Commit message: Almost working
Other:
- note added: "1"
- note added: "2"
- note added: "3"
- note added: "4"
- note added: "5"
- note added: "6"
- note added: "7"
- note added: "8"
Changed lines of the file:
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@@
+		)
+	)
+	(text "3"
+		(exclude_from_sim no)
+		(at 210.82 39.116 0)
+		(effects
+			(font
+				(size 1.27 1.27)
+			)
+		)
+	)
+	(text "7"
+		(exclude_from_sim no)
+		(at 214.63 51.054 0)
+		(effects
+			(font
+				(size 1.27 1.27)
+			)
+		)
+	)
+	(text "5"
+		(exclude_from_sim no)
+		(at 210.82 44.958 0)
+		(effects
+			(font
+				(size 1.27 1.27)
+			)
 		)
 	)
@@
 		)
 	)
+	(text "8"
+		(exclude_from_sim no)
+		(at 219.456 54.102 0)
+		(effects
+			(font
+				(size 1.27 1.27)
+			)
+		)
+	)
+	(text "2"
+		(exclude_from_sim no)
+		(at 210.82 36.576 0)
+		(effects
+			(font
+				(size 1.27 1.27)
+			)
+		)
+	)
+	(text "6"
+		(exclude_from_sim no)
+		(at 214.376 48.514 0)
+		(effects
+			(font
+				(size 1.27 1.27)
+			)
+		)
+	)
+	(text "4"
+		(exclude_from_sim no)
+		(at 210.82 42.164 0)
+		(effects
+			(font
+				(size 1.27 1.27)
+			)
+		)
+	)
 	(text "OLED DISPLAY: RB6448TSWHG04 (Ronboe)"
 		(exclude_from_sim no)
-		(at 184.15 29.21 0)
+		(at 173.482 29.464 0)
 		(effects
 			(font
@@
 		)
 	)
+	(text "1"
+		(exclude_from_sim no)
+		(at 210.82 34.036 0)
+		(effects
+			(font
+				(size 1.27 1.27)
+			)
+		)
+	)

Commit message: Update flip design.
Parts:
- removed U2: XC6206P332, Package_TO_SOT_SMD:SOT-23, symbol Regulator_Linear:IFX27001TFV26
- added C11: 4.7u10v, Capacitor_SMD:C_0402_1005Metric, symbol Device:C
- added D3, D4: D, Diode_SMD:D_SOD-323, symbol Device:D_Schottky
- added U2: RS3236-3.3YUTDN4, cnhardware:xdfn-reg, symbol cnhardware:RS3236-DFN-LDO
- C1, C2, C4, C5, C6: value 2.2u16v -> 4.7u10v; footprint Capacitor_SMD:C_0603_1608Metric -> Capacitor_SMD:C_0402_1005Metric; LCSC C23630 -> C23733
- R5: value 30 -> 49.9; LCSC C1091 -> C25120; now in the parts list
Connections:
- net GND: now also U2.2 (GND), U2.5 (FLAG_GND)
- net RFO2: no longer U1.11 (PC4/T1C1_/T1/MCO/A2)
- net VBUS: now also D3.2 (A), U2.3 (EN), U2.4 (IN)
- net VDD: now also U2.1 (OUT)
- net OVCC: now reaches C2.1, C3.1, J1.1 (Pin_1)
- net OVCC: now also D4.1 (K)
- net CHARGEPUMP: now reaches U1.10 (PC3/T1/T2)
- net CHARGEPUMP: now also U1.11 (PC4/T1C1_/T1/MCO/A2), C11.2
- new net: C11.1, D3.1 (K), D4.2 (A)
