File: charlietest/hexagonal_test/hexagonal_test.kicad_pcb (KiCad board)
At the start: 2 copper layers, 30 parts

Commit message: Playing with other structures
Parts:
- added D31: LED, LED_SMD:LED_0603_1608Metric, F.Cu at (76.5, 63.7)
- added D32: LED, LED_SMD:LED_0603_1608Metric, F.Cu at (85.5, 66.3)
- added D33: LED, LED_SMD:LED_0603_1608Metric, F.Cu at (87.8, 67.6)
- added D34: LED, LED_SMD:LED_0603_1608Metric, F.Cu at (78.8, 67.6)
- added D35: LED, LED_SMD:LED_0603_1608Metric, F.Cu at (78.8, 59.8)
- added D36: LED, LED_SMD:LED_0603_1608Metric, F.Cu at (78.8, 62.4)
- added D37: LED, LED_SMD:LED_0603_1608Metric, F.Cu at (81.0, 66.3)
- added D38: LED, LED_SMD:LED_0603_1608Metric, F.Cu at (81.0, 61.1)
- added D39: LED, LED_SMD:LED_0603_1608Metric, F.Cu at (81.0, 63.7)
- added D40: LED, LED_SMD:LED_0603_1608Metric, F.Cu at (83.2, 65.0)
- added D41: LED, LED_SMD:LED_0603_1608Metric, F.Cu at (81.0, 58.5)
- added D42: LED, LED_SMD:LED_0603_1608Metric, F.Cu at (76.5, 58.5)
- added D43: LED, LED_SMD:LED_0603_1608Metric, F.Cu at (78.8, 65.0)
- added D44: LED, LED_SMD:LED_0603_1608Metric, F.Cu at (87.8, 65.0)
- added D45: LED, LED_SMD:LED_0603_1608Metric, F.Cu at (83.2, 67.6)
- added D46: LED, LED_SMD:LED_0603_1608Metric, F.Cu at (83.2, 59.8)
- added D47: LED, LED_SMD:LED_0603_1608Metric, F.Cu at (83.2, 62.4)
- added D48: LED, LED_SMD:LED_0603_1608Metric, F.Cu at (76.5, 66.3)
- added D49: LED, LED_SMD:LED_0603_1608Metric, F.Cu at (90.0, 66.3)
- added D50: LED, LED_SMD:LED_0603_1608Metric, F.Cu at (90.0, 63.7)
- added D51: LED, LED_SMD:LED_0603_1608Metric, F.Cu at (85.5, 58.5)
- added D52: LED, LED_SMD:LED_0603_1608Metric, F.Cu at (85.5, 61.1)
- added D53: LED, LED_SMD:LED_0603_1608Metric, F.Cu at (76.5, 61.1)
- added D54: LED, LED_SMD:LED_0603_1608Metric, F.Cu at (83.7, 72.8)
- added D55: LED, LED_SMD:LED_0603_1608Metric, F.Cu at (85.5, 63.7)
- added D56: LED, LED_SMD:LED_0603_1608Metric, F.Cu at (87.8, 59.8)
- added D57: LED, LED_SMD:LED_0603_1608Metric, F.Cu at (87.8, 62.4)
- added D58: LED, LED_SMD:LED_0603_1608Metric, F.Cu at (90.0, 61.1)
- added D59: LED, LED_SMD:LED_0603_1608Metric, F.Cu at (90.0, 58.5)
- added D60: LED, LED_SMD:LED_0603_1608Metric, F.Cu at (87.8, 72.8)
Routing:
- net C4: track 68.3 -> 24.3 mm, vias 8 -> 0
- net C5: track 61.5 -> 22.1 mm, vias 10 -> 0
- net C1: track 54.3 -> 18.0 mm, vias 2 -> 3
- net C3: track 53.1 -> 19.7 mm, vias 6 -> 0
- net C2: track 52.2 -> 23.8 mm, vias 4 -> 3
- net C0: track 43.2 -> 25.9 mm, vias 0 -> 6
Other:
- board text added: "size = 2 3/2*size, size -> 3*.75 sqrt(3)*size -> 1.73205*.75"

Commit message: bump
Parts:
- added D61: LED, LED_SMD:LED_0603_1608Metric, F.Cu at (92.7, 71.1)
- added D62: LED, LED_SMD:LED_0603_1608Metric, F.Cu at (92.7, 73.7)
- added D63: LED, LED_SMD:LED_0603_1608Metric, F.Cu at (92.7, 76.2)
- added D64: LED, LED_SMD:LED_0603_1608Metric, F.Cu at (92.7, 78.8)
- added D65: LED, LED_SMD:LED_0603_1608Metric, F.Cu at (96.7, 71.1)
- added D66: LED, LED_SMD:LED_0603_1608Metric, F.Cu at (96.7, 73.7)
- added D67: LED, LED_SMD:LED_0603_1608Metric, F.Cu at (96.7, 76.2)
- added D68: LED, LED_SMD:LED_0603_1608Metric, F.Cu at (96.7, 78.8)
- added D69: LED, LED_SMD:LED_0603_1608Metric, F.Cu at (100.8, 71.1)
- added D70: LED, LED_SMD:LED_0603_1608Metric, F.Cu at (100.8, 73.7)
- added D71: LED, LED_SMD:LED_0603_1608Metric, F.Cu at (100.8, 76.2)
- added D72: LED, LED_SMD:LED_0603_1608Metric, F.Cu at (100.8, 78.8)
- added D73: LED, LED_SMD:LED_0603_1608Metric, F.Cu at (120.0, 79.7)
- added D74: LED, LED_SMD:LED_0603_1608Metric, F.Cu at (123.8, 80.6)
- added D75: LED, LED_SMD:LED_0603_1608Metric, F.Cu at (124.0, 87.6)
- added D76: LED, LED_SMD:LED_0603_1608Metric, F.Cu at (124.0, 90.2)
- added D77: LED, LED_SMD:LED_0603_1608Metric, F.Cu at (128.1, 82.4)
- added D78: LED, LED_SMD:LED_0603_1608Metric, F.Cu at (128.1, 85.0)
- added D79: LED, LED_SMD:LED_0603_1608Metric, F.Cu at (128.1, 87.6)
- added D80: LED, LED_SMD:LED_0603_1608Metric, F.Cu at (128.1, 90.2)
- added D81: LED, LED_SMD:LED_0603_1608Metric, F.Cu at (132.1, 82.4)
- added D82: LED, LED_SMD:LED_0603_1608Metric, F.Cu at (132.1, 85.0)
- added D83: LED, LED_SMD:LED_0603_1608Metric, F.Cu at (132.1, 87.6)
- added D84: LED, LED_SMD:LED_0603_1608Metric, F.Cu at (132.1, 90.2)
Connections:
- D11 pad 1: C5 -> C6
- D12 pad 1: C5 -> C6
- D15 pad 1: C5 -> C6
- D16 pad 1: C5 -> C6
- D17 pad 1: C3 -> C5
- D18 pad 1: C3 -> C5
- D21 pad 1: C5 -> C6
- D22 pad 1: C5 -> C6
- D23 pad 1: C3 -> C5
- D24 pad 1: C3 -> C5
- D25 pad 1: C1 -> C3
- D26 pad 1: C1 -> C3
- D27 pad 1: C5 -> C6
- D28 pad 1: C5 -> C6
- D29 pad 1: C3 -> C5
- D30 pad 1: C3 -> C5
- D37 pad 1: D5 -> D6
- D40 pad 1: D5 -> D6
- D42 pad 1: D5 -> D6
- D44 pad 1: D5 -> D6
- D46 pad 1: D5 -> D6
- D47 pad 1: D3 -> D5
- D49 pad 1: D5 -> D6
- D5 pad 1: C5 -> C6
- D50 pad 1: D3 -> D5
- D51 pad 1: D5 -> D6
- D52 pad 1: D3 -> D5
- D53 pad 1: D5 -> D6
- D54 pad 1: D3 -> D5
- D55 pad 1: D1 -> D3
- D56 pad 1: D5 -> D6
- D57 pad 1: D3 -> D5
- D58 pad 1: D1 -> D3
- D59 pad 1: D5 -> D6
- D6 pad 1: C5 -> C6
- D60 pad 1: D3 -> D5
Routing:
- net C6: track 0.00 -> 18.3 mm
- net C5: track 22.1 -> 9.17 mm
- net C3: track 19.7 -> 6.87 mm
- net C4: track 24.3 -> 28.1 mm

Commit message: Poking around
Parts:
- added D1: LED, LED_SMD:LED_0603_1608Metric, F.Cu at (151.5, 81.4)
- added D10: LED, LED_SMD:LED_0603_1608Metric, F.Cu at (159.0, 83.1)
- added D11: LED, LED_SMD:LED_0603_1608Metric, F.Cu at (162.0, 83.1)
- added D12: LED, LED_SMD:LED_0603_1608Metric, F.Cu at (165.0, 83.1)
- added D13: LED, LED_SMD:LED_0603_1608Metric, F.Cu at (151.5, 84.9)
- added D14: LED, LED_SMD:LED_0603_1608Metric, F.Cu at (154.5, 84.9)
- added D15: LED, LED_SMD:LED_0603_1608Metric, F.Cu at (157.5, 84.9)
- added D16: LED, LED_SMD:LED_0603_1608Metric, F.Cu at (160.5, 84.9)
- added D17: LED, LED_SMD:LED_0603_1608Metric, F.Cu at (163.5, 84.9)
- added D18: LED, LED_SMD:LED_0603_1608Metric, F.Cu at (166.5, 84.9)
- added D19: LED, LED_SMD:LED_0603_1608Metric, F.Cu at (150.0, 86.6)
- added D2: LED, LED_SMD:LED_0603_1608Metric, F.Cu at (154.5, 81.4)
- added D20: LED, LED_SMD:LED_0603_1608Metric, F.Cu at (153.0, 86.6)
- added D21: LED, LED_SMD:LED_0603_1608Metric, F.Cu at (156.0, 86.6)
- added D22: LED, LED_SMD:LED_0603_1608Metric, F.Cu at (159.0, 86.6)
- added D23: LED, LED_SMD:LED_0603_1608Metric, F.Cu at (162.0, 86.6)
- added D24: LED, LED_SMD:LED_0603_1608Metric, F.Cu at (165.0, 86.6)
- added D25: LED, LED_SMD:LED_0603_1608Metric, F.Cu at (163.5, 88.3)
- added D26: LED, LED_SMD:LED_0603_1608Metric, F.Cu at (166.5, 88.3)
- added D27: LED, LED_SMD:LED_0603_1608Metric, F.Cu at (151.5, 88.3)
- added D28: LED, LED_SMD:LED_0603_1608Metric, F.Cu at (154.5, 88.3)
- added D29: LED, LED_SMD:LED_0603_1608Metric, F.Cu at (157.5, 88.3)
- added D3: LED, LED_SMD:LED_0603_1608Metric, F.Cu at (157.5, 81.4)
- added D30: LED, LED_SMD:LED_0603_1608Metric, F.Cu at (160.5, 88.3)
- added D4: LED, LED_SMD:LED_0603_1608Metric, F.Cu at (160.5, 81.4)
- added D5: LED, LED_SMD:LED_0603_1608Metric, F.Cu at (163.5, 81.4)
- added D6: LED, LED_SMD:LED_0603_1608Metric, F.Cu at (166.5, 81.4)
- added D7: LED, LED_SMD:LED_0603_1608Metric, F.Cu at (150.0, 83.1)
- added D73: LED, LED_SMD:LED_0603_1608Metric, F.Cu at (150.0, 90.1)
- added D74: LED, LED_SMD:LED_0603_1608Metric, F.Cu at (153.0, 90.1)
- added D75: LED, LED_SMD:LED_0603_1608Metric, F.Cu at (156.0, 90.1)
- added D76: LED, LED_SMD:LED_0603_1608Metric, F.Cu at (159.0, 90.1)
- added D77: LED, LED_SMD:LED_0603_1608Metric, F.Cu at (162.0, 90.1)
- added D78: LED, LED_SMD:LED_0603_1608Metric, F.Cu at (165.0, 90.1)
- added D79: LED, LED_SMD:LED_0603_1608Metric, F.Cu at (168.0, 90.1)
- added D8: LED, LED_SMD:LED_0603_1608Metric, F.Cu at (153.0, 83.1)
- added D80: LED, LED_SMD:LED_0603_1608Metric, F.Cu at (171.0, 90.1)
- added D81: LED, LED_SMD:LED_0603_1608Metric, F.Cu at (168.0, 86.6)
- added D82: LED, LED_SMD:LED_0603_1608Metric, F.Cu at (171.0, 86.6)
- added D83: LED, LED_SMD:LED_0603_1608Metric, F.Cu at (168.0, 83.1)
- added D84: LED, LED_SMD:LED_0603_1608Metric, F.Cu at (171.0, 83.1)
- added D85: LED, LED_SMD:LED_0603_1608Metric, F.Cu at (121.5, 81.4)
- added D85: LED, LED_SMD:LED_0603_1608Metric, F.Cu at (151.5, 91.8)
- added D86: LED, LED_SMD:LED_0603_1608Metric, F.Cu at (154.5, 91.8)
- added D86: LED, LED_SMD:LED_0603_1608Metric, F.Cu at (124.5, 81.4)
- added D87: LED, LED_SMD:LED_0603_1608Metric, F.Cu at (157.5, 91.8)
- added D87: LED, LED_SMD:LED_0603_1608Metric, F.Cu at (127.5, 81.4)
- added D88: LED, LED_SMD:LED_0603_1608Metric, F.Cu at (160.5, 91.8)
- added D88: LED, LED_SMD:LED_0603_1608Metric, F.Cu at (130.5, 81.4)
- added D89: LED, LED_SMD:LED_0603_1608Metric, F.Cu at (163.5, 91.8)
- added D89: LED, LED_SMD:LED_0603_1608Metric, F.Cu at (133.5, 81.4)
- added D9: LED, LED_SMD:LED_0603_1608Metric, F.Cu at (156.0, 83.1)
- added D90: LED, LED_SMD:LED_0603_1608Metric, F.Cu at (136.5, 81.4)
- added D90: LED, LED_SMD:LED_0603_1608Metric, F.Cu at (166.5, 91.8)
- added D91: LED, LED_SMD:LED_0603_1608Metric, F.Cu at (139.5, 81.4)
- added D91: LED, LED_SMD:LED_0603_1608Metric, F.Cu at (169.5, 91.8)
- added D92: LED, LED_SMD:LED_0603_1608Metric, F.Cu at (142.5, 81.4)
- added D92: LED, LED_SMD:LED_0603_1608Metric, F.Cu at (172.5, 91.8)
- added D93: LED, LED_SMD:LED_0603_1608Metric, F.Cu at (169.5, 88.3)
- added D93: LED, LED_SMD:LED_0603_1608Metric, F.Cu at (139.5, 77.9)
- added D94: LED, LED_SMD:LED_0603_1608Metric, F.Cu at (172.5, 88.4)
- added D94: LED, LED_SMD:LED_0603_1608Metric, F.Cu at (142.5, 78.0)
- added D95: LED, LED_SMD:LED_0603_1608Metric, F.Cu at (169.5, 84.9)
- added D95: LED, LED_SMD:LED_0603_1608Metric, F.Cu at (139.5, 74.5)
- added D96: LED, LED_SMD:LED_0603_1608Metric, F.Cu at (172.5, 84.9)
- added D96: LED, LED_SMD:LED_0603_1608Metric, F.Cu at (142.5, 74.5)
- added D97: LED, LED_SMD:LED_0603_1608Metric, F.Cu at (169.5, 81.4)
- added D97: LED, LED_SMD:LED_0603_1608Metric, F.Cu at (139.5, 71.0)
- added D98: LED, LED_SMD:LED_0603_1608Metric, F.Cu at (172.5, 81.4)
- added D98: LED, LED_SMD:LED_0603_1608Metric, F.Cu at (142.5, 71.0)
- moved D84 19.6 mm to (141.0, 72.7), turned to 180 degrees
- moved D80 16.7 mm to (141.0, 79.7), turned to 180 degrees
- moved D83 16.0 mm to (138.0, 72.7), turned to 180 degrees
- moved D79 12.7 mm to (138.0, 79.7), turned to 180 degrees
- moved D82 12.5 mm to (141.0, 76.2), turned to 180 degrees
- moved D76 11.7 mm to (129.0, 79.7), turned to 180 degrees
- moved D78 8.77 mm to (135.0, 79.7), turned to 180 degrees
- moved D81 8.57 mm to (138.0, 76.2), turned to 180 degrees
- moved D75 8.19 mm to (126.0, 79.7), turned to 180 degrees
- moved D77 4.81 mm to (132.0, 79.7), turned to 180 degrees
- moved D74 1.18 mm to (123.0, 79.7), turned to 180 degrees
- moved D73 0.06 mm to (120.0, 79.7), turned to 180 degrees
Connections:
- D17 pad 1: C5 -> C7
- D18 pad 1: C5 -> C7
- D23 pad 1: C5 -> C7
- D24 pad 1: C5 -> C7
- D25 pad 1: C3 -> C5
- D26 pad 1: C3 -> C5
- D29 pad 1: C5 -> C7
- D30 pad 1: C5 -> C7
- D75 pad 1: C5 -> C7
- D76 pad 1: C5 -> C7
- D77 pad 1: C3 -> C5
- D78 pad 1: C3 -> C5
- D79 pad 1: C1 -> C3
- D80 pad 1: C1 -> C3
- D81 pad 1: C3 -> C5
- D82 pad 1: C3 -> C5
- D83 pad 1: C5 -> C7
- D84 pad 1: C5 -> C7
Routing:
- net C7: track 0.00 -> 61.8 mm
- net C3: track 6.87 -> 53.9 mm, vias 0 -> 5
- net C6: track 18.3 -> 64.4 mm
- net C5: track 9.17 -> 53.9 mm
- net C2: track 23.8 -> 67.8 mm, vias 3 -> 10
- net C4: track 28.1 -> 70.5 mm, vias 0 -> 5
- net C0: track 25.9 -> 67.0 mm, vias 6 -> 15
- net C1: track 18.0 -> 52.9 mm, vias 3 -> 10
