File: charlietest/hexagonal_test/hexagonal_test.kicad_sch (KiCad schematic)
At the start: 30 parts

Commit message: Playing with other structures
Parts:
- added D31, D32, D33, D34, D35, D36, D37, D38, D39, D40, D41, D42, D43, D44, D45, D46, D47, D48, D49, D50, D51, D52, D53, D54, D55, D56, D57, D58, D59, D60: LED, LED_SMD:LED_0603_1608Metric, symbol Device:LED
Connections:
- new net D0: D35.2 (A), D38.2 (A), D41.2 (A), D43.2 (A), D46.2 (A), D49.2 (A), D52.2 (A), D54.2 (A), D55.2 (A), D58.2 (A)
- new net D1: D31.2 (A), D33.2 (A), D36.2 (A), D39.2 (A), D42.2 (A), D44.2 (A), D47.2 (A), D50.2 (A), D55.1 (K), D58.1 (K)
- new net D2: D31.1 (K), D33.1 (K), D35.1 (K), D38.1 (K), D45.2 (A), D48.2 (A), D51.2 (A), D53.2 (A), D57.2 (A), D60.2 (A)
- new net D3: D32.2 (A), D34.2 (A), D37.2 (A), D40.2 (A), D47.1 (K), D50.1 (K), D52.1 (K), D54.1 (K), D57.1 (K), D60.1 (K)
- new net D4: D32.1 (K), D34.1 (K), D36.1 (K), D39.1 (K), D41.1 (K), D43.1 (K), D45.1 (K), D48.1 (K), D56.2 (A), D59.2 (A)
- new net D5: D37.1 (K), D40.1 (K), D42.1 (K), D44.1 (K), D46.1 (K), D49.1 (K), D51.1 (K), D53.1 (K), D56.1 (K), D59.1 (K)

Commit message: bump
Parts:
- added D61, D62, D63, D64, D65, D66, D67, D68, D69, D70, D71, D72, D73, D74, D75, D76, D77, D78, D79, D80, D81, D82, D83, D84: LED, LED_SMD:LED_0603_1608Metric, symbol Device:LED
Connections:
- net C0: now also D79.2 (A), D80.2 (A)
- net C1: now also D77.2 (A), D78.2 (A), D79.1 (K), D80.1 (K); no longer D25.1 (K), D26.1 (K)
- net C2: now also D81.2 (A), D82.2 (A)
- net C3: now also D25.1 (K), D26.1 (K), D75.2 (A), D76.2 (A), D77.1 (K), D78.1 (K), D81.1 (K), D82.1 (K); no longer D17.1 (K), D18.1 (K), D23.1 (K), D24.1 (K), D29.1 (K), D30.1 (K)
- net C4: now also D83.2 (A), D84.2 (A)
- net C5: now also D17.1 (K), D18.1 (K), D23.1 (K), D24.1 (K), D29.1 (K), D30.1 (K), D73.2 (A), D74.2 (A), D75.1 (K), D76.1 (K), D83.1 (K), D84.1 (K); no longer D11.1 (K), D12.1 (K), D15.1 (K), D16.1 (K), D21.1 (K), D22.1 (K), D27.1 (K), D28.1 (K), D5.1 (K), D6.1 (K)
- net D0: now also D61.2 (A), D62.2 (A)
- net D1: now also D61.1 (K), D62.1 (K), D67.2 (A), D68.2 (A); no longer D55.1 (K), D58.1 (K)
- net D2: now also D63.2 (A), D64.2 (A)
- net D3: now also D55.1 (K), D58.1 (K), D63.1 (K), D64.1 (K), D67.1 (K), D68.1 (K), D69.2 (A), D70.2 (A); no longer D47.1 (K), D50.1 (K), D52.1 (K), D54.1 (K), D57.1 (K), D60.1 (K)
- net D4: now also D65.2 (A), D66.2 (A)
- net D5: now also D47.1 (K), D50.1 (K), D52.1 (K), D54.1 (K), D57.1 (K), D60.1 (K), D65.1 (K), D66.1 (K), D69.1 (K), D70.1 (K), D71.2 (A), D72.2 (A); no longer D37.1 (K), D40.1 (K), D42.1 (K), D44.1 (K), D46.1 (K), D49.1 (K), D51.1 (K), D53.1 (K), D56.1 (K), D59.1 (K)
- new net C6: D11.1 (K), D12.1 (K), D15.1 (K), D16.1 (K), D21.1 (K), D22.1 (K), D27.1 (K), D28.1 (K), D5.1 (K), D6.1 (K), D73.1 (K), D74.1 (K)
- new net D6: D37.1 (K), D40.1 (K), D42.1 (K), D44.1 (K), D46.1 (K), D49.1 (K), D51.1 (K), D53.1 (K), D56.1 (K), D59.1 (K), D71.1 (K), D72.1 (K)
Other:
- moved on the sheet: D1, D10, D11, D12, D13, D14, D15, D16, D17, D18, D19, D2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

Commit message: Poking around
Parts:
- added D85, D86, D87, D88, D89, D90, D91, D92, D93, D94, D95, D96, D97, D98: LED, LED_SMD:LED_0603_1608Metric, symbol Device:LED
Connections:
- net C0: now also D91.2 (A), D92.2 (A)
- net C1: now also D89.2 (A), D90.2 (A), D91.1 (K), D92.1 (K); no longer D79.1 (K), D80.1 (K)
- net C2: now also D93.2 (A), D94.2 (A)
- net C3: now also D79.1 (K), D80.1 (K), D87.2 (A), D88.2 (A), D89.1 (K), D90.1 (K), D93.1 (K), D94.1 (K); no longer D25.1 (K), D26.1 (K), D77.1 (K), D78.1 (K), D81.1 (K), D82.1 (K)
- net C4: now also D95.2 (A), D96.2 (A)
- net C5: now also D25.1 (K), D26.1 (K), D77.1 (K), D78.1 (K), D81.1 (K), D82.1 (K), D85.2 (A), D86.2 (A), D87.1 (K), D88.1 (K), D95.1 (K), D96.1 (K); no longer D17.1 (K), D18.1 (K), D23.1 (K), D24.1 (K), D29.1 (K), D30.1 (K), D75.1 (K), D76.1 (K), D83.1 (K), D84.1 (K)
- net C6: now also D97.2 (A), D98.2 (A)
- new net C7: D17.1 (K), D18.1 (K), D23.1 (K), D24.1 (K), D29.1 (K), D30.1 (K), D75.1 (K), D76.1 (K), D83.1 (K), D84.1 (K), D85.1 (K), D86.1 (K), D97.1 (K), D98.1 (K)
Other:
- moved on the sheet: D25, D26, D77, D78, D79, D80, D81, D82
