File: ch570/ch570-with-tia-mon/ch570-with-tia-mon.kicad_pcb (KiCad board)
At the start: 2 copper layers, 8 x 72.1 mm, 33 parts, among them J2 USB_C_Receptacle_USB2.0_16P, J3 BAT/MX1.25, SW1 TS-1187A-B-A-B, SW2 TS-1187A-B-A-B, SW3 TS-1187A-B-A-B, U1 CH570Q, U2 AW32001, U4 MG6229D4-28, Y1 32MHz

Commit message: Poke design
Parts:
- moved U4 0.46 mm to (83.2, 75.4)
Connections:
- D2 pad 2: Net-(D2-A) -> VMON
- SW3 pad 1: Net-(D2-A) -> Net-(SW3-A)
- U3 pad 9: Net-(D2-A) -> Net-(SW3-A)
Routing:
- net Net-(D2-A): track 40.2 -> 0.00 mm, vias 2 -> 0
- net Net-(SW3-A): track 0.00 -> 22.3 mm, vias 0 -> 2
- net GND: track 240.1 -> 242.7 mm, vias 31 -> 33
- net VMON: track 43.0 -> 45.0 mm
- net Net-(U2-SYS): track 43.8 -> 42.8 mm
- net VDD: track 25.4 -> 26.0 mm
- net SCL: track 44.0 -> 44.7 mm
- net SDA: track 44.4 -> 45.0 mm

Commit message: Bump all designs per order
Parts:
- moved U4 0.13 mm to (83.2, 75.5)
Routing:
- net GND: track 242.7 -> 255.1 mm, vias 33 -> 44
- net Net-(SW3-A): track 22.3 -> 21.3 mm
- net SDA: track 45.0 -> 44.3 mm
- net SCL: track 44.7 -> 44.1 mm
- net VDD: track 26.0 -> 26.3 mm, vias 6 -> 5
- net (no net): vias 0 -> 7
Other:
- board size 8 x 72.1 mm -> 10 x 72.1 mm

Commit message: Bump design by order
Parts:
- added C9: 0.1u, Capacitor_SMD:C_0402_1005Metric, F.Cu at (84.5, 59.6)
- moved C7 0.85 mm to (83.1, 61.3), turned to 180 degrees
- moved R11 0.18 mm to (85.4, 59.7)
- moved R12 0.14 mm to (86.6, 59.7)
Routing:
- net GND: track 255.1 -> 257.4 mm
- net Net-(U3-PD7/RST/T2C4/OPP1/PA4/OPN2): track 3.31 -> 4.25 mm
- net Net-(D1-K): track 18.5 -> 19.0 mm

Commit message: Bump designs per purchase
Other:
- board text added: "NOTE: MUST USE 0.8mm THICK PCB"
Changed lines of the file:
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@@
+		)
+	)
+	(gr_text "NOTE:\n\nMUST USE 0.8mm THICK PCB"
+		(at 100 81 0)
+		(layer "F.Fab")
+		(effects
+			(font
+				(size 1 1)
+				(thickness 0.15)
+			)
+			(justify left bottom)
 		)
 	)
