File: ch32v006/ch32v006fun/ch32v006fun.kicad_pcb (KiCad board)
At the start: 2 copper layers, 40.6 x 44.5 mm, 25 parts, among them J2 PGM, J4 USB_C_Receptacle_USB2.0, J5 HOLE, J6 HOLE, SW1 BOOT, U1 CH32V006F8U6, U3 XC6206P332, Y2 24MHz

Commit message: Update with revA for 006 board
Routing:
- net GND: track 73.1 -> 76.0 mm, vias 89 -> 96
- net +5V: track 74.6 -> 73.6 mm, vias 2 -> 0
- net PC6: track 15.8 -> 15.2 mm, vias 2 -> 1
Other:
- board text added: "rev A"
