File: ch32v006/ch32v006fun/ch32v006fun.kicad_sch (KiCad schematic)
At the start: 25 parts, among them J2 PGM, J4 USB_C_Receptacle_USB2.0, J5 HOLE, J6 HOLE, SW1 BOOT, U1 CH32V006F8U6, U3 XC6206P332, Y2 24MHz

Commit message: Update with revA for 006 board
Parts:
- C1, C4, C5: LCSC C237173 -> C52923
- R3, R4: LCSC C258132 -> C25905
Changed lines of the file:
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@@
 			)
 		)
-		(property "LCSC" "C237173"
+		(property "LCSC" "C52923"
 			(at 129.54 54.61 0)
 			(effects
@@
 			)
 		)
-		(property "LCSC" "C258132"
+		(property "LCSC" "C25905"
 			(at 62.23 36.83 90)
 			(effects
@@
 			)
 		)
-		(property "LCSC" "C237173"
+		(property "LCSC" "C52923"
 			(at 99.06 54.61 0)
 			(effects
@@
 			)
 		)
-		(property "LCSC" "C237173"
+		(property "LCSC" "C52923"
 			(at 87.63 54.61 0)
 			(effects
@@
 			)
 		)
-		(property "LCSC" "C258132"
+		(property "LCSC" "C25905"
 			(at 55.88 39.37 90)
 			(effects
