File: addlepatedarray/synthtest/synthtest.kicad_pcb (KiCad board)
At the start: 2 copper layers, 60 parts, among them J1 RF0A+, J2 RF0A-, J3 RF0B-, J4 RF0B+, J5 RF1A-, J6 RF1B-, J7 RF1A+, J8 RF1B+, J9 REF, U1 ADF4351, U2 ADF4351, U4 CH32V003FxUx, U6 LDL1117-33, Y1 TG-5006CG-12H 26.0000M3

Commit message: Bump design
Parts:
- J1, J2, J3, J4, J5, J6, J7, J8, J9: footprint Connector_Coaxial:SMA_Molex_73251-1153_EdgeMount_Horizontal -> Connector_Coaxial:SMA_Amphenol_901-144_Vertical; moved to B.Cu
- R10, R7, R8, R9: footprint Resistor_SMD:R_0603_1608Metric -> Resistor_SMD:R_0402_1005Metric
- moved L3 141.2 mm to (202.8, 38.1), turned to 90 degrees
- moved L4 140.7 mm to (201.2, 37.5)
- moved L2 139.7 mm to (202.8, 40.8), turned to 90 degrees
- moved C2 126.8 mm to (197.2, 36.2)
- moved C21 126.5 mm to (194.5, 30.0), turned to 180 degrees
- moved C1 126.4 mm to (197.2, 35.2)
- moved C4 125.3 mm to (193.6, 35.8), turned to 90 degrees
- moved C20 124.9 mm to (202.5, 48.0), turned to -90 degrees
- moved C14 124.8 mm to (197.4, 44.8)
- moved C22 124.6 mm to (202.5, 32.0), turned to 90 degrees
- moved C13 124.4 mm to (197.4, 43.8)
- moved C6 124.3 mm to (190.6, 35.8), turned to 90 degrees
- moved C5 124.3 mm to (191.6, 35.8), turned to 90 degrees
- moved C3 123.5 mm to (192.6, 35.8), turned to 90 degrees
- moved L8 123.5 mm to (180.2, 40.8), turned to 90 degrees
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Routing:
- net GND: track 0.00 -> 149.2 mm, vias 0 -> 2
- net Net-(U2-RF_OUT_A-): track 0.00 -> 14.1 mm
- net Net-(U1-RF_OUT_A-): track 0.00 -> 14.1 mm
- net Net-(U2-RF_OUT_B-): track 0.00 -> 14.1 mm
- net Net-(U1-RF_OUT_B-): track 0.00 -> 14.1 mm
- net Net-(U1-RF_OUT_B+): track 0.00 -> 14.0 mm
- net Net-(U2-RF_OUT_B+): track 0.00 -> 14.0 mm
- net Net-(U1-RF_OUT_A+): track 0.00 -> 14.0 mm
- net Net-(U2-RF_OUT_A+): track 0.00 -> 14.0 mm
- net VVCO0: track 0.00 -> 11.1 mm, vias 0 -> 3
- net Net-(U2-VTUNE): track 0.00 -> 10.9 mm, vias 0 -> 2
- net Net-(U1-VTUNE): track 0.00 -> 10.2 mm, vias 0 -> 2
- net Net-(U1-VREF): track 0.00 -> 3.92 mm
- net Net-(U2-CPout): track 0.00 -> 3.25 mm
- net Net-(U1-CPout): track 0.00 -> 3.25 mm
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Other:
- board outline added: 65 x 30 mm

Commit message: Bump
Parts:
- added C27: 1n, Capacitor_SMD:C_0402_1005Metric, F.Cu at (199.1, 41.4)
- added C28: 1n, Capacitor_SMD:C_0402_1005Metric, F.Cu at (202.2, 42.3)
- added C29: 1u, Capacitor_SMD:C_0402_1005Metric, F.Cu at (199.2, 37.0)
- added C30: 1n, Capacitor_SMD:C_0402_1005Metric, F.Cu at (176.6, 41.3)
- added C31: 1n, Capacitor_SMD:C_0402_1005Metric, F.Cu at (191.4, 39.3)
- added C32: 1n, Capacitor_SMD:C_0402_1005Metric, F.Cu at (179.8, 42.4)
- added C33: 1n, Capacitor_SMD:C_0402_1005Metric, F.Cu at (192.0, 41.9)
- added C34: 1u, Capacitor_SMD:C_0402_1005Metric, F.Cu at (176.7, 37.4)
- added C35: 1n, Capacitor_SMD:C_0402_1005Metric, F.Cu at (168.8, 39.2)
- added C36: 1n, Capacitor_SMD:C_0402_1005Metric, F.Cu at (169.2, 42.0)
- added L10: 3.9nH, Inductor_SMD:L_0402_1005Metric, F.Cu at (179.8, 43.5)
- added L9: 3.9nH, Inductor_SMD:L_0402_1005Metric, F.Cu at (202.2, 43.6)
- moved R8 1.23 mm to (196.4, 45.6)
- moved R10 1.22 mm to (173.9, 45.6)
- moved R4 0.28 mm to (191.3, 37.7)
- moved C17 0.08 mm to (174.9, 44.7)
- moved C14 0.08 mm to (197.4, 44.7)
Routing:
- net GND: track 149.2 -> 235.9 mm, vias 2 -> 11
- net +3.3V: track 0.00 -> 37.7 mm, vias 0 -> 8
- net REFCLK: track 1.96 -> 21.8 mm
- net VVCO1: track 0.00 -> 14.0 mm, vias 0 -> 3
- net MUXOUT1: track 0.00 -> 6.67 mm
- net MUXOUT0: track 0.00 -> 5.37 mm
- net CE1: track 0.00 -> 4.01 mm
- net Net-(U2-VREF): track 0.00 -> 3.75 mm
- net LE1: track 0.00 -> 3.38 mm
- net VVCO0: track 11.1 -> 14.2 mm
- net MOSI: track 0.00 -> 2.50 mm
- net Net-(D1-K): track 0.00 -> 1.86 mm
- net SCK: track 0.00 -> 1.78 mm
- net Net-(U2-VCOM): track 0.83 -> 2.52 mm
- net Net-(J5-In): track 0.00 -> 1.52 mm
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
Commit message: Bump disign!
Parts:
- removed D3: LEDPWR, LED_SMD:LED_0603_1608Metric
- removed U6: LDL1117-33, Package_TO_SOT_SMD:SOT-223-3_TabPin2
- added C37: 1n, Capacitor_SMD:C_0402_1005Metric, F.Cu at (189.1, 38.8)
- added C38: 1n, Capacitor_SMD:C_0402_1005Metric, F.Cu at (191.7, 40.4)
- added C39: 1n, Capacitor_SMD:C_0402_1005Metric, F.Cu at (168.5, 40.4)
- added C40: 1n, Capacitor_SMD:C_0402_1005Metric, F.Cu at (171.2, 40.4)
- added C41: 1u, Capacitor_SMD:C_0402_1005Metric, F.Cu at (149.4, 50.3)
- added C42: 4.7u, Capacitor_SMD:C_0603_1608Metric, F.Cu at (152.2, 40.4)
- added C43: 1u, Capacitor_SMD:C_0402_1005Metric, F.Cu at (159.8, 44.8)
- added C44: 1u, Capacitor_SMD:C_0402_1005Metric, F.Cu at (156.4, 48.1)
- added C45: 4.7u, Capacitor_SMD:C_0603_1608Metric, F.Cu at (159.9, 36.4)
- added C46: 4.7u, Capacitor_SMD:C_0603_1608Metric, F.Cu at (165.2, 38.9)
- added C47: 4.7u, Capacitor_SMD:C_0603_1608Metric, F.Cu at (163.8, 41.9)
- added C48: 1u, Capacitor_SMD:C_0402_1005Metric, F.Cu at (151.6, 47.3)
- added J10: RJ45_Hanrun_HR911105A_Horizontal, cnhardware:HR915310A-RJ45-INTEGRATED-10MBIT, B.Cu at (156.6, 45.3)
- added J11: USB_C_Receptacle_USB2.0_14P, Connector_USB:USB_C_Receptacle_G-Switch_GT-USB-7051x, B.Cu at (150.5, 31.4)
- added J12: VCC, TestPoint:TestPoint_Pad_D1.0mm, F.Cu at (150.4, 38.6)
- added J13: SWC, TestPoint:TestPoint_Pad_D1.0mm, F.Cu at (146.3, 38.6)
- added J14: SWD, TestPoint:TestPoint_Pad_D1.0mm, F.Cu at (146.3, 35.8)
- added J15: GND, TestPoint:TestPoint_Pad_D1.0mm, F.Cu at (150.4, 35.8)
- added L11: 3.9nH, Inductor_SMD:L_0402_1005Metric, F.Cu at (150.9, 51.0)
- added R11: 100, Resistor_SMD:R_0402_1005Metric, F.Cu at (169.9, 40.9)
- added R12: 1.5k, cnhardware:R_0402_1005Metric_COMPACT, F.Cu at (162.5, 40.5)
- added R13: 5.1k, Resistor_SMD:R_0402_1005Metric, F.Cu at (146.5, 32.7)
- added R14: 5.1k, Resistor_SMD:R_0402_1005Metric, F.Cu at (152.3, 27.9)
- added R15: 33, Resistor_SMD:R_0402_1005Metric, F.Cu at (148.9, 35.5)
- added R16: 33, Resistor_SMD:R_0402_1005Metric, F.Cu at (147.9, 35.5)
- added R3: 100, Resistor_SMD:R_0402_1005Metric, F.Cu at (189.9, 40.5)
- added U3: CH32V208GBU6, Package_DFN_QFN:QFN-28-1EP_4x4mm_P0.45mm_EP2.6x2.6mm, F.Cu at (154.8, 45.0)
- added U5: WL2808E, Package_TO_SOT_SMD:SOT-23-5, F.Cu at (163.2, 44.7)
- added Y3: 32MHz, Crystal:Crystal_SMD_2016-4Pin_2.0x1.6mm, F.Cu at (159.6, 46.8)
- U4: value CH32V003FxUx -> WL2808E; footprint Package_DFN_QFN:QFN-20-1EP_3x3mm_P0.4mm_EP1.65x1.65mm -> Package_TO_SOT_SMD:SOT-23-5
- moved R6 14.4 mm to (162.6, 49.1)
- moved U4 10.2 mm to (163.0, 36.2), turned to 0 degrees
- moved J9 4.59 mm to (163.0, 30.0)
- moved Y1 4.59 mm to (160.5, 30.0)
- moved L10 3.85 mm to (183.7, 43.5)
- moved D2 3.76 mm to (170.5, 38.0)
- moved C10 3.50 mm to (173.8, 35.8)
- moved C11 3.50 mm to (172.8, 35.8)
- moved C12 3.50 mm to (171.8, 35.8)
- moved C16 3.50 mm to (178.4, 43.8)
- moved C17 3.50 mm to (178.4, 44.7)
- moved C18 3.50 mm to (177.0, 35.4)
- moved C23 3.50 mm to (183.5, 48.0)
- moved C24 3.50 mm to (175.5, 30.0)
- moved C25 3.50 mm to (175.5, 50.0)
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Connections:
- U1 pad 29: REFCLK -> Net-(U1-REFIN)
- U2 pad 29: REFCLK -> Net-(U2-REFIN)
- U4 pad 1: CE1 -> +5V
- U4 pad 2: unconnected-(U4-PA1-Pad2) -> GND
- U4 pad 3: unconnected-(U4-PA2-Pad3) -> +5V
- U4 pad 4: GND -> unconnected-(U4-NC-Pad4)
- U4 pad 5: unconnected-(U4-PD0-Pad5) -> +3.3V
Routing:
- net GND: track 235.9 -> 423.0 mm, vias 11 -> 283
- net REFCLK: track 21.8 -> 77.2 mm
- net CE0: track 0.00 -> 51.4 mm, vias 0 -> 2
- net SCK: track 1.78 -> 52.9 mm, vias 0 -> 3
- net LE0: track 0.00 -> 50.8 mm, vias 0 -> 2
- net MOSI: track 2.50 -> 52.3 mm, vias 0 -> 3
- net +3.3V: track 37.7 -> 79.2 mm, vias 8 -> 15
- net +3V3: track 0.00 -> 36.6 mm, vias 0 -> 6
- net MUXOUT0: track 5.37 -> 39.7 mm, vias 0 -> 4
- net +5V: track 0.00 -> 33.6 mm, vias 0 -> 2
- net D+: track 0.00 -> 26.3 mm, vias 0 -> 2
- net D-: track 0.00 -> 25.2 mm, vias 0 -> 2
- net SWC: track 0.00 -> 24.1 mm, vias 0 -> 2
- net XTALEN: track 0.00 -> 23.8 mm, vias 0 -> 4
- net SWD: track 0.00 -> 19.7 mm, vias 0 -> 2
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- added copper zone on B.Cu, net GND
- added copper zone on F.Cu, net GND

Commit message: Bump
Parts:
- moved Y1 0.20 mm to (160.2, 30.0)
- moved J15 0.07 mm to (150.4, 35.8)
Routing:
- net GND: track 423.0 -> 442.2 mm, vias 283 -> 286
- net SCK: track 52.9 -> 50.4 mm
- net MOSI: track 52.3 -> 53.1 mm

Commit message: Bump designs
Parts:
- J11: value USB_C_Receptacle_USB2.0_14P -> J20-C-V-C-1-SMT-TR-USB-VERTICAL; footprint Connector_USB:USB_C_Receptacle_G-Switch_GT-USB-7051x -> cnhardware:J20-C-V-C-1-SMT-TR-USB-VERTICAL
- moved R13 0.47 mm to (146.3, 33.1)
- moved R14 0.22 mm to (152.1, 27.8)
Routing:
- net GND: track 442.2 -> 425.3 mm, vias 286 -> 294
- net Net-(J11-D+-PadA6): track 5.41 -> 8.95 mm, vias 1 -> 2
- net Net-(J11-D--PadA7): track 6.75 -> 5.50 mm, vias 2 -> 1
- net Net-(J11-CC1): track 3.12 -> 4.33 mm
- net +5V: track 33.6 -> 34.2 mm, vias 2 -> 1
Other:
- board text added: "J20-C-V-C-1 USB"
- board text added: "amplifier addlepatedarray cnhardware rev -"
