File: addlepatedarray/synthtest/synthtest.kicad_sch (KiCad schematic)
At the start: 61 parts, among them J1 RF0A+, J2 RF0A-, J3 RF0B-, J4 RF0B+, J5 RF1A-, J6 RF1B-, J7 RF1A+, J8 RF1B+, J9 REF, U1 ADF4351, U2 ADF4351, U4 CH32V003FxUx, U6 LDL1117-33, Y1 TG-5006CG-12H 26.0000M3

Commit message: Bump design
Parts:
- removed U3: ~, Package_DFN_QFN:QFN-28-1EP_4x4mm_P0.4mm_EP2.3x2.3mm, symbol cnhardware:CH32V203G6
Other:
- moved on the sheet: J9
Changed lines of the file:
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@@
 	(text "TODO: Transition to 203 maybe?  Maybe 307 for all ethernet?"
 		(exclude_from_sim no)
-		(at 146.558 146.558 0)
+		(at 146.812 142.24 0)
 		(effects
 			(font
@@
 	(wire
 		(pts
-			(xy 50.8 148.59) (xy 48.26 148.59)
+			(xy 69.85 140.97) (xy 67.31 140.97)
 		)
 		(stroke
@@
 	(wire
 		(pts
-			(xy 38.1 148.59) (xy 43.18 148.59)
+			(xy 57.15 140.97) (xy 62.23 140.97)
 		)
 		(stroke
@@
 	(global_label "REFCLK"
 		(shape input)
-		(at 38.1 148.59 180)
+		(at 57.15 140.97 180)
 		(fields_autoplaced yes)
 		(effects
@@
 		)
 		(property "Intersheetrefs" "${INTERSHEET_REFS}"
-			(at 28.0391 148.59 0)
+			(at 47.0891 140.97 0)
 			(effects
 				(font
@@
 	(symbol
 		(lib_id "Connector:Conn_Coaxial_Small")
-		(at 45.72 148.59 0)
+		(at 64.77 140.97 0)
 		(unit 1)
 		(exclude_from_sim no)
@@
 		(dnp no)
 		(property "Reference" "J9"
-			(at 43.18 149.606 0)
+			(at 62.23 141.986 0)
 			(effects
 				(font
@@
 		)
 		(property "Value" "REF"
-			(at 41.91 147.574 0)
+			(at 60.96 139.954 0)
 			(effects
 				(font
@@
 		)
 		(property "Footprint" "Connector_Coaxial:SMA_Molex_73251-1153_EdgeMount_Horizontal"
-			(at 45.72 148.59 0)
+			(at 64.77 140.97 0)
 			(effects
 				(font
@@
 		)
 		(property "Datasheet" "~"
-			(at 45.72 148.59 0)
+			(at 64.77 140.97 0)
 			(effects
 				(font
@@
 		)
 		(property "Description" "small coaxial connector (BNC, SMA, SMB, SMC, Cinch/RCA, LEMO, ...)"
-			(at 45.72 148.59 0)
+			(at 64.77 140.97 0)
 			(effects
 				(font
@@
 		)
 		(property "LCSC" "C496550"
-			(at 45.72 148.59 0)
+			(at 64.77 140.97 0)
 			(effects
 				(font
@@
 	)
 	(symbol
-		(lib_id "cnhardware:CH32V203G6")
-		(at 147.32 165.1 0)
-		(unit 1)
-		(exclude_from_sim no)
-		(in_bom yes)
-		(on_board yes)
-		(dnp no)
-		(fields_autoplaced yes)
-		(property "Reference" "U3"
-			(at 162.56 152.3298 0)
-			(effects
-				(font
-					(size 1.27 1.27)
-				)
-			)
-		)
-		(property "Value" "~"
-			(at 162.56 154.2349 0)
-			(effects
-				(font
-					(size 1.27 1.27)
-				)
-			)
-		)
-		(property "Footprint" "Package_DFN_QFN:QFN-28-1EP_4x4mm_P0.4mm_EP2.3x2.3mm"
-			(at 147.32 158.75 0)
-			(effects
-				(font
-					(size 1.27 1.27)
-				)
-				(hide yes)
-			)
-		)
-		(property "Datasheet" ""
-			(at 147.32 168.91 0)
-			(effects
-				(font
-					(size 1.27 1.27)
-				)
-				(hide yes)
-			)
-		)
-		(property "Description" ""
-			(at 147.32 168.91 0)
-			(effects
-				(font
-					(size 1.27 1.27)
-				)
-				(hide yes)
-			)
-		)
-		(property "LCSC" "C5142280"
-			(at 147.32 168.91 0)
-			(effects
-				(font
-					(size 1.27 1.27)
-				)
-				(hide yes)
-			)
-		)
-		(pin "17"
-		)
-		(pin "19"
-		)
-		(pin "22"
-		)
-		(pin "16"
-		)
-		(pin "23"
-		)
-		(pin "18"
-		)
-		(pin "14"
-		)
-		(pin "21"
-		)
-		(pin "20"
-		)
-		(pin "15"
-		)
-		(pin "13"
-		)
-		(pin "3"
-		)
-		(pin "8"
-		)
-		(pin "6"
-		)
-		(pin "27"
-		)
-		(pin "12"
-		)
-		(pin "1"
-		)
-		(pin "25"
-		)
-		(pin "4"
-		)
-		(pin "7"
-		)
-		(pin "9"
-		)
-		(pin "5"
-		)
-		(pin "28"
-		)
-		(pin "26"
-		)
-		(pin "2"
-		)
-		(pin "11"
-		)
-		(pin "29"
-		)
-		(pin "24"
-		)
-		(pin "10"
-		)
-		(instances
-			(project ""
-				(path "/b7aed664-0534-4168-8983-734ced7f9c05"
-					(reference "U3")
-					(unit 1)
-				)
-			)
-		)
-	)
-	(symbol
 		(lib_id "Device:L_Small")
 		(at 241.3 88.9 90)
@@
 	(symbol
 		(lib_id "power:GND")
-		(at 50.8 148.59 0)
+		(at 69.85 140.97 0)
 		(unit 1)
 		(exclude_from_sim no)
@@
 		(fields_autoplaced yes)
 		(property "Reference" "#PWR069"
-			(at 50.8 154.94 0)
+			(at 69.85 147.32 0)
 			(effects
 				(font
@@
 		)
 		(property "Value" "GND"
-			(at 50.8 153.67 0)
+			(at 69.85 146.05 0)
 			(effects
 				(font
@@
 		)
 		(property "Footprint" ""
-			(at 50.8 148.59 0)
+			(at 69.85 140.97 0)
 			(effects
 				(font
@@
 		)
 		(property "Datasheet" ""
-			(at 50.8 148.59 0)
+			(at 69.85 140.97 0)
 			(effects
 				(font
@@
 		)
 		(property "Description" "Power symbol creates a global label with name \"GND\" , ground"
-			(at 50.8 148.59 0)
+			(at 69.85 140.97 0)
 			(effects
 				(font

Commit message: Bump design
Parts:
- J1, J2, J3, J4, J5, J6, J7, J8, J9: footprint Connector_Coaxial:SMA_Molex_73251-1153_EdgeMount_Horizontal -> Connector_Coaxial:SMA_Amphenol_901-144_Vertical; LCSC C496550 -> C5301852
- R10, R8: footprint Resistor_SMD:R_0603_1608Metric -> Resistor_SMD:R_0402_1005Metric; LCSC C23228 -> C25109
- R7, R9: footprint Resistor_SMD:R_0603_1608Metric -> Resistor_SMD:R_0402_1005Metric; LCSC C23151 -> C25109
Changed lines of the file:
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@@
 			)
 		)
-		(property "Footprint" "Connector_Coaxial:SMA_Molex_73251-1153_EdgeMount_Horizontal"
+		(property "Footprint" "Connector_Coaxial:SMA_Amphenol_901-144_Vertical"
 			(at 271.78 91.44 0)
 			(effects
@@
 			)
 		)
-		(property "LCSC" "C496550"
+		(property "LCSC" "C5301852"
 			(at 271.78 91.44 0)
 			(effects
@@
 			)
 		)
-		(property "Footprint" "Connector_Coaxial:SMA_Molex_73251-1153_EdgeMount_Horizontal"
+		(property "Footprint" "Connector_Coaxial:SMA_Amphenol_901-144_Vertical"
 			(at 271.78 81.28 0)
 			(effects
@@
 			)
 		)
-		(property "LCSC" "C496550"
+		(property "LCSC" "C5301852"
 			(at 271.78 81.28 0)
 			(effects
@@
 			)
 		)
-		(property "Footprint" "Resistor_SMD:R_0603_1608Metric"
+		(property "Footprint" "Resistor_SMD:R_0402_1005Metric"
 			(at 120.65 104.648 90)
 			(effects
@@
 			)
 		)
-		(property "LCSC" "C23228"
+		(property "LCSC" "C25109"
 			(at 120.65 102.87 0)
 			(effects
@@
 			)
 		)
-		(property "Footprint" "Connector_Coaxial:SMA_Molex_73251-1153_EdgeMount_Horizontal"
+		(property "Footprint" "Connector_Coaxial:SMA_Amphenol_901-144_Vertical"
 			(at 134.62 82.55 0)
 			(effects
@@
 			)
 		)
-		(property "LCSC" "C496550"
+		(property "LCSC" "C5301852"
 			(at 134.62 82.55 0)
 			(effects
@@
 			)
 		)
-		(property "Footprint" "Resistor_SMD:R_0603_1608Metric"
+		(property "Footprint" "Resistor_SMD:R_0402_1005Metric"
 			(at 252.73 105.918 90)
 			(effects
@@
 			)
 		)
-		(property "LCSC" "C23228"
+		(property "LCSC" "C25109"
 			(at 252.73 104.14 0)
 			(effects
@@
 			)
 		)
-		(property "Footprint" "Connector_Coaxial:SMA_Molex_73251-1153_EdgeMount_Horizontal"
+		(property "Footprint" "Connector_Coaxial:SMA_Amphenol_901-144_Vertical"
 			(at 139.7 80.01 0)
 			(effects
@@
 			)
 		)
-		(property "LCSC" "C496550"
+		(property "LCSC" "C5301852"
 			(at 139.7 80.01 0)
 			(effects
@@
 			)
 		)
-		(property "Footprint" "Connector_Coaxial:SMA_Molex_73251-1153_EdgeMount_Horizontal"
+		(property "Footprint" "Connector_Coaxial:SMA_Amphenol_901-144_Vertical"
 			(at 139.7 90.17 0)
 			(effects
@@
 			)
 		)
-		(property "LCSC" "C496550"
+		(property "LCSC" "C5301852"
 			(at 139.7 90.17 0)
 			(effects
@@
 			)
 		)
-		(property "Footprint" "Connector_Coaxial:SMA_Molex_73251-1153_EdgeMount_Horizontal"
+		(property "Footprint" "Connector_Coaxial:SMA_Amphenol_901-144_Vertical"
 			(at 64.77 140.97 0)
 			(effects
@@
 			)
 		)
-		(property "LCSC" "C496550"
+		(property "LCSC" "C5301852"
 			(at 64.77 140.97 0)
 			(effects
@@
 			)
 		)
-		(property "Footprint" "Connector_Coaxial:SMA_Molex_73251-1153_EdgeMount_Horizontal"
+		(property "Footprint" "Connector_Coaxial:SMA_Amphenol_901-144_Vertical"
 			(at 266.7 93.98 0)
 			(effects
@@
 			)
 		)
-		(property "LCSC" "C496550"
+		(property "LCSC" "C5301852"
 			(at 266.7 93.98 0)
 			(effects
@@
 			)
 		)
-		(property "Footprint" "Resistor_SMD:R_0603_1608Metric"
+		(property "Footprint" "Resistor_SMD:R_0402_1005Metric"
 			(at 247.142 115.57 90)
 			(effects
@@
 			)
 		)
-		(property "LCSC" "C23151"
+		(property "LCSC" "C25109"
 			(at 248.92 115.57 0)
 			(effects
@@
 			)
 		)
-		(property "Footprint" "Connector_Coaxial:SMA_Molex_73251-1153_EdgeMount_Horizontal"
+		(property "Footprint" "Connector_Coaxial:SMA_Amphenol_901-144_Vertical"
 			(at 134.62 92.71 0)
 			(effects
@@
 			)
 		)
-		(property "LCSC" "C496550"
+		(property "LCSC" "C5301852"
 			(at 134.62 92.71 0)
 			(effects
@@
 			)
 		)
-		(property "Footprint" "Connector_Coaxial:SMA_Molex_73251-1153_EdgeMount_Horizontal"
+		(property "Footprint" "Connector_Coaxial:SMA_Amphenol_901-144_Vertical"
 			(at 266.7 83.82 0)
 			(effects
@@
 			)
 		)
-		(property "LCSC" "C496550"
+		(property "LCSC" "C5301852"
 			(at 266.7 83.82 0)
 			(effects
@@
 			)
 		)
-		(property "Footprint" "Resistor_SMD:R_0603_1608Metric"
+		(property "Footprint" "Resistor_SMD:R_0402_1005Metric"
 			(at 115.062 114.3 90)
 			(effects
@@
 			)
 		)
-		(property "LCSC" "C23151"
+		(property "LCSC" "C25109"
 			(at 116.84 114.3 0)
 			(effects

Commit message: Bump
Parts:
- added C27, C28, C30, C31, C32, C33, C35, C36: 1n, Capacitor_SMD:C_0402_1005Metric, symbol Device:C
- added C29, C34: 1u, Capacitor_SMD:C_0402_1005Metric, symbol Device:C
- added L10, L9: 3.9nH, Inductor_SMD:L_0402_1005Metric, symbol Device:L_Small
Connections:
- net +3.3V: now also C27.2, C30.2, C31.2, C33.2, C35.2, C36.2, L10.1, L9.1
- net GND: now also C27.1, C28.1, C29.2, C30.1, C31.1, C32.1, C33.1, C34.2, C35.1, C36.1
- net VVCO0: now also C28.2, C29.1, L9.2
- net VVCO1: now also C32.2, C34.1, L10.2
Other:
- note added: "To investigate: 1. REFIN on ADF4351 - should it be hard lined in or with GND offset? 2. Consider LP5907 for LDO 3. Add ferrite bead to AVDDs? And Vs of XTAL? TODO: * Terminate the reference oscillator"
- note removed: "To investigate: 1. REFIN on ADF4351 - should it be hard lined in or with GND offset? 2. Consider LP5907 for LDO 3. Add ferrite bead to AVDDs? And Vs of XTAL?"

Commit message: Bump disign!
Parts:
- removed D3: LEDPWR, LED_SMD:LED_0603_1608Metric, symbol Device:LED
- removed U4: CH32V003FxUx, Package_DFN_QFN:QFN-20-1EP_3x3mm_P0.4mm_EP1.65x1.65mm, symbol MCU_WCH_CH32V0:CH32V003FxUx
- removed U6: LDL1117-33, Package_TO_SOT_SMD:SOT-223-3_TabPin2, symbol Regulator_Linear:AMS1117-3.3
- added C37, C38, C39, C40: 1n, Capacitor_SMD:C_0402_1005Metric, symbol Device:C
- added C41, C43, C44, C48: 1u, Capacitor_SMD:C_0402_1005Metric, symbol Device:C
- added C42, C45, C46, C47: 4.7u, Capacitor_SMD:C_0603_1608Metric, symbol Device:C
- added J10: RJ45_Hanrun_HR911105A_Horizontal, cnhardware:HR915310A-RJ45-INTEGRATED-10MBIT, symbol Connector:RJ45_Hanrun_HR911105A_Horizontal
- added J11: USB_C_Receptacle_USB2.0_14P, Connector_USB:USB_C_Receptacle_G-Switch_GT-USB-7051x, symbol Connector:USB_C_Receptacle_USB2.0_14P
- added J12: VCC, TestPoint:TestPoint_Pad_D1.0mm, symbol Connector_Generic:Conn_01x01
- added J13: SWC, TestPoint:TestPoint_Pad_D1.0mm, symbol Connector_Generic:Conn_01x01
- added J14: SWD, TestPoint:TestPoint_Pad_D1.0mm, symbol Connector_Generic:Conn_01x01
- added J15: GND, TestPoint:TestPoint_Pad_D1.0mm, symbol Connector_Generic:Conn_01x01
- added L11: 3.9nH, Inductor_SMD:L_0402_1005Metric, symbol Device:L_Small
- added R11, R3: 100, Resistor_SMD:R_0402_1005Metric, symbol Device:R
- added R12: 1.5k, cnhardware:R_0402_1005Metric_COMPACT, symbol Device:R
- added R13, R14: 5.1k, Resistor_SMD:R_0402_1005Metric, symbol Device:R
- added R15, R16: 33, Resistor_SMD:R_0402_1005Metric, symbol Device:R
- added U3: CH32V208GBU6, Package_DFN_QFN:QFN-28-1EP_4x4mm_P0.45mm_EP2.6x2.6mm, symbol cnhardware:CH32V208GBU6
- added U4, U5: WL2808E, Package_TO_SOT_SMD:SOT-23-5, symbol Regulator_Linear:MCP1802x-xx02xOT
- added Y3: 32MHz, Crystal:Crystal_SMD_2016-4Pin_2.0x1.6mm, symbol Device:Crystal_GND24_Small
Connections:
- net +3.3V: now also C46.1, U4.5 (VOUT)
- net +5V: now also C45.1, C47.1, J11.A4 (VBUS), J11.A9 (VBUS), J11.B4 (VBUS), J11.B9 (VBUS), U4.1 (VIN), U4.3 (~{SHDN}), U5.1 (VIN), U5.3 (~{SHDN})
- net CE0: now also U3.28 (PC14)
- net CE1: now also U3.6 (PA1)
- net D+: now also R16.2, U3.25 (PB7/U2+)
- net D-: now also R15.2, U3.24 (PB6/U2-)
- net GND: now also C41.2, C42.2, C43.2, C44.2, C45.2, C46.2, C47.2, C48.2, J10.8, J10.SH, J11.A1 (GND), J11.A12 (GND), J11.B1 (GND), J11.B12 (GND), J11.S1 (SHIELD), J15.1 (Pin_1), R11.2, R12.2, R13.2, R14.2, R3.2, U3.29 (GND), U4.2 (GND), U5.2 (GND), Y3.2, Y3.4
- net LE0: now also U3.1 (PC15)
- net LE1: now also U3.7 (PA2)
- net MOSI: now also U3.12 (PA7)
- net MUXOUT0: now also U3.5 (PA0)
- net MUXOUT1: now also U3.8 (PA3)
- net REFCLK: now also C37.1, C39.1; no longer U1.29 (REFIN), U2.29 (REFIN)
- net SCK: now also U3.10 (PA5)
- net SWD: now also J14.1 (Pin_1), U3.20 (SWD)
- net XTALEN: now also U3.18 (PA11/USB1DM)
- net at R6.1: now also J10.11
- new net: J11.A5 (CC1), R13.1
- new net: C48.1, U3.21 (VINTA)
- new net: J10.10, R12.1
- new net: C41.1, J10.4 (TCT), J10.5 (RCT), L11.2
- new net: J11.B5 (CC2), R14.1
- new net: J11.A6 (D+), J11.B6 (D+), R16.1
- new net: J11.A7 (D-), J11.B7 (D-), R15.1
- new net: C38.2, U1.29 (REFIN)
- new net: C39.2, C40.1, R11.1
- new net: C40.2, U2.29 (REFIN)
- new net: U3.3 (OSC_OUT), Y3.1
- new net: U3.2 (OSC_IN), Y3.3
- new net: C37.2, C38.1, R3.1
- new net +3V3: C42.1, C43.1, C44.1, J12.1 (Pin_1), L11.1, U3.13 (VDD_VIO), U3.27 (VDD), U3.4 (VDDA), U5.5 (VOUT)
- new net ERXN: J10.6 (RD-), U3.15 (PC7)
- new net ERXP: J10.3 (RD+), U3.14 (PC6)
- new net ETXN: J10.2 (TD-), U3.17 (PC9)
- new net ETXP: J10.1 (TD+), U3.16 (PC8)
- new net LEDG: J10.9, U3.11 (PA6)
- new net LEDY: J10.12, U3.22 (ANT)
- new net SWC: J13.1 (Pin_1), U3.23 (SWC)
Other:
- note added: "40mm trace, balanced to each on ref clock (one 7.5GHz wavelength). Kind of irrelevant, since it's terminating into two 100 ohm resistors."
- note added: "Oscillator: * Clipped sinewave (https://ez.analog.com/rf/f/q-a/75586/how-to-drive-multiple-pll-refin-pins-with-a-single-tcxo) * 3.3V * +/- 5ppm over lifeimte. Distortion < 1ppm. ADF435x: * ADF4350: 137MHz miniumum * ADF4351: 37.5MHz minimum * PSU @ 3.0-3.6V (Use 3.3V) * Not using Fast Lock mode. Regulator: * Vdropout < 1V * >800mA * PSRR 65dB or less @ 1kHz (80dB or less @ 100Hz) * SOT-23 LDL1117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"
- note added: "To investigate: 1. REFIN on ADF4351 - should it be hard lined in or with GND offset? 2. Consider LP5907 for LDO 3. Add ferrite bead to AVDDs? And Vs of XTAL?"
- note removed: "Oscillator: * Clipped sinewave (https://ez.analog.com/rf/f/q-a/75586/how-to-drive-multiple-pll-refin-pins-with-a-single-tcxo) * 3.3V * +/- 5ppm over lifeimte. Distortion < 1ppm. ADF435x: * ADF4350: 137MHz miniumum * ADF4351: 37.5MHz minimum * PSU @ 3.0-3.6V (Use 3.3V) * Not using Fast Lock mode. Regulator: * Vdropout < 1V * >800mA * PSRR 65dB or less @ 1kHz (80dB or less @ 100Hz)"
- note removed: "TODO: Transition to 203 maybe? Maybe 307 for all ethernet?"
- note removed: "To investigate: 1. REFIN on ADF4351 - should it be hard lined in or with GND offset? 2. Consider LP5907 for LDO 3. Add ferrite bead to AVDDs? And Vs of XTAL? TODO: * Terminate the reference oscillator"
- moved on the sheet: C30, C31, C32, C34, C35, J9, L10, R6, Y1

Commit message: Bump designs
Parts:
- J11: value USB_C_Receptacle_USB2.0_14P -> J20-C-V-C-1-SMT-TR-USB-VERTICAL; footprint Connector_USB:USB_C_Receptacle_G-Switch_GT-USB-7051x -> cnhardware:J20-C-V-C-1-SMT-TR-USB-VERTICAL
Changed lines of the file:
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@@
 			)
 		)
-		(property "Value" "USB_C_Receptacle_USB2.0_14P"
+		(property "Value" "J20-C-V-C-1-SMT-TR-USB-VERTICAL"
 			(at 30.48 144.78 0)
 			(effects
@@
 			)
 		)
-		(property "Footprint" "Connector_USB:USB_C_Receptacle_G-Switch_GT-USB-7051x"
+		(property "Footprint" "cnhardware:J20-C-V-C-1-SMT-TR-USB-VERTICAL"
 			(at 34.29 165.1 0)
 			(effects
