File: ch32v30x/ch32v305-scopesend/ch32v305-scopesend.kicad_sch (KiCad schematic)
At the start: 61 parts, among them J1 Conn_01x05, J2 USB_C_Receptacle_USB2.0, J3 PA15, J4 PA15, J5 MAG_DEFLECTION, SW1 Download, U1 CH32V305RBT6, U2 AD9767, U3 XC6206P332MR-G, U4 XC6206P332MR-G, U5 TPS563201, Y1 Crystal

Commit message: Udpate design
Parts:
- removed U6, U7, U8, U9: (no value), cnhardware:S-PVQFN-N12, symbol cnhardware:OPA567AIRHGT
- added R1: 5.1k, Resistor_SMD:R_0402_1005Metric, symbol Device:R
- added U6: OPA564, Package_SO:HSOP-20-1EP_11.0x15.9mm_P1.27mm_SlugUp, symbol cnhardware:OPA564AIDWDR-TOP-SINK
Connections:
- net VO2: now also U6.5 (VOUT), U6.6 (VOUT)
- new net: R1.2, U6.12 (ISET)
Other:
- note added: "Originally tried: OPA567AIRHGR but voltage limits :("
- note added: "Use 2x OPA564"
