File: xmastree/mainboard/mainboard.kicad_sch (KiCad schematic)
At the start: 24 parts, among them J1 ATX-24, J2 ATX, J3 Conn_01x05, J3 PA15, J4 PA15, J4 USB_C_Receptacle_USB2.0, SW1 Download, U1 AMS1117, U2 CH32V305RBT6, Y1 Crystal

Commit message: Bump design
Parts:
- removed J4: PA15, symbol Connector_Generic:Conn_01x01
- removed Y1: Crystal, symbol Device:Crystal
- added C10: 1u, Resistor_SMD:R_0402_1005Metric, symbol Device:C
- added D1, D2, D3, D4: DT1240A-08LP3810, Package_DFN_QFN:UDFN-9_1.0x3.8mm_P0.5mm, symbol Power_Protection:DT1240A-08LP3810
- added J10: PA7, TestPoint:TestPoint_Pad_D1.0mm, symbol Connector_Generic:Conn_01x01
- added J11, J12, J13, J14, J15, J16, J17, J18, J19, J20, J21, J22, J23, J24, J25, J26, J27, J28, J29, J30, J31, J32, J33, J34, J35, J36, J37, J38, J39, J40, J41, J5: LED, TerminalBlock_TE-Connectivity:TerminalBlock_TE_282834-3_1x03_P2.54mm_Horizontal, symbol Connector_Generic:Conn_01x03
- added J3: PA0, TestPoint:TestPoint_Pad_D1.0mm, symbol Connector_Generic:Conn_01x01
- added J42, J43, J44, J45: ATX, Connector_Molex:Molex_Mini-Fit_Jr_5566-08A2_2x04_P4.20mm_Vertical, symbol Connector_Generic_Shielded:Conn_02x04_Top_Bottom_Shielded
- added J8: PA15, TestPoint:TestPoint_Pad_D1.0mm, symbol Connector_Generic:Conn_01x01
- added J9: PA2, TestPoint:TestPoint_Pad_D1.0mm, symbol Connector_Generic:Conn_01x01
- added R10, R11, R12, R13, R14, R15, R16, R17, R18, R19, R20, R21, R22, R23, R24, R25, R26, R27, R28, R29, R30, R31, R32, R33, R34, R35, R36, R37, R6, R7, R8, R9: 120, Resistor_SMD:R_0402_1005Metric, symbol Device:R
- added R38, R39: 22, Resistor_SMD:R_0402_1005Metric, symbol Device:R
- added Y2: 8MHz, Crystal:Crystal_SMD_3225-4Pin_3.2x2.5mm_HandSoldering, symbol Device:Crystal_GND24_Small
- J1: footprint Connector_Molex:Molex_Mini-Fit_Jr_5566-24A_2x12_P4.20mm_Vertical -> Connector_Molex:Molex_Mini-Fit_Jr_5566-24A2_2x12_P4.20mm_Vertical
- J4: renamed from J3; value PA15 -> PA1; footprint (none) -> TestPoint:TestPoint_Pad_D1.0mm
- J7: renamed from J3; value Conn_01x05 -> PAGM; footprint (none) -> Connector_PinHeader_2.54mm:PinHeader_1x05_P2.54mm_Vertical; LCSC (none) -> C32713271
- renumbered C4 to C1, C5 to C2, C1 to C4, C14 to C5, C9 to C6, C6 to C7, C2 to C8, C13 to C9, J4 to J6, R7 to R3, R3 to R5, U2 to U1, U1 to U2
Connections:
- net BOOT0: now also U1.60 (BOOT0)
- net PA15: now also U1.50 (PA15), J8.1 (Pin_1); no longer J4.1 (Pin_1)
- net RST: now also U1.7 (~{RST})
- net USBDM: now also R38.2
- net USBDP: now also R39.2
- net VDD: now also J7.4 (Pin_4), C10.2
- net GND: now reaches C2.1
- net GND: now also C1.1, C3.1, C4.1, C5.1, C6.1, C7.1, C8.1, C9.1, J1.15 (GND), J1.17 (GND), J1.18 (GND), J1.19 (GND), J1.24 (GND), J1.3 (GND), J1.5 (GND), J1.7 (GND), J2.4 (Pin_4), J2.5 (Pin_5), J2.7 (Pin_7), J2.8 (Pin_8), J2.SH (Shield), J6.A1 (GND), J6.A12 (GND), J6.B1 (GND), J6.B12 (GND), J6.S1 (SHIELD), J7.5 (Pin_5), R2.1, R3.2, R4.2, R5.2, U1.12 (VSSA), U1.18 (VSS), U1.31 (VSS), U1.47 (VSS), U1.63 (VSS), C10.1, D1.3 (A), D2.3 (A), D3.3 (A), D4.3 (A), J11.1 (Pin_1), J12.1 (Pin_1), J13.1 (Pin_1), J14.1 (Pin_1), J15.1 (Pin_1), J16.1 (Pin_1), J17.1 (Pin_1), J18.1 (Pin_1), J19.1 (Pin_1), J20.1 (Pin_1), J21.1 (Pin_1), J22.1 (Pin_1), J23.1 (Pin_1), J24.1 (Pin_1), J25.1 (Pin_1), J26.1 (Pin_1), J27.1 (Pin_1), J28.1 (Pin_1), J29.1 (Pin_1), J30.1 (Pin_1), J31.1 (Pin_1), J32.1 (Pin_1), J33.1 (Pin_1), J34.1 (Pin_1), J35.1 (Pin_1), J36.1 (Pin_1), J37.1 (Pin_1), J38.1 (Pin_1), J39.1 (Pin_1), J40.1 (Pin_1), J41.1 (Pin_1), J42.4 (Pin_4), J42.5 (Pin_5), J42.7 (Pin_7), J42.8 (Pin_8), J42.SH (Shield), J43.4 (Pin_4), J43.5 (Pin_5), J43.7 (Pin_7), J43.8 (Pin_8), J43.SH (Shield), J44.4 (Pin_4), J44.5 (Pin_5), J44.7 (Pin_7), J44.8 (Pin_8), J44.SH (Shield), J45.4 (Pin_4), J45.5 (Pin_5), J45.8 (Pin_8), J45.SH (Shield), J5.1 (Pin_1), Y2.2, Y2.4
- net at C2.2, U1.5 (OSC_IN): now also Y2.3
- net at C1.2, U1.6 (OSC_OUT): now also Y2.1
- net 12V1: now reaches J2.1 (Pin_1)
- net 12V1: now also J2.2 (Pin_2), J2.3 (Pin_3), J11.3 (Pin_3), J12.3 (Pin_3), J13.3 (Pin_3), J14.3 (Pin_3), J15.3 (Pin_3), J5.3 (Pin_3)
- net 12V6: now reaches J1.10 (+12V), J1.11 (+12V)
- net 12V6: now also J40.3 (Pin_3), J41.3 (Pin_3)
- net PA9: now reaches J1.16 (PS_ON#)
- net PA9: now also U1.42 (PA9)
- net PA10: now reaches J1.8 (PWR_OK)
- net PA10: now also U1.43 (PA10)
- net at U1.10 (PC2): now also R23.1
- net at U1.11 (PC3): now also R31.1
- net PA0: now reaches U1.14 (PA0)
- net PA0: now also J3.1 (Pin_1)
- net PA1: now reaches U1.15 (PA1)
- net PA1: now also J4.1 (Pin_1)
- net PA2: now reaches U1.16 (PA2)
- net PA2: now also J9.1 (Pin_1)
- net at U1.2 (PC13): now also R36.1
- net PA7: now reaches U1.23 (PA7)
- net PA7: now also J10.1 (Pin_1)
- net at U1.24 (PC4): now also R24.1
- net at U1.25 (PC5): now also R32.1
- net at U1.26 (PB0): now also R6.1
- net at U1.27 (PB1): now also R7.1
- net at U1.28 (PB2): now also R8.1
- net at U1.29 (PB10): now also R15.1
- net at U1.3 (PC14): now also R29.1
- net at U1.30 (PB11): now also R17.1
- net at U1.33 (PB12): now also R18.1
- net at U1.34 (PB13): now also R20.1
- net at U1.35 (PB14): now also R19.1
- net at U1.36 (PB15): now also R21.1
- net at U1.37 (PC6): now also R25.1
- net at U1.38 (PC7): now also R33.1
- net at U1.39 (PC8): now also R26.1
- net at U1.4 (PC15): now also R37.1
- net at U1.40 (PC9): now also R34.1
- net at U1.51 (PC10): now also R27.1
- net at U1.52 (PC11): now also R35.1
- net at U1.53 (PC12): now also R28.1
- net at U1.55 (PB3): now also R9.1
- net at U1.56 (PB4): now also R10.1
- net at U1.57 (PB5): now also R12.1
- net at U1.58 (PB6): now also R11.1
- net at U1.59 (PB7): now also R13.1
- net at U1.61 (PB8): now also R14.1
- net at U1.62 (PB9): now also R16.1
- net at U1.8 (PC0): now also R22.1
- net at U1.9 (PC1): now also R30.1
- net D+: no longer names the net of J6.A6 (D+), J6.B6 (D+)
- net D+: now also R39.1
- net D-: no longer names the net of J6.A7 (D-), J6.B7 (D-)
- net D-: now also R38.1
- new net 12V2: J16.3 (Pin_3), J17.3 (Pin_3), J18.3 (Pin_3), J19.3 (Pin_3), J20.3 (Pin_3), J21.3 (Pin_3), J42.1 (Pin_1), J42.2 (Pin_2), J42.3 (Pin_3)
- new net 12V3: J22.3 (Pin_3), J23.3 (Pin_3), J24.3 (Pin_3), J25.3 (Pin_3), J26.3 (Pin_3), J27.3 (Pin_3), J43.1 (Pin_1), J43.2 (Pin_2), J43.3 (Pin_3)
- new net 12V4: J28.3 (Pin_3), J29.3 (Pin_3), J30.3 (Pin_3), J31.3 (Pin_3), J32.3 (Pin_3), J33.3 (Pin_3), J44.1 (Pin_1), J44.2 (Pin_2), J44.3 (Pin_3)
- new net 12V5: J34.3 (Pin_3), J35.3 (Pin_3), J36.3 (Pin_3), J37.3 (Pin_3), J38.3 (Pin_3), J39.3 (Pin_3), J45.1 (Pin_1), J45.2 (Pin_2), J45.3 (Pin_3)
- new net LED0: D1.9 (K8), J5.2 (Pin_2), R6.2
- new net LED1: D1.8 (K7), J11.2 (Pin_2), R7.2
- new net LED10: D2.7 (K6), J20.2 (Pin_2), R15.2
- new net LED11: D2.6 (K5), J21.2 (Pin_2), R17.2
- new net LED12: D2.5 (K4), J22.2 (Pin_2), R18.2
- new net LED13: D2.4 (K3), J23.2 (Pin_2), R20.2
- new net LED14: D2.2 (K2), J24.2 (Pin_2), R19.2
- new net LED15: D2.1 (K1), J25.2 (Pin_2), R21.2
- new net LED16: D3.9 (K8), J26.2 (Pin_2), R22.2
- new net LED17: D3.8 (K7), J27.2 (Pin_2), R30.2
- new net LED18: D3.7 (K6), J28.2 (Pin_2), R23.2
- new net LED19: D3.6 (K5), J29.2 (Pin_2), R31.2
- new net LED2: D1.7 (K6), J12.2 (Pin_2), R8.2
- new net LED20: D3.5 (K4), J30.2 (Pin_2), R24.2
- new net LED21: D3.4 (K3), J31.2 (Pin_2), R32.2
- new net LED22: D3.2 (K2), J32.2 (Pin_2), R25.2
- new net LED23: D3.1 (K1), J33.2 (Pin_2), R33.2
- new net LED24: D4.9 (K8), J34.2 (Pin_2), R26.2
- new net LED25: D4.8 (K7), J35.2 (Pin_2), R34.2
- new net LED26: D4.7 (K6), J36.2 (Pin_2), R27.2
- new net LED27: D4.6 (K5), J37.2 (Pin_2), R35.2
- new net LED28: D4.5 (K4), J38.2 (Pin_2), R28.2
- new net LED29: D4.4 (K3), J39.2 (Pin_2), R36.2
- new net LED3: D1.6 (K5), J13.2 (Pin_2), R9.2
- new net LED30: D4.2 (K2), J40.2 (Pin_2), R29.2
- new net LED31: D4.1 (K1), J41.2 (Pin_2), R37.2
- new net LED4: D1.5 (K4), J14.2 (Pin_2), R10.2
- new net LED5: D1.4 (K3), J15.2 (Pin_2), R12.2
- new net LED6: D1.2 (K2), J16.2 (Pin_2), R11.2
- new net LED7: D1.1 (K1), J17.2 (Pin_2), R13.2
- new net LED8: D2.9 (K8), J18.2 (Pin_2), R14.2
- new net LED9: D2.8 (K7), J19.2 (Pin_2), R16.2
Other:
- note removed: "TODO: Use JST connector TVS the JSTs"
- moved on the sheet: C1, C2, J1, J2, J4, J6, R4, R5, U1

Commit message: Bump design per order
Parts:
- J10, J3, J4, J8, J9: now left out of the parts list
Changed lines of the file:
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@@
 		(unit 1)
 		(exclude_from_sim no)
-		(in_bom yes)
+		(in_bom no)
 		(on_board yes)
 		(dnp no)
@@
 		(unit 1)
 		(exclude_from_sim no)
-		(in_bom yes)
+		(in_bom no)
 		(on_board yes)
 		(dnp no)
@@
 		(unit 1)
 		(exclude_from_sim no)
-		(in_bom yes)
+		(in_bom no)
 		(on_board yes)
 		(dnp no)
@@
 		(unit 1)
 		(exclude_from_sim no)
-		(in_bom yes)
+		(in_bom no)
 		(on_board yes)
 		(dnp no)
@@
 		(unit 1)
 		(exclude_from_sim no)
-		(in_bom yes)
+		(in_bom no)
 		(on_board yes)
 		(dnp no)

Commit message: Update
Parts:
- removed J10: PA7, TestPoint:TestPoint_Pad_D1.0mm, symbol Connector_Generic:Conn_01x01
- removed J9: PA2, TestPoint:TestPoint_Pad_D1.0mm, symbol Connector_Generic:Conn_01x01
- J3: value PA0 -> PA11
- J4: value PA1 -> PA12
Connections:
- net PA7 is gone; now on an unnamed net: U1.23 (PA7)
- net USBDM: now also U1.58 (PB6); no longer U1.44 (PA11)
- net USBDP: now also U1.59 (PB7); no longer U1.45 (PA12)
- net at R11.1: now also U1.22 (PA6); no longer U1.58 (PB6)
- net at R13.1: no longer U1.59 (PB7)
- net PA0: no longer names the net of U1.14 (PA0)
- net PA0: no longer J3.1 (Pin_1)
- net PA1: no longer names the net of U1.15 (PA1)
- net PA1: no longer J4.1 (Pin_1)
- net PA2: no longer names the net of U1.16 (PA2)
- new net PA11: J3.1 (Pin_1), U1.44 (PA11)
- new net PA12: J4.1 (Pin_1), U1.45 (PA12)
- no-connect marks 0 -> 6
Other:
- note added: "CHANGES: 1. USB to PB 2. Use PA6/7 3. TODO: Fix connector for PCIE"
- moved on the sheet: R11, R13

Commit message: Per order
Parts:
- J2, J42, J43, J44, J45: footprint Connector_Molex:Molex_Mini-Fit_Jr_5566-08A2_2x04_P4.20mm_Vertical -> cnhardware:Molex_Mini-Fit_-PCI_EXPRESS-_2x04_P4.20mm_Vertical; LCSC C589025 -> C2886679
Other:
- note added: "Rev A: 1. USB to PB 2. Use PA6/7 3. Fixed"
- note removed: "CHANGES: 1. USB to PB 2. Use PA6/7 3. TODO: Fix connector for PCIE"
Changed lines of the file:
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@@
 	(generator_version "9.0")
 	(paper "A4")
-	(text "CHANGES:\n1. USB to PB\n2. Use PA6/7\n3. TODO: Fix connector for PCIE"
+	(text "Rev A:\n1. USB to PB\n2. Use PA6/7\n3. Fixed"
 		(exclude_from_sim no)
 		(at 157.226 141.224 0)
 		(effects
 			(font
-				(size 3.81 3.81)
-				(thickness 0.762)
-				(bold yes)
+				(size 1.27 1.27)
+				(thickness 0.1588)
 			)
 		)
@@
 			)
 		)
-		(property "Footprint" "Connector_Molex:Molex_Mini-Fit_Jr_5566-08A2_2x04_P4.20mm_Vertical"
+		(property "Footprint" "cnhardware:Molex_Mini-Fit_-PCI_EXPRESS-_2x04_P4.20mm_Vertical"
 			(at 144.78 24.13 0)
 			(effects
@@
 			)
 		)
-		(property "LCSC" "C589025"
+		(property "LCSC" "C2886679"
 			(at 144.78 24.13 0)
 			(effects
@@
 			)
 		)
-		(property "Footprint" "Connector_Molex:Molex_Mini-Fit_Jr_5566-08A2_2x04_P4.20mm_Vertical"
+		(property "Footprint" "cnhardware:Molex_Mini-Fit_-PCI_EXPRESS-_2x04_P4.20mm_Vertical"
 			(at 116.84 24.13 0)
 			(effects
@@
 			)
 		)
-		(property "LCSC" "C589025"
+		(property "LCSC" "C2886679"
 			(at 116.84 24.13 0)
 			(effects
@@
 			)
 		)
-		(property "Footprint" "Connector_Molex:Molex_Mini-Fit_Jr_5566-08A2_2x04_P4.20mm_Vertical"
+		(property "Footprint" "cnhardware:Molex_Mini-Fit_-PCI_EXPRESS-_2x04_P4.20mm_Vertical"
 			(at 173.99 24.13 0)
 			(effects
@@
 			)
 		)
-		(property "LCSC" "C589025"
+		(property "LCSC" "C2886679"
 			(at 173.99 24.13 0)
 			(effects
@@
 			)
 		)
-		(property "Footprint" "Connector_Molex:Molex_Mini-Fit_Jr_5566-08A2_2x04_P4.20mm_Vertical"
+		(property "Footprint" "cnhardware:Molex_Mini-Fit_-PCI_EXPRESS-_2x04_P4.20mm_Vertical"
 			(at 233.68 24.13 0)
 			(effects
@@
 			)
 		)
-		(property "LCSC" "C589025"
+		(property "LCSC" "C2886679"
 			(at 233.68 24.13 0)
 			(effects
@@
 			)
 		)
-		(property "Footprint" "Connector_Molex:Molex_Mini-Fit_Jr_5566-08A2_2x04_P4.20mm_Vertical"
+		(property "Footprint" "cnhardware:Molex_Mini-Fit_-PCI_EXPRESS-_2x04_P4.20mm_Vertical"
 			(at 204.47 24.13 0)
 			(effects
@@
 			)
 		)
-		(property "LCSC" "C589025"
+		(property "LCSC" "C2886679"
 			(at 204.47 24.13 0)
 			(effects
