File: ch570/ch570sao9v/ch570sao9v.kicad_sch (KiCad schematic)
At the start: 42 parts, among them J1 SAO, SW1 TS-1187A-B-A-B, SW2 TS-1187A-B-A-B, SW3 TS-1187A-B-A-B, SW4 SW_SPDT, U2 TPS54302, U3 CH572Q, U4 HX3608_BOOST, Y1 32MHz

Commit message: Tweak design
Parts:
- L1, L2: LCSC C702769 -> C37428
Changed lines of the file:
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@@
 			)
 		)
-		(property "LCSC" "C702769"
+		(property "LCSC" "C37428"
 			(at 234.95 135.89 90)
 			(effects
@@
 			)
 		)
-		(property "LCSC" "C702769"
+		(property "LCSC" "C37428"
 			(at 210.82 137.16 90)
 			(effects

Commit message: Bump design
Parts:
- added TP7: VBAT, TestPoint:TestPoint_Pad_D1.0mm, symbol Connector:TestPoint
- added TP8, TP9: GND, TestPoint:TestPoint_Pad_D1.0mm, symbol Connector:TestPoint
Connections:
- net +9V: now also SW4.2 (B); no longer SW4.1 (A)
- net GND: now also TP8.1, TP9.1
- net at BT1.1 (+): now also SW4.3 (C), TP7.1; no longer SW4.2 (B)
Other:
- note added: "Question: Can we re-use BS1 after boot?"
- moved on the sheet: SW4

Commit message: bump
Parts:
- SW1, SW2, SW3: LCSC C318884 -> (none)
- SW4: LCSC C221841 -> C963206
Changed lines of the file:
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@@
 			)
 		)
-		(property "LCSC" "C318884"
-			(at 123.19 85.09 0)
-			(effects
-				(font
-					(size 1.27 1.27)
-				)
-				(hide yes)
-			)
-		)
 		(pin "1"
 		)
@@
 			)
 		)
-		(property "LCSC" "C318884"
-			(at 123.19 92.71 0)
-			(effects
-				(font
-					(size 1.27 1.27)
-				)
-				(hide yes)
-			)
-		)
 		(pin "1"
 		)
@@
 			)
 		)
-		(property "LCSC" "C318884"
-			(at 123.19 77.47 0)
-			(effects
-				(font
-					(size 1.27 1.27)
-				)
-				(hide yes)
-			)
-		)
 		(pin "1"
 		)
@@
 			)
 		)
-		(property "LCSC" "C221841"
+		(property "LCSC" "C963206"
 			(at 114.3 124.46 0)
 			(effects

Commit message: Add notes in todo
Other:
- note added: "TODO: Examine possible holes for Keystone 590"
Changed lines of the file:
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@@
 	(generator_version "9.0")
 	(paper "A4")
+	(text "TODO: Examine possible holes for Keystone 590"
+		(exclude_from_sim no)
+		(at 50.292 31.75 0)
+		(effects
+			(font
+				(size 1.27 1.27)
+			)
+		)
+	)
 	(text "Question: Can we re-use BS1 after boot?"
 		(exclude_from_sim no)

Commit message: Update part
Parts:
- C14: value 100n -> 10n; LCSC C307331 -> C15195
Connections:
- net VDD: now also U1.6 (VCOT)
- net ADC renamed MEAS
Other:
- note added: "Question: Can we re-use BS1 after boot? No. You cannot. Verified that BS1=0 = SPI"
- note added: "TODO: Examine possible holes for Keystone 590 TODO: Connect pins 5&6 NOTE: ADC cap changed. TODO: Flip to top for display."
- note removed: "Question: Can we re-use BS1 after boot?"
- note removed: "TODO: Examine possible holes for Keystone 590"
- moved on the sheet: C14, J1, R6, SW1, SW2, SW3, TP2, U3, Y1

Commit message: Update all parts from tonight
Parts:
- added D2: 1N4148, Diode_SMD:D_SOD-323, symbol Diode:1N4148
Connections:
- net +9V: now also D2.1 (K); no longer SW4.2 (B)
- new net: D2.2 (A), SW4.2 (B)
Changed lines of the file:
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@@
 	(wire
 		(pts
+			(xy 119.38 124.46) (xy 119.38 114.3)
+		)
+		(stroke
+			(width 0)
+			(type default)
+		)
+	)
+	(wire
+		(pts
 			(xy 195.58 129.54) (xy 204.47 129.54)
 		)
@@
 	(wire
 		(pts
+			(xy 119.38 114.3) (xy 121.92 114.3)
+		)
+		(stroke
+			(width 0)
+			(type default)
+		)
+	)
+	(wire
+		(pts
 			(xy 238.76 60.96) (xy 251.46 60.96)
 		)
@@
 	(symbol
 		(lib_id "power:+9V")
-		(at 119.38 124.46 270)
+		(at 129.54 114.3 270)
 		(unit 1)
 		(exclude_from_sim no)
@@
 		(fields_autoplaced yes)
 		(property "Reference" "#PWR022"
-			(at 115.57 124.46 0)
+			(at 125.73 114.3 0)
 			(effects
 				(font
@@
 		)
 		(property "Value" "+9V"
-			(at 123.19 124.4599 90)
+			(at 133.35 114.2999 90)
 			(effects
 				(font
@@
 		)
 		(property "Footprint" ""
-			(at 119.38 124.46 0)
+			(at 129.54 114.3 0)
 			(effects
 				(font
@@
 		)
 		(property "Datasheet" ""
-			(at 119.38 124.46 0)
+			(at 129.54 114.3 0)
 			(effects
 				(font
@@
 		)
 		(property "Description" "Power symbol creates a global label with name \"+9V\""
-			(at 119.38 124.46 0)
+			(at 129.54 114.3 0)
 			(effects
 				(font
@@
 		)
 		(instances
-			(project "ch570sao"
+			(project "ch570sao9v"
 				(path "/8b3ca9c1-ec01-472e-975f-b13c767b5c47"
 					(reference "#PWR022")
@@
 					(unit 1)
 				)
+			)
+		)
+	)
+	(symbol
+		(lib_id "Diode:1N4148")
+		(at 125.73 114.3 180)
+		(unit 1)
+		(exclude_from_sim no)
+		(in_bom yes)
+		(on_board yes)
+		(dnp no)
+		(fields_autoplaced yes)
+		(property "Reference" "D2"
+			(at 125.73 107.95 0)
+			(effects
+				(font
+					(size 1.27 1.27)
+				)
+			)
+		)
+		(property "Value" "1N4148"
+			(at 125.73 110.49 0)
+			(effects
+				(font
+					(size 1.27 1.27)
+				)
+			)
+		)
+		(property "Footprint" "Diode_SMD:D_SOD-323"
+			(at 125.73 114.3 0)
+			(effects
+				(font
+					(size 1.27 1.27)
+				)
+				(hide yes)
+			)
+		)
+		(property "Datasheet" "https://assets.nexperia.com/documents/data-sheet/1N4148_1N4448.pdf"
+			(at 125.73 114.3 0)
+			(effects
+				(font
+					(size 1.27 1.27)
+				)
+				(hide yes)
+			)
+		)
+		(property "Description" "100V 0.15A standard switching diode, DO-35"
+			(at 125.73 114.3 0)
+			(effects
+				(font
+					(size 1.27 1.27)
+				)
+				(hide yes)
+			)
+		)
+		(property "Sim.Device" "D"
+			(at 125.73 114.3 0)
+			(effects
+				(font
+					(size 1.27 1.27)
+				)
+				(hide yes)
+			)
+		)
+		(property "Sim.Pins" "1=K 2=A"
+			(at 125.73 114.3 0)
+			(effects
+				(font
+					(size 1.27 1.27)
+				)
+				(hide yes)
+			)
+		)
+		(property "LCSC" "C2128"
+			(at 125.73 114.3 0)
+			(effects
+				(font
+					(size 1.27 1.27)
+				)
+				(hide yes)
+			)
+		)
+		(pin "2"
+		)
+		(pin "1"
+		)
+		(instances
+			(project "ch570sao9v"
+				(path "/8b3ca9c1-ec01-472e-975f-b13c767b5c47"
+					(reference "D2")
+					(unit 1)
+				)
