File: ch584/froggyswadge/froggyswadge.kicad_sch (KiCad schematic)
At the start: 88 parts, among them J1 SAO, J2 PJ-307C, J3 RB130-2864KSWXG22, P1 USB_C_Plug_USB2.0, Q1 PMOS, Q2 PMOS, SW1 TS-1187A-B-A-B, SW2 TS-1187A-B-A-B, SW3 TS-1187A-B-A-B, SW4 TS-1187A-B-A-B, SW5 TS-1187A-B-A-B, SW6 TS-1187A-B-A-B, SW7 TS-1187A-B-A-B, U2 SM5701_2.2V, U3 XC6206PxxxMR, U4 XT1861B332MR-G, U6 LSM6DSL, Y1 32MHz, Y2 32.768kHz

Commit message: Update design
Parts:
- added J4, J5, J6, J7: MOUNT, cnhardware:SMTSO20xx, symbol Connector_Generic:Conn_01x01
- U1: value ~ -> CH584F
Connections:
- net GND: now also J4.1 (Pin_1), J5.1 (Pin_1), J6.1 (Pin_1), J7.1 (Pin_1)

Commit message: Bump design
Parts:
- J3: footprint Connector_FFC-FPC:Hirose_FH12-16S-0.5SH_1x16-1MP_P0.50mm_Horizontal -> cnhardware:FPC-16-P0.50mm-HC-FPC-05-09-16RLTAG-TOP-AND-BOTTOM; LCSC (none) -> C5213753
Changed lines of the file:
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@@
 			)
 		)
-		(property "Footprint" "Connector_FFC-FPC:Hirose_FH12-16S-0.5SH_1x16-1MP_P0.50mm_Horizontal"
+		(property "Footprint" "cnhardware:FPC-16-P0.50mm-HC-FPC-05-09-16RLTAG-TOP-AND-BOTTOM"
 			(at 168.91 148.59 0)
 			(effects
@@
 			(at 168.91 148.59 0)
 			(effects
+				(font
+					(size 1.27 1.27)
+				)
+				(hide yes)
+			)
+		)
+		(property "LCSC" "C5213753"
+			(at 168.91 148.59 0)
+			(effects

Commit message: Bump design
Parts:
- removed R17: MICSHUNT, cnhardware:R_0402_1005Metric_COMPACT, symbol Device:R_Small
- removed R9: IMUSHUNT, cnhardware:R_0402_1005Metric_COMPACT, symbol Device:R_Small
- removed U1: CH584F, Package_DFN_QFN:VQFN-32-1EP_4x4mm_P0.4mm_EP2.8x2.8mm, symbol cnhardware:CH584F
- added C35: 1μF, Capacitor_SMD:C_0402_1005Metric, symbol Swadge_Parts:C
- added R9: 5.1kΩ, cnhardware:R_0402_1005Metric_COMPACT, symbol Swadge_Parts:R_US
- added TP1: BATT, TestPoint:TestPoint_Pad_D1.0mm, symbol Connector:TestPoint
- added TP2: VDCID, TestPoint:TestPoint_Pad_D1.0mm, symbol Connector:TestPoint
- added TP3: OLEDVDD, TestPoint:TestPoint_Pad_D1.0mm, symbol Connector:TestPoint
- added TP4: GND, TestPoint:TestPoint_Pad_D1.0mm, symbol Connector:TestPoint
- added U1: ~, Package_DFN_QFN:QFN-48-1EP_5x5mm_P0.35mm_EP3.7x3.7mm, symbol cnhardware:CH584M
- D1, D2, D3, D4, D5, D6, D7: footprint Swadge_Parts:SK6812_SIDE_2 -> cnhardware:LC8812-3210_XL-3210RGBC; LCSC C2890037 -> C41413182
- J4, J5, J6, J7: LCSC (none) -> C2916318
- R10: value 560kΩ -> 5.1kΩ; LCSC C132339 -> C25905
- R15: LCSC (none) -> C17168
Connections:
- net BARB is gone; now on net GND: SW4.2 (B), SW5.2 (B), SW6.2 (B)
- net +2V2: now also R10.1, U6.5 (VDDIO), R9.1, U1.3 (VIO33)
- net +3V3: now also C35.1
- net AUDIOM: now also U1.18 (PB6)
- net AUDIOP: now also U1.20 (PB4)
- net B0: now also U1.46 (PA12); no longer SW4.1 (A)
- net B1: now also SW4.1 (A), U1.45 (PA13); no longer SW2.1 (A), SW5.1 (A)
- net B2: now also SW2.1 (A), U1.5 (PA8); no longer SW3.1 (A), SW6.1 (A)
- net BATT: now also TP1.1
- net BATTMID22: now also U1.4 (PA7); no longer R10.2
- net GND: now also SW1.2 (B), SW2.2 (B), SW3.2 (B), C35.2, TP4.1, U1.34 (ANT), U1.49 (GND); no longer U6.1 (SA0)
- net LED: now also U1.44 (PA14)
- net MIC: now also U1.37 (PA5)
- net OLEDCS: now also U1.30 (PB18)
- net OLEDDC: now also U1.36 (PA4)
- net OLEDMOSI: now also U1.40 (PA1)
- net OLEDRST: now also U1.38 (PA6)
- net OLEDSCK: now also U1.39 (PA0)
- net PGM_TCK: now also U1.11 (PB15)
- net PGM_TIO: now also U1.12 (PB14)
- net SAOG1: now also U1.26 (PB22)
- net SAOG2: now also U1.25 (PB23)
- net SCL_SAO: now also U1.27 (PB21); no longer U6.13 (SCL)
- net SDA_SAO: now also U1.28 (PB20); no longer U6.14 (SDA)
- net USB_D+: now also U1.15 (PB11)
- net USB_D-: now also U1.16 (PB10)
- net at L1.2: now also U1.2 (VSW)
- net at Y2.1: now also U1.48 (PA10)
- net at Y2.2: now also U1.47 (PA11)
- net at C1.1: now also U1.33 (VINTA)
- net at Y1.1: now also U1.32 (X32MI)
- net at Y1.3: now also U1.31 (X32MO)
- net IMUON: now reaches C34.2, R6.1, U6.12 (CS)
- net IMUON: now also U1.19 (PB5); no longer U6.5 (VDDIO)
- net at C25.1, J3.7 (Pin_7), R15.1: now also TP3.1
- net MICON: now reaches R2.2
- net MICON: now also U1.29 (PB19)
- removed net BARA: R10.1, SW1.2 (B), SW2.2 (B), SW3.2 (B)
- net VCIA renamed VDCI
- net VDCI: now also TP2.1, U1.1 (VDCID), U1.35 (VCIA)
- new net B3: SW5.1 (A), U1.43 (PA15)
- new net B4: SW3.1 (A), U1.42 (PA3)
- new net B5: SW6.1 (A), U1.41 (PA2)
- new net IMUSDO: U1.17 (PB7), U6.1 (SA0)
- new net NFC+: U1.9 (PB17)
- new net NFC-: U1.10 (PB16)
- new net NFCI: U1.7 (PB9)
- new net NFCM: U1.8 (PB8)
- new net SCL: R10.2, U1.13 (PB13), U6.13 (SCL)
- new net SDA: R9.2, U1.14 (PB12), U6.14 (SDA)
Other:
- note added: "RGB LEDs: Consider: XL-3210-RGBC-2812B"
- moved on the sheet: C1, C10, C17, C2, C22, C3, C34, C7, C8, J4, J5, J6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

Commit message: Bump to rev A
Parts:
- SW1, SW2, SW3, SW4, SW5, SW6, SW7: value TS-1187A-B-A-B -> SILICONE
- U1: footprint Package_DFN_QFN:QFN-48-1EP_5x5mm_P0.35mm_EP3.7x3.7mm -> cnhardware:QFN-48-WCH-VARIANT-CH584-CH585-1EP_5x5mm_P0.35mm_EP3.7x3.7mm
Connections:
- net OLEDCS: now also U1.6 (PA9); no longer U1.30 (PB18)
Changed lines of the file:
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@@
 	(global_label "OLEDCS"
 		(shape input)
-		(at 80.01 63.5 0)
+		(at 34.29 60.96 180)
 		(fields_autoplaced yes)
 		(effects
@@
 				(size 1.27 1.27)
 			)
-			(justify left)
+			(justify right)
 		)
 		(property "Intersheetrefs" "${INTERSHEET_REFS}"
-			(at 90.2523 63.5 0)
+			(at 24.0477 60.96 0)
 			(effects
 				(font
 					(size 1.27 1.27)
 				)
-				(justify left)
+				(justify right)
 				(hide yes)
 			)
@@
 			)
 		)
-		(property "Value" "TS-1187A-B-A-B"
+		(property "Value" "SILICONE"
 			(at 237.49 114.3 0)
 			(effects
@@
 			)
 		)
-		(property "Value" "TS-1187A-B-A-B"
+		(property "Value" "SILICONE"
 			(at 261.62 114.3 0)
 			(effects
@@
 			)
 		)
-		(property "Value" "TS-1187A-B-A-B"
+		(property "Value" "SILICONE"
 			(at 261.62 106.68 0)
 			(effects
@@
 			)
 		)
-		(property "Value" "TS-1187A-B-A-B"
+		(property "Value" "SILICONE"
 			(at 237.49 121.92 0)
 			(effects
@@
 			)
 		)
-		(property "Value" "TS-1187A-B-A-B"
+		(property "Value" "SILICONE"
 			(at 237.49 129.54 0)
 			(effects
@@
 			)
 		)
-		(property "Footprint" "Package_DFN_QFN:QFN-48-1EP_5x5mm_P0.35mm_EP3.7x3.7mm"
+		(property "Footprint" "cnhardware:QFN-48-WCH-VARIANT-CH584-CH585-1EP_5x5mm_P0.35mm_EP3.7x3.7mm"
 			(at 57.15 62.23 0)
 			(effects
@@
 			)
 		)
-		(property "Value" "TS-1187A-B-A-B"
+		(property "Value" "SILICONE"
 			(at 261.62 121.92 0)
 			(effects
@@
 			)
 		)
-		(property "Value" "TS-1187A-B-A-B"
+		(property "Value" "SILICONE"
 			(at 237.49 106.68 0)
 			(effects
