File: ch584/tadpoleswadge/tadpoleswadge.kicad_pcb (KiCad board)
At the start: 2 copper layers, 81.5 x 72.2 mm, 96 parts, among them J1 SAO, J2 PJ-307C, J3 RB130-2864KSWXG22, J4 MOUNT, J5 MOUNT, J6 MOUNT, J7 MOUNT, P1 USB_C_Plug_USB2.0, Q1 PMOS, Q2 PMOS, SW1 SILICONE, SW2 SILICONE, SW3 SILICONE, SW4 SILICONE, SW5 SILICONE, SW6 SILICONE, SW7 SILICONE, U2 SM5701_2.2V, U3 XC6206PxxxMR, U4 XT1861B332MR-G, U6 LSM6DSL, Y1 32MHz, Y2 32.768kHz

Commit message: Bump
Parts:
- removed BT1: Battery, Swadge_Parts:2460
- removed C17, C18, C19, C20, C25, C29, C3, C6: 10μF, Capacitor_SMD:C_0603_1608Metric
- removed C2: 100nF, Capacitor_SMD:C_0402_1005Metric
- removed C22: 4.7nF, cnhardware:R_0402_1005Metric_COMPACT
- removed C24, C26, C27, C28, C30, C31, C33, C34: 1μF, Capacitor_SMD:C_0402_1005Metric
- removed D4, D5, D6, D7: SK6812-SIDE-A, cnhardware:LC8812-3210_XL-3210RGBC
- removed J6: MOUNT, cnhardware:SMTSO20xx
- removed L1, L2: 10uH, Inductor_SMD:L_0603_1608Metric
- removed Q1, Q2: PMOS, Swadge_Parts:SOT-23
- removed R16: 560kΩ, cnhardware:R_0402_1005Metric_COMPACT
- removed SW3, SW5, SW6, SW7: SILICONE, cnhardware:BTC007_Button_Silicone
- removed Y1: 32MHz, Crystal:Crystal_SMD_2016-4Pin_2.0x1.6mm
- removed Y2: 32.768kHz, Crystal:Crystal_SMD_3215-2Pin_3.2x1.5mm
- added BT2: Battery, cnhardware:2460, B.Cu at (212.5, 89.8)
- added C36: 10μF, Capacitor_SMD:C_0603_1608Metric, F.Cu at (104.0, 99.3)
- added C37: 1μF, Capacitor_SMD:C_0402_1005Metric, F.Cu at (122.0, 105.0)
- added C38: 100nF, Capacitor_SMD:C_0402_1005Metric, F.Cu at (122.0, 107.0)
- added C40: 0.1u, Capacitor_SMD:C_0402_1005Metric, F.Cu at (229.5, 96.8)
- added C41: 1u, Capacitor_SMD:C_0402_1005Metric, F.Cu at (124.9, 101.0)
- added C42: 1u, Capacitor_SMD:C_0402_1005Metric, F.Cu at (224.1, 86.3)
- added L6: 10uH, Inductor_SMD:L_0603_1608Metric, F.Cu at (104.0, 106.9)
- added R23: 5.1k, Resistor_SMD:R_0402_1005Metric, F.Cu at (222.2, 88.8)
- added TP10: LED-, TestPoint:TestPoint_Pad_D1.0mm, B.Cu at (201.8, 65.9)
- added TP11: V3.2, TestPoint:TestPoint_Pad_D1.0mm, B.Cu at (199.2, 64.5)
- added TP12: LED, TestPoint:TestPoint_Pad_D1.0mm, F.Cu at (145.0, 49.5)
- added TP13: VSYS, TestPoint:TestPoint_Pad_D1.0mm, F.Cu at (145.0, 52.5)
- added TP14: 3V2, TestPoint:TestPoint_Pad_D1.0mm, F.Cu at (145.0, 55.6)
- added TP5: VDCID, TestPoint:TestPoint_Pad_D1.0mm, F.Cu at (138.9, 58.6)
- added TP6: LCDSCK, TestPoint:TestPoint_Pad_D1.0mm, F.Cu at (141.9, 46.4)
- added TP7: LCDRS, TestPoint:TestPoint_Pad_D1.0mm, F.Cu at (141.9, 49.5)
- added TP8: LCDRS, TestPoint:TestPoint_Pad_D1.0mm, F.Cu at (141.9, 52.5)
- added TP9: LCDRS, TestPoint:TestPoint_Pad_D1.0mm, F.Cu at (141.9, 55.6)
- added U5: ~, Package_DFN_QFN:VQFN-32-1EP_4x4mm_P0.4mm_EP2.8x2.8mm, F.Cu at (212.2, 79.2)
- added U7: RB017A1505A_Connector, Swadge_Parts:HCTL HC-FPC-03-10-15RLTAG-TUCKED, F.Cu at (212.6, 80.0)
- added U8: AW32001, cnhardware:WLCSP-9-P0.5mm, F.Cu at (221.8, 86.1)
- added Y3: 32.768kHz, Crystal:Crystal_SMD_3215-2Pin_3.2x1.5mm, F.Cu at (208.4, 75.3)
- added Y4: 32MHz, Crystal:Crystal_SMD_2016-4Pin_2.0x1.6mm, F.Cu at (217.9, 79.7)
- C1, C15: value 1μF -> 10μF; footprint Capacitor_SMD:C_0402_1005Metric -> Capacitor_SMD:C_0603_1608Metric
- J3: value RB130-2864KSWXG22 -> PGM; footprint cnhardware:FPC-16-P0.50mm-HC-FPC-05-09-16RLTAG-TOP-AND-BOTTOM -> Connector_PinHeader_2.54mm:PinHeader_1x04_P2.54mm_Vertical; moved to B.Cu
- L5: value 10uH -> 3.3uH; footprint Inductor_SMD:L_0603_1608Metric -> Inductor_SMD:L_0805_2012Metric
- P1: moved to B.Cu
- R15: value OLEDSHUNT -> 100k
- R4: value 1MΩ -> 33Ω
- R5: value 1MΩ -> 420k
- R6: value 33Ω -> 100k
- R7: value 5.1kΩ -> 420k
- TP1, TP4: moved to F.Cu
- TP2: value VDCID -> LCDRESET; moved to F.Cu
- TP3: value OLEDVDD -> LCDCS; moved to F.Cu
- U1: value ~ -> MT3406; footprint cnhardware:QFN-48-WCH-VARIANT-CH584-CH585-1EP_5x5mm_P0.35mm_EP3.7x3.7mm -> Package_TO_SOT_SMD:SOT-23-5
- U2: value SM5701_2.2V -> RB017A1505A_Connector; footprint Package_TO_SOT_SMD:SOT-23 -> cnhardware:0.3K-HX-15PWB-LCD-CONNECTOR-TOP
- U3: value XC6206PxxxMR -> KXTJ3-1057; footprint Package_TO_SOT_SMD:SOT-23-3 -> Package_LGA:Kionix_LGA-12_2x2mm_P0.5mm_LayoutBorder2x4y
- U4: value XT1861B332MR-G -> LN6206P222MR-G; footprint Package_TO_SOT_SMD:SOT-23 -> Swadge_Parts:SOT-23
- U6: value LSM6DSL -> LN6206P222MR-G; footprint Swadge_Parts:LGA-14_3x2.5mm_P0.5mm_LayoutBorder3x4y -> Swadge_Parts:SOT-23
- moved SW1 155.2 mm to (233.5, 85.0)
- moved U4 152.3 mm to (226.2, 79.0), turned to 0 degrees
- moved R5 151.6 mm to (231.2, 95.0), turned to 0 degrees
- moved L5 150.8 mm to (228.1, 97.5), turned to -90 degrees
- moved R7 144.1 mm to (222.2, 79.0), turned to -90 degrees
- moved R6 141.6 mm to (234.8, 96.9), turned to 90 degrees
- moved SW2 139.9 mm to (212.5, 110.0)
- moved J3 130.4 mm to (229.5, 84.1)
- moved U2 130.3 mm to (207.2, 67.8)
- moved U1 129.0 mm to (232.2, 97.3), turned to 0 degrees
- moved J4 126.2 mm to (192.5, 100.0)
- moved J1 124.4 mm to (189.9, 62.5)
- moved D2 123.2 mm to (233.6, 78.5)
- moved SW4 119.4 mm to (191.5, 85.0)
- moved U6 117.9 mm to (207.9, 91.2), turned to -90 degrees
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Connections:
- C1 pad 1: Net-(U1-VINTA) -> +2V2
- C10 pad 1: +2V2 -> VSW
- C15 pad 1: +3V3 -> +BATT
- C21 pad 1: VBUS -> +5V
- C23 pad 1: Net-(J3-Pin_2) -> VSW
- C23 pad 2: Net-(J3-Pin_1) -> GND
- C32 pad 1: +3V3 -> +3V2
- C35 pad 1: +3V3 -> +3V2
- C4 pad 1: +3V3 -> +3V2
- C5 pad 1: +3V3 -> +3V2
- C7 pad 1: +2V2 -> VSW
- C8 pad 1: +2V2 -> VSW
- D1 pad 2: +3V3 -> +3V2
- D11 pad 4: VBUS -> +5V
- D2 pad 2: +3V3 -> +3V2
- D3 pad 2: +3V3 -> +3V2
- D3 pad 3: Net-(D3-OUT) -> unconnected-(D3-OUT-Pad3)
- J1 pad 1: +3V3 -> +BATT
- J1 pad 3: SDA_SAO -> SDA
- J1 pad 4: SCL_SAO -> SCL
- J3 pad 1: Net-(J3-Pin_1) -> +3V2
- J3 pad 2: Net-(J3-Pin_2) -> PGM_TCK
- J3 pad 3: Net-(J3-Pin_3) -> PGM_TIO
- J3 pad 4: Net-(J3-Pin_4) -> GND
- L5 pad 1: BATTMID33 -> +3V2
- L5 pad 2: BATTLX33 -> Net-(U1-SW)
- P1 pad A4_B9: VBUS -> +5V
- P1 pad A9_B4: VBUS -> +5V
- R10 pad 1: +2V2 -> VSW
- R11 pad 1: +2V2 -> VSW
- R12 pad 1: +2V2 -> VSW
- R15 pad 1: Net-(J3-Pin_7) -> Net-(U2-FMARK)
- R15 pad 2: +2V2 -> PGM_TCK
- R2 pad 2: MICON -> VSW
- R4 pad 1: BATT -> PWRINT
- R4 pad 2: PGM_TCK -> B0
- R5 pad 1: BATT -> +3V2
- R5 pad 2: PGM_TIO -> Net-(U1-FB)
- R6 pad 1: IMUON -> GND
- R6 pad 2: Net-(U6-VDD) -> Net-(U1-FB)
- R7 pad 1: +2V2 -> BATTMON
- R7 pad 2: SDA_SAO -> VSYS
- R8 pad 1: +2V2 -> VSW
- R8 pad 2: SCL_SAO -> LCDRESET
- R9 pad 1: +2V2 -> VSW
- TP1 pad 1: BATT -> +BATT
- TP2 pad 1: VDCI -> LCDRESET
- TP3 pad 1: Net-(J3-Pin_7) -> LCDCS
- TP4 pad 1: GND -> Net-(BT2--)
- U1 pad 1: VDCI -> VSYS
- U1 pad 2: Net-(U1-VSW) -> GND
- U1 pad 3: +2V2 -> Net-(U1-SW)
- U1 pad 4: BATTMID22 -> VSYS
- U1 pad 5: B2 -> Net-(U1-FB)
- U2 pad 2: BATTLX22 -> VSW
- U2 pad 3: +2V2 -> LCDCS
- U3 pad 2: +2V2 -> SDA
- U3 pad 3: VBUS -> VSW
- U4 pad 2: BATTLX33 -> +2V2
- U4 pad 3: +3V3 -> +BATT
- U6 pad 1: IMUSDO -> GND
- U6 pad 2: unconnected-(U6-SDx-Pad2) -> VSW
- U6 pad 3: unconnected-(U6-SCx-Pad3) -> +3V2
Routing:
- net GND: track 594.0 -> 7.12 mm, vias 325 -> 5
- net +3V3: track 171.7 -> 0.00 mm, vias 3 -> 0
- net +2V2: track 103.7 -> 0.00 mm, vias 7 -> 0
- net SCL_SAO: track 61.2 -> 0.00 mm, vias 2 -> 0
- net B4: track 57.5 -> 0.00 mm, vias 4 -> 0
- net B3: track 57.4 -> 0.00 mm, vias 4 -> 0
- net PGM_TIO: track 57.3 -> 0.00 mm, vias 3 -> 0
- net LED: track 55.0 -> 0.00 mm, vias 4 -> 0
- net SDA_SAO: track 52.3 -> 0.00 mm, vias 3 -> 0
- net SAOG2: track 52.1 -> 0.00 mm, vias 2 -> 0
- net B1: track 49.7 -> 0.00 mm, vias 2 -> 0
- net SAOG1: track 49.5 -> 0.00 mm, vias 3 -> 0
- net B5: track 44.3 -> 0.00 mm, vias 2 -> 0
- net B2: track 41.5 -> 0.00 mm, vias 2 -> 0
- net OLEDRST: track 36.4 -> 0.00 mm, vias 4 -> 0
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- removed copper zone on B.Cu, net GND
- removed copper zone on F.Cu, net GND
Other:
- board size 81.5 x 72.2 mm -> 55.8 x 70 mm
- board text removed: "${REFERENCE}"
- board text removed: "froggyswadge revB ch584 cnhardware"

Commit message: Bump design
Parts:
- removed the C10 at (96.0, 104.4)
- removed the D2 at (233.6, 78.5)
- removed the J1 at (189.9, 62.5)
- added C23: 1μF, Capacitor_SMD:C_0402_1005Metric, F.Cu at (191.7, 66.9)
- added C24: 1μF, Capacitor_SMD:C_0402_1005Metric, F.Cu at (200.3, 78.7)
- added D5: EC3210R, cnhardware:EC3210R-OPSCO-RGB-LED, F.Cu at (233.5, 78.5)
- added J6: SAO, Connector_PinSocket_2.54mm:PinSocket_2x03_P2.54mm_Vertical, F.Cu at (190.2, 60.1)
- D1, D3: value SK6812-SIDE-A -> EC3210R; footprint cnhardware:LC8812-3210_XL-3210RGBC -> cnhardware:EC3210R-OPSCO-RGB-LED
- P1: moved to F.Cu
- TP1: renamed from TP5; moved to B.Cu
- TP10: renamed from TP8; value LCDRS -> RS; moved to B.Cu
- TP11: renamed from TP6; value LCDSCK -> SCK; moved to B.Cu
- TP12: renamed from TP3; value LCDCS -> CS; moved to B.Cu
- TP13: renamed from TP7; value LCDRS -> RS; moved to B.Cu
- TP14: renamed from TP2; value LCDRESET -> RST; moved to B.Cu
- TP2: renamed from TP1; moved to B.Cu
- TP3: renamed from TP4; moved to B.Cu
- TP4: renamed from TP13; moved to B.Cu
- TP5: renamed from TP14; moved to B.Cu
- TP8: renamed from TP12; moved to B.Cu
- TP9: value LCDRS -> FM; moved to B.Cu
- U2: renamed from U5; value ~ -> CH584F
- moved C3 125.8 mm to (224.9, 88.7)
- moved C21 125.5 mm to (223.3, 83.8)
- moved C18 116.7 mm to (233.4, 77.1), turned to 180 degrees
- moved C17 116.7 mm to (211.9, 88.5), turned to 180 degrees
- moved C2 112.3 mm to (214.3, 78.0), turned to -30 degrees
- moved C1 110.3 mm to (203.9, 76.5), turned to -90 degrees
- moved L1 106.7 mm to (206.3, 76.5), turned to -90 degrees
- moved C6 102.7 mm to (193.1, 73.5), turned to -90 degrees
- moved C8 100.9 mm to (200.7, 105.8), turned to 180 degrees
- moved C7 100.7 mm to (200.7, 103.3), turned to 180 degrees
- moved C20 98.4 mm to (220.3, 105.0), turned to 90 degrees
- moved L2 96.9 mm to (200.7, 108.4)
- moved L3 96.7 mm to (200.6, 100.9)
- moved C11 95.9 mm to (219.9, 87.8), turned to 90 degrees
- moved TP2 95.6 mm to (223.6, 90.8), turned to 180 degrees
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- renumbered BT2 to BT1, C40 to C10, C41 to C11, C42 to C12, C37 to C13, C38 to C14, C23 to C15, C7 to C16, C8 to C17, C5 to C18, C4 to C19, C36 to C2, C32 to C20, C35 to C22, C15 to C3, C16 to C4, C12 to C5, C11 to C6, C14 to C7, C13 to C8, D11 to D2, J2 to J1, J3 to J2, J4 to J3, J5 to J4, J7 to J5, L6 to L1, L3 to L2, L4 to L3, L5 to L4, R2 to R1, R11 to R10, R9 to R11, R10 to R12, R15 to R13, R8 to R14, R28 to R15, R27 to R16, R14 to R17, R13 to R18, R1 to R2, R23 to R4, R4 to R5, R5 to R6, R6 to R7, R7 to R8, R12 to R9, SW4 to SW2, SW2 to SW3, TP10 to TP6, TP11 to TP7, U4 to U1, U8 to U3, U1 to U4, U3 to U5, U2 to U8, Y3 to Y1, Y4 to Y2
Connections:
- BT1 pad 2: Net-(BT2--) -> GND
- D1 pad 1: LED -> GND
- D1 pad 2: +3V2 -> Net-(D1-Pin_2)
- D1 pad 3: Net-(D1-OUT) -> LED
- D1 pad 4: GND -> +3V2
- D3 pad 1: Net-(D2-OUT) -> GND
- D3 pad 2: +3V2 -> Net-(D3-Pin_2)
- D3 pad 3: unconnected-(D3-OUT-Pad3) -> Net-(D1-Pin_2)
- D3 pad 4: GND -> +3V2
- R13 pad 1: Net-(U2-FMARK) -> LCDFMARK
- TP3 pad 1: Net-(BT2--) -> GND
- U2 pad 27: MIC -> B2
- U2 pad 28: B2 -> MIC
- U7 pad 11: Net-(U2-FMARK) -> LCDFMARK
- U8 pad 11: Net-(U2-FMARK) -> LCDFMARK
Routing:
- net GND: track 7.12 -> 547.4 mm, vias 5 -> 242
- net +3V2: track 4.77 -> 158.2 mm, vias 3 -> 11
- net +BATT: track 0.00 -> 64.9 mm, vias 0 -> 3
- net Net-(D1-Pin_2): track 0.00 -> 55.7 mm
- net SDA: track 0.00 -> 55.4 mm, vias 0 -> 6
- net VSW: track 1.50 -> 56.0 mm, vias 1 -> 8
- net +5V: track 0.00 -> 54.0 mm, vias 0 -> 4
- net SCL: track 0.00 -> 50.8 mm, vias 0 -> 5
- net B0: track 0.00 -> 45.0 mm, vias 0 -> 4
- net LCDRS: track 1.73 -> 46.5 mm, vias 1 -> 6
- net Net-(D3-Pin_2): track 0.00 -> 40.8 mm
- net LCD_BLD: track 3.13 -> 41.3 mm, vias 2 -> 7
- net AUDIOP: track 0.00 -> 35.3 mm, vias 0 -> 2
- net Net-(P1-DN1): track 0.00 -> 32.4 mm, vias 0 -> 2
- net SAOG1: track 0.00 -> 31.6 mm, vias 0 -> 4
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- added copper zone on B.Cu, net GND
- added copper zone on F.Cu, net GND
Other:
- board size 55.8 x 70 mm -> 55.8 x 66.5 mm
- board text added: "3v2 tck tio gnd"
- board text added: "tadadpoleswadge cnhardware rev -"
