File: ch584/tadpoleswadge/tadpoleswadge.kicad_sch (KiCad schematic)
At the start: 83 parts, among them J1 SAO, J2 PJ-307C, J3 PGM, J4 MOUNT, J5 MOUNT, J6 MOUNT, J7 MOUNT, P1 USB_C_Plug_USB2.0, SW1 SILICONE, SW2 SILICONE, SW4 SILICONE, U1 MT3406, U2 RB017A1505A_Connector, U3 KXTJ3-1057, U4 LN6206P222MR-G, U6 LN6206P222MR-G, U8 AW32001, Y3 32.768kHz, Y4 32MHz

Commit message: Bump
Parts:
- C1, C10, C11, C12, C13, C14, C15, C16, C21, C23, C32, C35, C36, C37, C38, C4, C5, C7, C8, C9, R1, R10, R11, R12, R13, R14, R15, R2, R27, R28, R3, R4, R5, R6, R7, R8, R9: Cost100 10 -> .01
- D1, D2, D3: Cost100 (none) -> 0.0352
- D11: Cost100 95 -> 0.0481
- J1: Cost @ 2.5k 0.0471 -> (none)
- J2: Cost @ 2.5k 0.0261 -> (none); Cost100 (none) -> 0.0261
- J4, J5, J6, J7: Cost100 (none) -> 0.0719
- L3, L4, L6: Cost100 (none) -> 0.0413
- L5: Cost100 (none) -> 0.0212
- MK1: Cost @ 2.5k .1579 -> (none)
- P1: Cost @ 2.5k 0.0334 -> (none); Cost100 7.19 -> 0.0334
- R23: Cost100 (none) -> .01
- SW1, SW2, SW4: Cost100 (none) -> .04
- TP1, TP10, TP11, TP12, TP2, TP3, TP4, TP6, TP7, TP8, TP9: now left out of the parts list
- U1: Cost100 (none) -> 0.019
- U2: Cost @ 2.5k 0.0688 -> (none); Cost100 6 -> .0688
- U3: Cost100 (none) -> 0.1932
- U4, U6: Cost100 (none) -> 0.0228
- U5: Cost100 (none) -> 0.5371
- U8: Cost100 (none) -> 0.1905
- Y3: Cost100 (none) -> 0.0857
- Y4: Cost100 (none) -> 0.0465
Other:
- note added: "TODO: 1. If all I want on is the RTC, what voltage can the CH585 go down to? 2. Can R4 be removed? Shorted? 3. Can we remove LCDRESET? If not, remove R8 4. TODO: Can we enter shipping mode with a PFET? (To cut front power)"
- note removed: "TODO: 1. If all I want on is the RTC, what voltage can the CH585 go down to? 2. Can R4 be removed? Shorted? 3. Can we remove LCDRESET? If not, remove R8"
- moved on the sheet: C35, R15, TP10, TP11, U2, U4

Commit message: Update boards
Other:
- note added: "AW32001 = 0x49 (7 bit)"
- note added: "Electrical: CH584: NO-USB: 1.85-3.6V USB: 3.15-3.45V Accel: IO: 1.2 -3.6V VDD: 1.62-3.6V Ipwdn = <1uA Ioper=2-100uA Mic: VCC: 2.1V-3.6V Ioper=300uA LCD: VCC: 2.65-2.8-3.3 (10mA) VIO: 1.8-2.8 VBL: 2.8-3.2 (40mA)"
- note added: "For prototyping, consider C2890041 or C5378735 for RGB side, because it's economical."
- note removed: "QMC6309 = 0x7C (7 bit) LSM6DS3 = 0x6a (7 bit) QMI8658 = 0x6b (7 bit) AW32001 = 0x49 (7 bit) TODO: * Are QMI8658 / LSM6DS3"
Changed lines of the file:
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@@
 	(text "TODO:\n1. If all I want on is the RTC, what voltage can the CH585 go down to?\n2. Can R4 be removed?  Shorted?\n3. Can we remove LCDRESET? If not, remove R8\n4. TODO: Can we enter shipping mode with a PFET? (To cut front power)"
 		(exclude_from_sim no)
-		(at 99.314 171.958 0)
+		(at 74.93 184.912 0)
 		(effects
 			(font
@@
 		)
 	)
-	(text "QMC6309 = 0x7C (7 bit)\nLSM6DS3 = 0x6a (7 bit)\nQMI8658 = 0x6b (7 bit)\nAW32001 = 0x49 (7 bit)\n\nTODO:\n * Are QMI8658 / LSM6DS3"
+	(text "Electrical:\nCH584:\n  NO-USB: 1.85-3.6V\n  USB: 3.15-3.45V\n\nAccel:\n  IO:  1.2 -3.6V\n  VDD: 1.62-3.6V\n  Ipwdn = <1uA\n  Ioper=2-100uA\n\nMic:\n  VCC: 2.1V-3.6V\n  Ioper=300uA\n\nLCD:\n  VCC: 2.65-2.8-3.3 (10mA)\n  VIO: 1.8-2.8\n  VBL: 2.8-3.2 (40mA)"
 		(exclude_from_sim no)
-		(at 135.636 147.828 0)
+		(at 116.586 146.558 0)
+		(effects
+			(font
+				(size 1.27 1.27)
+			)
+			(justify left)
+		)
+	)
+	(text "AW32001 = 0x49 (7 bit)"
+		(exclude_from_sim no)
+		(at 90.424 131.318 0)
 		(effects
 			(font
@@
 		(effects
 			(font
+				(size 1.27 1.27)
+			)
+		)
+	)
+	(text "For prototyping, consider C2890041 or C5378735 for RGB side, because it's economical."
+		(exclude_from_sim no)
+		(at 240.03 4.064 0)
+		(effects
+			(font

Commit message: Bump
Parts:
- removed J6: MOUNT, cnhardware:SMTSO20xx, symbol Connector_Generic:Conn_01x01
- added TP13: VSYS, TestPoint:TestPoint_Pad_D1.0mm, symbol Connector:TestPoint
- added TP14: 3V2, TestPoint:TestPoint_Pad_D1.0mm, symbol Connector:TestPoint
- added U7: RB017A1505A_Connector, Swadge_Parts:HCTL HC-FPC-03-10-15RLTAG-TUCKED, symbol Swadge_Parts:RB017A1505A_Connector
- BT2: footprint cnhardware:BatteryHolder_Bulgin_BX0123_1xCR123 -> cnhardware:2460; LCSC C5290177 -> (none)
- U2: footprint Swadge_Parts:HCTL HC-FPC-03-10-15RLTAG-TUCKED -> cnhardware:0.3K-HX-15PWB-LCD-CONNECTOR-TOP; Cost100 .0688 -> .20; Digikey A141392TR-ND -> (none); LCSC C3012328 -> C2919525
Connections:
- net +3V2: now also TP14.1, U7.10 (VDD2.8V), U7.14 (LED+), U7.15 (LED+)
- net GND: now also U7.1 (GND), U7.16 (GND), U7.17 (GND), U7.6 (GND), U7.9 (GND)
- net LCDCS: now also U7.3 (CS)
- net LCDMOSI: now also U7.8 (SDA)
- net LCDRESET: now also U7.4 (RESET)
- net LCDRS: now also U7.5 (RS)
- net LCDSCK: now also U7.7 (SCL)
- net LCD_BLD: now also U7.12 (LED-), U7.13 (LED-)
- net VSW: now also U7.2 (VCC1.8V)
- net VSYS: now also TP13.1
- net at R15.1, U2.11 (FMARK): now also U7.11 (FMARK)
Other:
- note added: "TODO: 1. If all I want on is the RTC, what voltage can the CH585 go down to? 2. Can R4 be removed? Shorted? 3. Can we remove LCDRESET? If not, remove R8 4. TODO: Can we enter shipping mode with a PFET? (To cut front power) 5. CAn we remove MT3406"
- note removed: "TODO: 1. If all I want on is the RTC, what voltage can the CH585 go down to? 2. Can R4 be removed? Shorted? 3. Can we remove LCDRESET? If not, remove R8 4. TODO: Can we enter shipping mode with a PFET? (To cut front power)"

Commit message: Bump design
Parts:
- removed C10: 10μF, Capacitor_SMD:C_0603_1608Metric, symbol Swadge_Parts:C
- removed D2, D3: SK6812-SIDE-A, cnhardware:LC8812-3210_XL-3210RGBC, symbol Swadge_Parts:SK6812-SIDE-A
- added C23, C24: 1μF, Capacitor_SMD:C_0402_1005Metric, symbol Swadge_Parts:C
- added D1, D3, D5: EC3210R, cnhardware:EC3210R-OPSCO-RGB-LED, symbol Connector_Generic:Conn_01x04
- C10: renamed from C40; value 0.1u -> 100nF; Cost100 (none) -> .01; LCSC C307331 -> C1525
- C11: renamed from C41; value 1u -> 1μF; Cost100 (none) -> .01
- C12: renamed from C42; value 1u -> 1μF; Cost100 (none) -> .01
- D4: renamed from D1; value SK6812-SIDE-A -> LC8812-3210_XL-3210RGBC; now not fitted; now left out of the parts list
- J6: renamed from J1; footprint Swadge_Parts:PinHeader_2x03_P2.54mm_Vertical -> Connector_PinSocket_2.54mm:PinSocket_2x03_P2.54mm_Vertical
- R13: renamed from R15; LCSC C25905 -> C25741
- R4: renamed from R23; value 5.1k -> 5.1kΩ; footprint Resistor_SMD:R_0402_1005Metric -> cnhardware:R_0402_1005Metric_COMPACT
- R6: renamed from R5; value 420k -> 430k; LCSC C25905 -> C25786
- R7: renamed from R6; LCSC C25905 -> C25741
- R8: renamed from R7; value 420k -> 430k; LCSC C25905 -> C25786
- SW1, U7: now left out of the parts list
- SW2: renamed from SW4; now left out of the parts list
- SW3: renamed from SW2; now left out of the parts list
- TP1: renamed from TP5; now left out of the parts list
- TP10: renamed from TP8; value LCDRS -> RS
- TP11: renamed from TP6; value LCDSCK -> SCK
- TP12: renamed from TP3; value LCDCS -> CS
- TP13: renamed from TP7; value LCDRS -> RS
- TP14: renamed from TP2; value LCDRESET -> RST
- TP9: value LCDRS -> FM
- renumbered BT2 to BT1, C37 to C13, C38 to C14, C23 to C15, C7 to C16, C8 to C17, C5 to C18, C4 to C19, C36 to C2, C32 to C20, C35 to C22, C15 to C3, C16 to C4, C12 to C5, C11 to C6, C14 to C7, C13 to C8, D11 to D2, J2 to J1, J3 to J2, J4 to J3, J5 to J4, J7 to J5, L6 to L1, L3 to L2, L4 to L3, L5 to L4, R2 to R1, R11 to R10, R9 to R11, R10 to R12, R8 to R14, R28 to R15, R27 to R16, R14 to R17, R13 to R18, R1 to R2, R4 to R5, R12 to R9, TP1 to TP2, TP4 to TP3, TP13 to TP4, TP14 to TP5, TP10 to TP6, TP11 to TP7, TP12 to TP8, U4 to U1, U5 to U2, U8 to U3, U1 to U4, U3 to U5, U2 to U8, Y3 to Y1, Y4 to Y2
Connections:
- net +3V2: now also J6.1 (Pin_1), C23.1, D1.4 (Pin_4), D3.4 (Pin_4), D5.4 (Pin_4); no longer D4.2 (VDD)
- net +BATT: now also C24.1; no longer J6.1 (Pin_1)
- net B2: now also U2.27 (PA5); no longer U2.28 (PA15)
- net GND: now also BT1.2 (-), TP3.1, C23.2, C24.2, D1.1 (Pin_1), D3.1 (Pin_1), D5.1 (Pin_1); no longer D4.4 (GND)
- net LCDFMARK: now also R13.1, U7.11 (FMARK), U8.11 (FMARK)
- net LED: now also D1.3 (Pin_3); no longer D4.1 (IN)
- net MIC: now also U2.28 (PA15); no longer U2.27 (PA5)
- new net: D3.2 (Pin_2), D5.3 (Pin_3)
- new net: D1.2 (Pin_2), D3.3 (Pin_3)
Other:
- moved on the sheet: C18, C19, C20
