File: test/rf-playground/rf-playground.kicad_pcb (KiCad board)
At the start: 2 copper layers, 79 x 40 mm, 6 parts, among them J1 SMA

Commit message: bump design
Parts:
- added C4: C, Capacitor_SMD:C_0603_1608Metric, F.Cu at (101.2, 69.5)
- added J2: SMA, Connector_Coaxial:SMA_Amphenol_132289_EdgeMount, F.Cu at (97.4, 71.2)
- moved A1 0.14 mm to (133.6, 80.0)
- moved A1 0.10 mm to (134.4, 80.0)
Routing:
- net GND: track 10.1 -> 19.6 mm, vias 107 -> 114
- net Net-(J2-Pin_1): track 0.00 -> 4.19 mm
Other:
- board size 79 x 40 mm -> 84.5 x 40 mm
