File: test/rf-playground/rf-playground.kicad_sch (KiCad schematic)
At the start: 5 parts, among them J1 SMA

Commit message: bump design
Parts:
- added C4: C, Capacitor_SMD:C_0603_1608Metric, symbol Device:C
- added J2: SMA, Connector_Coaxial:SMA_Amphenol_132289_EdgeMount, symbol Connector_Generic:Conn_01x02
Connections:
- net GND: now also C4.2, J2.2 (Pin_2)
- new net: C4.1, J2.1 (Pin_1)

Commit message: Update notes
Other:
- note added: "Todo: 1. More vias 2. Smaller connectors for SMA (They aren't SMA) 3. Bigger board?"
Changed lines of the file:
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@@
 	(generator_version "9.0")
 	(paper "A4")
+	(text "Todo: \n1. More vias\n2. Smaller connectors for SMA (They aren't SMA)\n3. Bigger board?"
+		(exclude_from_sim no)
+		(at 163.576 53.848 0)
+		(effects
+			(font
+				(size 1.27 1.27)
+			)
+		)
+	)
 	(junction
 		(at 110.49 45.72)
@@
 		)
 		(instances
-			(project ""
+			(project "rf-playground"
 				(path "/26b57e6e-3bb2-4e80-8017-95c613862993"
 					(reference "C1")
@@
 		)
 		(instances
-			(project ""
+			(project "rf-playground"
 				(path "/26b57e6e-3bb2-4e80-8017-95c613862993"
 					(reference "J1")
@@
 		)
 		(instances
-			(project ""
+			(project "rf-playground"
 				(path "/26b57e6e-3bb2-4e80-8017-95c613862993"
 					(reference "#PWR01")
@@
 		)
 		(instances
-			(project ""
+			(project "rf-playground"
 				(path "/26b57e6e-3bb2-4e80-8017-95c613862993"
 					(reference "A1")
