File: ch584/froggyswadge/layer3/layer3.kicad_pcb (KiCad board)
At the start: 2 copper layers, 81.5 x 72.2 mm, 4 parts, among them J7 MOUNT

Commit message: Bump
Changed lines of the file:
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@@
 		(pad "" np_thru_hole circle
 			(at 0 0)
-			(size 6.2 6.2)
-			(drill 3.73)
+			(size 2.2 2.2)
+			(drill 2.2)
 			(layers)
 			(pinfunction "Pin_1")
@@
 		(pad "" np_thru_hole circle
 			(at 0 0)
-			(size 6.2 6.2)
-			(drill 3.73)
+			(size 2.2 2.2)
+			(drill 2.2)
 			(layers)
 			(pinfunction "Pin_1")
@@
 		(pad "" np_thru_hole circle
 			(at 0 0)
-			(size 6.2 6.2)
-			(drill 3.73)
+			(size 2.2 2.2)
+			(drill 2.2)
 			(layers)
 			(pinfunction "Pin_1")
@@
 		(pad "" np_thru_hole circle
 			(at 0 0)
-			(size 6.2 6.2)
-			(drill 3.73)
-			(layers)
-			(pinfunction "Pin_1")
+			(size 2.2 2.2)
+			(drill 2.2)
+			(layers)
+			(pinfunction "Pin_1")

Commit message: Update notes
Other:
- outline, holes or cut-outs redrawn
- board text added: "froggyswadge revB cover L3"
Changed lines of the file:
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@@
 			(drillshape 0)
 			(scaleselection 1)
-			(outputdirectory "layer3-revA")
+			(outputdirectory "layer3-revB")
 		)
 	)
@@
 	)
 	(gr_arc
-		(start 157.434103 97.388225)
-		(mid 156.56146 117.526565)
-		(end 137.061538 122.63218)
+		(start 82.402645 82.793213)
+		(mid 85.06 57.07)
+		(end 110.891554 55.855083)
+		(stroke
+			(width 0.05)
+			(type default)
+		)
+		(layer "Edge.Cuts")
+	)
+	(gr_curve
+		(pts
+			(xy 82.545898 96.936086) (xy 84.641898 90.316086) (xy 84.973394 87.09034) (xy 82.402646 82.793213)
+		)
+		(stroke
+			(width 0.05)
+			(type default)
+		)
+		(layer "Edge.Cuts")
+	)
+	(gr_rect
+		(start 84.8 58.01)
+		(end 95.41 65.84)
+		(stroke
+			(width 0.05)
+			(type default)
+		)
+		(fill no)
+		(layer "Edge.Cuts")
+	)
+	(gr_circle
+		(center 93.639176 104.05541)
+		(end 96.839176 104.05541)
+		(stroke
+			(width 0.05)
+			(type solid)
+		)
+		(fill no)
+		(layer "Edge.Cuts")
+	)
+	(gr_circle
+		(center 99.18 64.99)
+		(end 100.78 66.31)
+		(stroke
+			(width 0.05)
+			(type default)
+		)
+		(fill no)
+		(layer "Edge.Cuts")
+	)
+	(gr_circle
+		(center 101.716877 95.989447)
+		(end 104.916877 95.989447)
+		(stroke
+			(width 0.05)
+			(type solid)
+		)
+		(fill no)
+		(layer "Edge.Cuts")
+	)
+	(gr_circle
+		(center 101.88284 111.657148)
+		(end 105.08284 111.657148)
+		(stroke
+			(width 0.05)
+			(type solid)
+		)
+		(fill no)
+		(layer "Edge.Cuts")
+	)
+	(gr_rect
+		(start 103.74 60.61)
+		(end 138.46 84.94)
+		(stroke
+			(width 0.1)
+			(type solid)
+		)
+		(fill no)
+		(layer "Edge.Cuts")
+	)
+	(gr_arc
+		(start 109.244933 120.979048)
+		(mid 88.161755 117.54558)
+		(end 82.545897 96.936086)
+		(stroke
+			(width 0.05)
+			(type default)
+		)
+		(layer "Edge.Cuts")
+	)
+	(gr_curve
+		(pts
+			(xy 109.244933 120.979047) (xy 119.831898 116.176086) (xy 128.861178 118.548274) (xy 137.061538 122.63218)
+		)
+		(stroke
+			(width 0.05)
+			(type default)
+		)
+		(layer "Edge.Cuts")
+	)
+	(gr_circle
+		(center 109.89458 103.84348)
+		(end 113.09458 103.84348)
+		(stroke
+			(width 0.05)
+			(type solid)
+		)
+		(fill no)
+		(layer "Edge.Cuts")
+	)
+	(gr_circle
+		(center 123.73458 100.24348)
+		(end 126.93458 100.24348)
+		(stroke
+			(width 0.05)
+			(type solid)
+		)
+		(fill no)
+		(layer "Edge.Cuts")
+	)
+	(gr_arc
+		(start 132.276707 55.981834)
+		(mid 121.566877 58.829447)
+		(end 110.891554 55.855083)
 		(stroke
 			(width 0.05)
@@
 		(layer "Edge.Cuts")
 	)
+	(gr_circle
+		(center 139.110914 109.281746)
+		(end 142.310914 109.281746)
+		(stroke
+			(width 0.05)
+			(type solid)
+		)
+		(fill no)
+		(layer "Edge.Cuts")
+	)
+	(gr_line
+		(start 140.546877 60.579447)
+		(end 143.096801 53.576361)
+		(stroke
+			(width 0.05)
+			(type default)
+		)
+		(layer "Edge.Cuts")
+	)
+	(gr_line
+		(start 140.546877 60.94)
+		(end 140.546877 60.579447)
+		(stroke
+			(width 0.05)
+			(type default)
+		)
+		(layer "Edge.Cuts")
+	)
+	(gr_line
+		(start 145.126877 79.399447)
+		(end 155.945309 83.378822)
+		(stroke
+			(width 0.05)
+			(type default)
+		)
+		(layer "Edge.Cuts")
+	)
+	(gr_circle
+		(center 148.730914 100.231746)
+		(end 151.930914 100.231746)
+		(stroke
+			(width 0.05)
+			(type solid)
+		)
+		(fill no)
+		(layer "Edge.Cuts")
+	)
+	(gr_line
+		(start 149.016877 64.289447)
+		(end 140.546877 60.94)
+		(stroke
+			(width 0.05)
+			(type default)
+		)
+		(layer "Edge.Cuts")
+	)
+	(gr_line
+		(start 149.406877 67.799447)
+		(end 145.126877 79.399447)
+		(stroke
+			(width 0.05)
+			(type default)
+		)
+		(layer "Edge.Cuts")
+	)
+	(gr_line
+		(start 149.636877 63.949447)
+		(end 149.016877 64.289447)
+		(stroke
+			(width 0.05)
+			(type default)
+		)
+		(layer "Edge.Cuts")
+	)
+	(gr_line
+		(start 152.086877 57.199447)
+		(end 149.636877 63.949447)
+		(stroke
+			(width 0.05)
+			(type default)
+		)
+		(layer "Edge.Cuts")
+	)
+	(gr_line
+		(start 152.456877 57.199448)
+		(end 152.086877 57.199447)
+		(stroke
+			(width 0.05)
+			(type default)
+		)
+		(layer "Edge.Cuts")
+	)
 	(gr_arc
 		(start 152.456877 57.199447)
@@
 	)
 	(gr_arc
-		(start 109.244933 120.979048)
-		(mid 88.161755 117.54558)
-		(end 82.545897 96.936086)
-		(stroke
-			(width 0.05)
-			(type default)
-		)
-		(layer "Edge.Cuts")
-	)
-	(gr_circle
-		(center 93.639176 104.05541)
-		(end 96.839176 104.05541)
-		(stroke
-			(width 0.05)
-			(type solid)
-		)
-		(fill no)
-		(layer "Edge.Cuts")
-	)
-	(gr_circle
-		(center 139.110914 109.281746)
-		(end 142.310914 109.281746)
-		(stroke
-			(width 0.05)
-			(type solid)
-		)
-		(fill no)
-		(layer "Edge.Cuts")
-	)
-	(gr_line
-		(start 149.636877 63.949447)
-		(end 149.016877 64.289447)
-		(stroke
-			(width 0.05)
-			(type default)
-		)
-		(layer "Edge.Cuts")
-	)
-	(gr_line
-		(start 149.016877 64.289447)
-		(end 140.546877 60.94)
-		(stroke
-			(width 0.05)
-			(type default)
-		)
-		(layer "Edge.Cuts")
-	)
-	(gr_rect
-		(start 103.74 60.61)
-		(end 138.46 84.94)
-		(stroke
-			(width 0.1)
-			(type solid)
-		)
-		(fill no)
+		(start 157.434103 97.388225)
+		(mid 156.56146 117.526565)
+		(end 137.061538 122.63218)
+		(stroke
+			(width 0.05)
+			(type default)
+		)
 		(layer "Edge.Cuts")
 	)
@@
 		(layer "Edge.Cuts")
 	)
-	(gr_circle
-		(center 101.716877 95.989447)
-		(end 104.916877 95.989447)
-		(stroke
-			(width 0.05)
-			(type solid)
-		)
-		(fill no)
-		(layer "Edge.Cuts")
-	)
-	(gr_line
-		(start 152.456877 57.199448)
-		(end 152.086877 57.199447)
-		(stroke
-			(width 0.05)
-			(type default)
-		)
-		(layer "Edge.Cuts")
-	)
-	(gr_circle
-		(center 123.73458 100.24348)
-		(end 126.93458 100.24348)
-		(stroke
-			(width 0.05)
-			(type solid)
-		)
-		(fill no)
-		(layer "Edge.Cuts")
-	)
-	(gr_line
-		(start 152.086877 57.199447)
-		(end 149.636877 63.949447)
-		(stroke
-			(width 0.05)
-			(type default)
-		)
-		(layer "Edge.Cuts")
-	)
-	(gr_line
-		(start 145.126877 79.399447)
-		(end 155.945309 83.378822)
-		(stroke
-			(width 0.05)
-			(type default)
-		)
-		(layer "Edge.Cuts")
-	)
-	(gr_line
-		(start 149.406877 67.799447)
-		(end 145.126877 79.399447)
-		(stroke
-			(width 0.05)
-			(type default)
-		)
-		(layer "Edge.Cuts")
-	)
 	(gr_line
 		(start 159.579533 71.389036)
@@
 		(layer "Edge.Cuts")
 	)
-	(gr_line
-		(start 140.546877 60.94)
-		(end 140.546877 60.579447)
-		(stroke
-			(width 0.05)
-			(type default)
-		)
-		(layer "Edge.Cuts")
-	)
-	(gr_circle
-		(center 101.88284 111.657148)
-		(end 105.08284 111.657148)
-		(stroke
-			(width 0.05)
-			(type solid)
-		)
-		(fill no)
-		(layer "Edge.Cuts")
-	)
-	(gr_arc
-		(start 132.276707 55.981834)
-		(mid 121.566877 58.829447)
-		(end 110.891554 55.855083)
-		(stroke
-			(width 0.05)
-			(type default)
-		)
-		(layer "Edge.Cuts")
-	)
-	(gr_line
-		(start 140.546877 60.579447)
-		(end 143.096801 53.576361)
-		(stroke
-			(width 0.05)
-			(type default)
-		)
-		(layer "Edge.Cuts")
-	)
-	(gr_circle
-		(center 148.730914 100.231746)
-		(end 151.930914 100.231746)
-		(stroke
-			(width 0.05)
-			(type solid)
-		)
-		(fill no)
-		(layer "Edge.Cuts")
-	)
-	(gr_curve
-		(pts
-			(xy 109.244933 120.979047) (xy 119.831898 116.176086) (xy 128.861178 118.548274) (xy 137.061538 122.63218)
-		)
-		(stroke
-			(width 0.05)
-			(type default)
-		)
-		(layer "Edge.Cuts")
-	)
-	(gr_circle
-		(center 109.89458 103.84348)
-		(end 113.09458 103.84348)
-		(stroke
-			(width 0.05)
-			(type solid)
-		)
-		(fill no)
-		(layer "Edge.Cuts")
-	)
-	(gr_arc
-		(start 82.402645 82.793213)
-		(mid 85.06 57.07)
-		(end 110.891554 55.855083)
-		(stroke
-			(width 0.05)
-			(type default)
-		)
-		(layer "Edge.Cuts")
-	)
-	(gr_curve
-		(pts
-			(xy 82.545898 96.936086) (xy 84.641898 90.316086) (xy 84.973394 87.09034) (xy 82.402646 82.793213)
-		)
-		(stroke
-			(width 0.05)
-			(type default)
-		)
-		(layer "Edge.Cuts")
+	(gr_text "froggyswadge\nrevB cover L3"
+		(at 131.07 92.71 0)
+		(layer "F.Mask")
+		(effects
+			(font
+				(size 1 1)
+				(thickness 0.15)
+			)
+			(justify left bottom)
+		)
 	)
 	(embedded_fonts no)
