File: ch584/tadpoleswadge/layer2/layer2.kicad_pcb (KiCad board)
At the start: 2 copper layers, 55.8 x 60 mm, 0 parts

Commit message: Update notes
Other:
- outline, holes or cut-outs redrawn
- board text added: "tadpoleswadge reva layer2"
- board text removed: "tadpoleswadge rev- layer2"
