File: padauk/pfs122b-s16/pfs122b-s16.kicad_pcb (KiCad board)
At the start: 2 copper layers, 41.9 x 35.6 mm, 8 parts, among them J1 2.54mm Header 2x08P, J2 2.54mm Header 2x08P, U1 PFS122B-S16

Commit message: Bump designs
Other:
- board text added: "ALT: PMS120-S16"
Changed lines of the file:
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@@
 	)
 	(gr_text "PFS122B-S16\ndemoboard\ncnhardware"
-		(at 83.82 48.895 352)
+		(at 83.82 48.895 351.75)
 		(layer "F.SilkS")
 		(effects
+			(font
+				(size 1 1)
+				(thickness 0.2)
+				(bold yes)
+			)
+		)
+	)
+	(gr_text "ALT: PMS120-S16"
+		(at 81.915 74.93 351.801)
+		(layer "F.SilkS")
+		(effects
