File: lighting/hyperspecusb/polyspecusb.kicad_sch (KiCad schematic)
At the start: 54 parts, among them J2 USB_C_Receptacle_USB2.0, Q1 AO3401A, Q2 AO3401A, Q3 AO3401A, Q4 AO3401A, Q5 AO3401A, Q6 AO3401A, Q7 AO3401A, Q8 AO3401A, U1 CH32V006F8U6, U2 RY8401, U3 CH570Q, Y1 32M

Commit message: Bump design
Parts:
- added C11, C12, C13: 22n, Capacitor_SMD:C_0402_1005Metric, symbol Device:C
- added D8, D9: LED, cnhardware:LED_3535_3W_W_PAD, symbol cnhardware:LED_3535_3W_W_TP
- added L10, L11: 4.7u, Inductor_SMD:L_1008_2520Metric, symbol Device:L
- added Q10, Q9: AO3400A, cnhardware:SOT-23-EXTRASPACE, symbol Transistor_FET:Q_NMOS_GSD
- added R12: 0, swadgeparts:R_0805_2012Metric, symbol Device:R
- Q1, Q2, Q3, Q4, Q5, Q6, Q7, Q8: value AO3401A -> AO3400A; footprint Package_TO_SOT_SMD:SOT-23 -> cnhardware:SOT-23-EXTRASPACE; LCSC C15127 -> C20917
Connections:
- net GND: now also Q1.2 (S), Q2.2 (S), Q3.2 (S), Q4.2 (S), Q5.2 (S), Q6.2 (S), Q7.2 (S), Q8.2 (S), C11.1, C12.1, C13.1, Q10.2 (S), Q9.2 (S); no longer Q1.3 (D), Q2.3 (D), Q3.3 (D), Q4.3 (D), Q5.3 (D), Q6.3 (D), Q7.3 (D), Q8.3 (D)
- net SWD: now also R12.2; no longer U1.15 (PD1/SWIO/AETR/T1CH3/SCL/URX)
- net VBUS: now also C11.2, C12.2, C13.2, D8.1, D9.1, L10.2, L11.2
- net BST7: now reaches D4.2, L5.1
- net BST7: now also Q4.3 (D); no longer Q4.2 (S)
- net BST5: now reaches D6.2, L7.1
- net BST5: now also Q6.3 (D); no longer Q6.2 (S)
- net BST4: now reaches D7.2, L8.1
- net BST4: now also Q7.3 (D); no longer Q7.2 (S)
- net LED8: now reaches U1.16 (PD2/A3/T1CH1/T2CH3/T1CH2N)
- net LED8: now also Q10.1 (G)
- net LED9: now reaches U1.17 (PD3/A4/T2CH2/AETR/UCTS/T1CH4)
- net LED9: now also Q9.1 (G)
- net BST3: now reaches D0.2, L9.1
- net BST3: now also Q8.3 (D); no longer Q8.2 (S)
- net BST1: now reaches D2.2, L3.1
- net BST1: now also Q1.3 (D); no longer Q1.2 (S)
- net BST0: now reaches D3.2, L4.1
- net BST0: now also Q3.3 (D); no longer Q3.2 (S)
- net BST2: now reaches D1.2, L2.1
- net BST2: now also Q2.3 (D); no longer Q2.2 (S)
- net BST6: now reaches D5.2, L6.1
- net BST6: now also Q5.3 (D); no longer Q5.2 (S)
- new net: R12.1, U1.15 (PD1/SWIO/AETR/T1CH3/SCL/URX)
- new net BST8: D9.2, L11.1, Q10.3 (D)
- new net BST9: D8.2, L10.1, Q9.3 (D)
Other:
- note added: "TODO: 1. Consider 10-channel. 2. Make sure you use N-channel fets!"
- moved on the sheet: D0, D1, D2, D3, D4, D5, D6, D7, L2, L3, L4, L5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

Commit message: Bump
Other:
- note added: "Recommended roll: * Royal Blue 440nm + 30 * Blue 470nm + 25 * Cyan 495nm + 25 * Green 520nm + 40 Green 560? * Cyan yellow 575nm (Looks phosphor) +<<>> * Yellow 590-595nm (May be orange)? + 30 * Red 620nm +40 * Deep Red 660nm +60 * IR 730nm"
- note added: "Retily Avaialable LEDs: * Warm White 3000K * Cold White 6500K * Cold White 10000K * Cold White 20000K * Cold White 30000K * UV 365-370nm * UV 380-385nm * UV 395-400nm * UV 410-420nm * UV 420-430nm * Full Spectrum Pink * Royal Blue 440nm * Royal Blue 450nm * Blue 470nm * Cyan 495nm * Green 520nm * Cyan yellow 575nm (Looks phosphor) * Yellow 590-595nm * Orange 595nm (Looks phosphor) * Red 620nm * D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"
- note removed: "TODO: 1. Consider 10-channel. 2. Make sure you use N-channel fets!"
- moved on the sheet: D0, D1, D2, D3, D4, D5, D6, D7, D8, D9, L10, L11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

Commit message: Add notes
Other:
- note added: "Recommended roll: * Royal Blue 440nm + 30 * Blue 470nm + 25 * Cyan 495nm + 25 * Green 520nm + 40 Green 560? //* Cyan yellow 575nm (Looks phosphor) +<<>> * Yellow 580-585nm (May be orange)? + 30 * Red 620nm +40 * Deep Red 660nm +60 * IR 730nm"
- note added: "TODO: Add USB/PD protection"
- note removed: "Recommended roll: * Royal Blue 440nm + 30 * Blue 470nm + 25 * Cyan 495nm + 25 * Green 520nm + 40 Green 560? * Cyan yellow 575nm (Looks phosphor) +<<>> * Yellow 590-595nm (May be orange)? + 30 * Red 620nm +40 * Deep Red 660nm +60 * IR 730nm"
Changed lines of the file:
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@@
 		)
 	)
-	(text "Recommended roll:\n\n* Royal Blue 440nm + 30\n* Blue 470nm + 25\n* Cyan 495nm + 25\n* Green 520nm + 40\nGreen 560?\n* Cyan yellow 575nm  (Looks phosphor) +<<>>\n* Yellow 590-595nm (May be orange)? + 30\n* Red 620nm +40\n* Deep Red 660nm +60\n* IR 730nm"
+	(text "Recommended roll:\n\n* Royal Blue 440nm + 30\n* Blue 470nm + 25\n* Cyan 495nm + 25\n* Green 520nm + 40\nGreen 560?\n//* Cyan yellow 575nm  (Looks phosphor) +<<>>\n* Yellow 580-585nm (May be orange)? + 30\n* Red 620nm +40\n* Deep Red 660nm +60\n* IR 730nm"
 		(exclude_from_sim no)
 		(at 139.446 145.542 0)
@@
 		)
 	)
+	(text "TODO: Add USB/PD protection"
+		(exclude_from_sim no)
+		(at 212.598 161.798 0)
+		(effects
+			(font
+				(size 1.27 1.27)
+			)
+		)
+	)
