File: ch32m007/ch32m007e8r6-testboard/ch32m007e8r6-testboard.kicad_pcb (KiCad board)
At the start: 2 copper layers, 10 parts, among them J1 HDR, J2 PGM, J3 HDR, U1 CH32M007E8R6, U3 XC6206P332

Commit message: Bump design
Parts:
- removed C7, C8: 1u, Capacitor_SMD:C_0402_1005Metric
- removed U3: XC6206P332, Package_TO_SOT_SMD:SOT-23
- J2: footprint Connector_PinHeader_2.54mm:PinHeader_1x05_P2.54mm_Horizontal -> Connector_PinHeader_2.54mm:PinHeader_1x05_P2.54mm_Vertical
- moved C2 36.7 mm to (120.4, 93.7), turned to 120 degrees
- moved C1 36.3 mm to (119.8, 91.7), turned to -90 degrees
- moved C4 32.5 mm to (118.8, 91.6), turned to -90 degrees
Connections:
- J2 pad 5: +5V -> Net-(J1-Pin_23)
Routing:
- net SWD: track 0.00 -> 36.0 mm, vias 0 -> 1
- net SWC: track 0.00 -> 24.1 mm
- net GND: track 0.00 -> 22.4 mm, vias 0 -> 38
- net Net-(J3-Pin_1): track 0.00 -> 20.3 mm
- net Net-(J1-Pin_3): track 0.00 -> 19.2 mm
- net Net-(J3-Pin_3): track 0.00 -> 18.8 mm
- net +3V3: track 0.00 -> 18.1 mm, vias 0 -> 1
- net Net-(J1-Pin_5): track 0.00 -> 17.6 mm
- net Net-(J3-Pin_5): track 0.00 -> 17.4 mm
- net Net-(J1-Pin_7): track 0.00 -> 16.1 mm
- net Net-(J3-Pin_7): track 0.00 -> 16.0 mm
- net Net-(J1-Pin_10): track 0.00 -> 14.5 mm
- net Net-(J1-Pin_23): track 0.00 -> 14.5 mm
- net Net-(J3-Pin_10): track 0.00 -> 14.4 mm
- net Net-(J1-Pin_11): track 0.00 -> 13.1 mm
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- added copper zone on B.Cu, net GND
- added copper zone on F.Cu, net GND
Other:
- board outline added: 40.6 x 31.8 mm
- board text added: "PA1 PC5 PC4 PC2 PC1 PB3 LO3 HO3 LO2 HO2 LO1 HO1"
- board text added: "SWD PD2 PD3 PD4 PD5 PD6 PD7 PA4 PA5 VDD VSS VHV"
- board text added: "ch32m007e8r6 testboard rev -"
