File: ch32v20x/ch32v203f8u6funboard/ch32v203f8u6funboard.kicad_pcb (KiCad board)
At the start: 2 copper layers, 35.6 x 31.8 mm, 13 parts, among them J1 HEADER, J3 PGM, J4 USB_C_Receptacle_USB2.0, J5 HEADER, U1 CH32V203F8U6, U3 XC6206P332

Commit message: Bump designs
Routing:
- net (no net): track 0.00 -> 5.20 mm
