File: ch32v20x/ch32v203funboard/ch32v203funboard.kicad_pcb (KiCad board)
At the start: 2 copper layers, 43.2 x 35.2 mm, 21 parts, among them J1 HEADER, J2 HEADER, J3 PGM, J4 USB_C_Receptacle_USB2.0, SW1 BOOT, U2 SRV05-4, U3 XC6206P332, Y2 8MHz

Commit message: Bump
Routing:
- net D+: track 31.7 -> 29.6 mm
- net D-: track 34.0 -> 34.7 mm
- net GND: vias 76 -> 77
Other:
- board text added: "(QFN28)"
- board text added: "CH32V203"
- board text added: "Fly like a"
- board text added: "G6"
Changed lines of the file:
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@@
 			(effects
 				(font
-					(size 1 1)
-					(thickness 0.15)
+					(size 0.8 0.8)
+					(thickness 0.2)
+					(bold yes)
 				)
 			)
@@
 	)
 	(footprint "Connector_PinHeader_2.54mm:PinHeader_1x05_P2.54mm_Vertical"
+		(locked yes)
 		(layer "F.Cu")
 		(at 137.7 98.53 90)
@@
 			(effects
 				(font
-					(size 1 1)
-					(thickness 0.15)
+					(size 0.8 0.8)
+					(thickness 0.2)
 				)
 			)
@@
 			(effects
 				(font
-					(size 1 1)
-					(thickness 0.15)
+					(size 0.8 0.8)
+					(thickness 0.2)
+					(bold yes)
 				)
 			)
@@
 			(effects
 				(font
-					(size 1 1)
-					(thickness 0.15)
+					(size 0.8 0.8)
+					(thickness 0.2)
+					(bold yes)
 				)
 			)
@@
 			(effects
 				(font
-					(size 1 1)
-					(thickness 0.15)
+					(size 0.8 0.8)
+					(thickness 0.2)
+					(bold yes)
 				)
 			)
@@
 			(effects
 				(font
-					(size 1 1)
-					(thickness 0.15)
+					(size 0.8 0.8)
+					(thickness 0.2)
+					(bold yes)
 				)
 			)
@@
 			(effects
 				(font
-					(size 1 1)
-					(thickness 0.15)
+					(size 0.8 0.8)
+					(thickness 0.2)
+					(bold yes)
 				)
 			)
@@
 		(layer "Edge.Cuts")
 	)
+	(gr_text "Fly like a "
+		(at 132.4 87 0)
+		(layer "F.SilkS")
+		(effects
+			(font
+				(size 0.8 0.8)
+				(thickness 0.2)
+				(bold yes)
+			)
+			(justify left bottom)
+		)
+	)
+	(gr_text "(QFN28)"
+		(at 132.94 90.51 0)
+		(layer "F.SilkS")
+		(effects
+			(font
+				(size 0.8 0.8)
+				(thickness 0.2)
+				(bold yes)
+			)
+			(justify left bottom)
+		)
+	)
 	(gr_text "-"
 		(at 134.88 95.31 0)
@@
 		)
 	)
+	(gr_text "CH32V203"
+		(at 129.4 85.73 0)
+		(layer "F.SilkS")
+		(effects
+			(font
+				(size 1.5 1.5)
+				(thickness 0.375)
+				(bold yes)
+			)
+			(justify left bottom)
+		)
+	)
+	(gr_text "G6"
+		(at 133.75 89.11 0)
+		(layer "F.SilkS")
+		(effects
+			(font
+				(size 1.5 1.5)
+				(thickness 0.375)
+				(bold yes)
+			)
+			(justify left bottom)
+		)
+	)
 	(gr_text "5V\nGND\n3V3\nPA9\nD-\nD+\nA15\nPB3\nPB4\nPB5\nPB6\nPB7\nPB8"
 		(at 121.99 87.66 0)
@@
 	)
 	(via
+		(at 135.34 84.92)
+		(size 0.6)
+		(drill 0.3)
+		(layers "F.Cu" "B.Cu")
+		(free yes)
+		(net 1)
+	)
+	(via
 		(at 143.85 92.29)
 		(size 0.6)
@@
 	)
 	(via
-		(at 132.84 81.75)
+		(at 133.46 82.25)
 		(size 0.6)
 		(drill 0.3)
@@
 	)
 	(via
-		(at 138.91 86.34)
+		(at 137.53 85.98)
 		(size 0.6)
 		(drill 0.3)
@@
 	)
 	(segment
-		(start 139.84 85.47)
-		(end 140.045515 86.181196)
+		(start 138.11 87.3)
+		(end 137.39 87.32)
+		(width 0.2)
+		(layer "F.Cu")
+		(net 6)
+	)
+	(segment
+		(start 135.21 86.49)
+		(end 130.44 84.24)
 		(width 0.2)
 		(layer "F.Cu")
@@
 	)
 	(segment
-		(start 139.28 84.9)
-		(end 138.77 85.5)
+		(start 139.84 85.47)
+		(end 140.045515 86.181196)
 		(width 0.2)
 		(layer "F.Cu")
@@
 	)
 	(segment
-		(start 135.52 85.84)
-		(end 130.44 84.24)
-		(width 0.2)
-		(layer "F.Cu")
-		(net 6)
-	)
-	(segment
 		(start 140.21 76.88)
 		(end 140.22 77.705)
@@
 	)
 	(segment
-		(start 141.1625 82.06)
-		(end 140.11 83.19)
+		(start 128.265 85.09)
+		(end 125.725 85.09)
 		(width 0.2)
 		(layer "F.Cu")
@@
 	)
 	(segment
-		(start 140.11 83.19)
-		(end 139.28 84.9)
+		(start 136.45 86.58)
+		(end 135.21 86.49)
 		(width 0.2)
 		(layer "F.Cu")
@@
 	)
 	(segment
-		(start 141.13 76.72)
-		(end 140.8 76.61)
+		(start 140.045515 86.181196)
+		(end 138.11 87.3)
 		(width 0.2)
 		(layer "F.Cu")
@@
 	)
 	(segment
-		(start 140.42 86.46)
-		(end 140.81443 86.652891)
+		(start 137.39 87.32)
+		(end 136.45 86.58)
 		(width 0.2)
 		(layer "F.Cu")
@@
 	)
 	(segment
-		(start 140.5 76.61)
-		(end 140.28 76.76)
+		(start 141.13 76.72)
+		(end 140.8 76.61)
 		(width 0.2)
 		(layer "F.Cu")
@@
 	)
 	(segment
-		(start 140.52 79.17)
-		(end 140.95 79.46)
+		(start 140.42 86.46)
+		(end 140.81443 86.652891)
 		(width 0.2)
 		(layer "F.Cu")
@@
 	)
 	(segment
-		(start 125.725 85.09)
-		(end 128.265 85.09)
+		(start 140.5 76.61)
+		(end 140.28 76.76)
 		(width 0.2)
 		(layer "F.Cu")
@@
 	)
 	(segment
-		(start 138.77 85.5)
-		(end 135.52 85.84)
+		(start 140.52 79.17)
+		(end 140.95 79.46)
 		(width 0.2)
 		(layer "F.Cu")
@@
 	)
 	(segment
+		(start 128.265 82.55)
+		(end 125.725 82.55)
+		(width 0.2)
+		(layer "F.Cu")
+		(net 7)
+	)
+	(segment
 		(start 143.0625 83.0675)
 		(end 143.0625 81.96)
@@
 	)
 	(segment
-		(start 125.725 82.55)
-		(end 128.265 82.55)
-		(width 0.2)
-		(layer "F.Cu")
-		(net 7)
-	)
-	(segment
 		(start 141.68484 87.032076)
 		(end 141.31 86.4)
@@
 	)
 	(segment
-		(start 135.678905 85.178905)
-		(end 128.265 82.55)
-		(width 0.2)
-		(layer "F.Cu")
-		(net 7)
-	)
-	(segment
 		(start 140.91 86.25)
 		(end 140.39 85.94)
@@
 	)
 	(segment
+		(start 135.39 85.87)
+		(end 128.265 82.55)
+		(width 0.2)
+		(layer "F.Cu")
+		(net 7)
+	)
+	(segment
 		(start 140.85 78.78)
 		(end 141.2 79.04)
@@
 	)
 	(via
-		(at 135.678905 85.178905)
+		(at 135.39 85.87)
 		(size 0.6)
 		(drill 0.3)
@@
 	)
 	(segment
-		(start 136.96 84.07)
-		(end 141.43 83.71)
+		(start 135.39 85.87)
+		(end 136.96 84.07)
 		(width 0.2)
 		(layer "B.Cu")
@@
 	)
 	(segment
-		(start 135.678905 85.178905)
-		(end 136.96 84.07)
+		(start 136.96 84.07)
+		(end 141.43 83.71)
 		(width 0.2)
 		(layer "B.Cu")
@@
 	)
 	(segment
-		(start 142.03125 86.832076)
-		(end 141.56 86)
+		(start 137.06 84.929002)
+		(end 133.81 83.18)
 		(width 0.2)
 		(layer "F.Cu")
@@
 	)
 	(segment
-		(start 125.725 80.01)
-		(end 128.265 80.01)
+		(start 142.03125 86.832076)
+		(end 141.56 86)
 		(width 0.2)
 		(layer "F.Cu")
@@
 	)
 	(segment
-		(start 141.56 86)
-		(end 141.06 85.62)
+		(start 128.265 80.01)
+		(end 125.725 80.01)
 		(width 0.2)
 		(layer "F.Cu")
@@
 	)
 	(segment
-		(start 133.75 83.03)
-		(end 136.95 84.91)
+		(start 141.56 86)
+		(end 141.06 85.62)
 		(width 0.2)
 		(layer "F.Cu")
@@
 	)
 	(segment
-		(start 128.265 80.01)
-		(end 133.75 83.03)
+		(start 133.81 83.18)
+		(end 128.265 80.01)
 		(width 0.2)
 		(layer "F.Cu")
@@
 	)
 	(via
-		(at 136.95 84.91)
+		(at 137.06 84.929002)
 		(size 0.6)
 		(drill 0.3)
@@
 	(segment
 		(start 141.06 85.62)
-		(end 136.95 84.91)
+		(end 137.06 84.929002)
 		(width 0.2)
 		(layer "B.Cu")

Commit message: Bump designs
Routing:
- net (no net): track 0.00 -> 5.20 mm
- net PA1: track 10.2 -> 12.7 mm
