File: ch32v20x/ch32v203funboard/ch32v203funboard.kicad_sch (KiCad schematic)
At the start: 21 parts, among them J1 HEADER, J2 HEADER, J3 PGM, J4 USB_C_Receptacle_USB2.0, SW1 BOOT, U2 SRV05-4, U3 XC6206P332, Y2 8MHz

Commit message: Bump designs
Parts:
- J4: LCSC C709358 -> C2765186
- U1: value ~ -> (none)
