File: ch32v20x/ch32v208funboard/ch32v208funboard.kicad_pcb (KiCad board)
At the start: 2 copper layers, 40.6 x 31.8 mm, 17 parts, among them J1 HDR, J2 ANTENNA, J3 USB_C_Receptacle_USB2.0, J4 HDR, U1 CH32V208GBU6, U3 XC6206P332, Y2 32MHz

Commit message: Bump funboard
Parts:
- removed J2: ANTENNA, RF_Antenna:Texas_SWRA117D_2.4GHz_Right
- added A1: PRO-OB-440, RF_Antenna:Abracon_PRO-OB-440, F.Cu at (120.2, 84.9)
- added C10: 1p8, Capacitor_SMD:C_0603_1608Metric, F.Cu at (117.1, 103.2)
- added C9: 1p8, Capacitor_SMD:C_0603_1608Metric, F.Cu at (124.5, 81.5)
- added L1: 1n8, Inductor_SMD:L_0603_1608Metric, F.Cu at (117.1, 105.7)
- J3: footprint cnhardware:USB_C_SMT_ONLY_Receptacle_USB2.0 -> cnhardware:USB_C_MOD_Receptacle_HRO_TYPE-C-31-M-12
Connections:
- J1 pad 1: GND -> Net-(J1-Pin_1)
- J1 pad 2: GND -> Net-(J1-Pin_1)
- J4 pad 1: Net-(J4-Pin_1) -> +5V
- J4 pad 2: Net-(J4-Pin_1) -> +5V
- U1 pad 28: Net-(J4-Pin_1) -> Net-(J1-Pin_1)
Routing:
- net Net-(J4-Pin_1): track 22.9 -> 0.00 mm, vias 1 -> 0
- net Net-(J1-Pin_1): track 0.00 -> 21.6 mm, vias 0 -> 2
- net +5V: track 14.9 -> 27.5 mm
- net GND: track 128.0 -> 115.4 mm

Commit message: Bump designs
Parts:
- added J2: PGM, Connector_PinHeader_2.54mm:PinHeader_1x05_P2.54mm_Vertical, F.Cu at (125.1, 81.3)
- C10, C9: footprint Capacitor_SMD:C_0603_1608Metric -> Capacitor_SMD:C_0402_1005Metric
- L1: footprint Inductor_SMD:L_0603_1608Metric -> Inductor_SMD:L_0402_1005Metric
- moved L1 20.7 mm to (118.8, 85.1), turned to 180 degrees
- moved C10 18.0 mm to (116.9, 85.1), turned to 180 degrees
- moved C8 8.23 mm to (127.2, 58.9), turned to -90 degrees
- moved C9 4.99 mm to (121.1, 85.1)
- moved C7 4.18 mm to (125.6, 67.5), turned to 90 degrees
- moved A1 3.96 mm to (120.0, 88.9)
- moved R2 3.14 mm to (117.7, 63.6)
- moved R3 2.78 mm to (121.9, 63.6)
- moved J3 2.54 mm to (120.0, 57.8)
- moved U3 2.38 mm to (123.5, 66.9)
- moved C1 2.09 mm to (121.0, 67.8), turned to 90 degrees
- moved C2 0.99 mm to (118.4, 78.8), turned to 180 degrees
Connections:
- net Net-(J4-Pin_3) renamed PA13/SWD
- net Net-(J4-Pin_5) renamed PA14/SWCLK
- A1 pad 1: GND -> Net-(A1-Pad1)
- A1 pad 2: Net-(A1-Pad2) -> GND
- C10 pad 1: Net-(A1-Pad2) -> Net-(A1-Pad1)
- L1 pad 2: Net-(A1-Pad2) -> Net-(A1-Pad1)
Routing:
- net GND: track 115.4 -> 74.9 mm, vias 70 -> 88
- net PA13/SWD: track 20.6 -> 48.2 mm, vias 1 -> 4
- net PA14/SWCLK: track 17.5 -> 36.3 mm, vias 0 -> 2
- net +5V: track 27.5 -> 43.2 mm, vias 0 -> 1
- net Net-(U1-ANT): track 12.3 -> 17.9 mm
- net Net-(A1-Pad1): track 0.00 -> 2.84 mm
- net D+: track 12.4 -> 15.2 mm
- net CC2: track 2.46 -> 0.00 mm
- net D-: track 12.4 -> 14.7 mm
- net Net-(J1-Pin_21): track 14.8 -> 16.9 mm
- net Net-(J1-Pin_19): track 13.2 -> 14.6 mm
- net Net-(J1-Pin_15): track 11.8 -> 13.2 mm
- net VDD: track 63.5 -> 64.7 mm, vias 4 -> 5
- net Net-(J1-Pin_13): track 12.4 -> 11.7 mm
- net Net-(J4-Pin_19): track 14.8 -> 15.4 mm
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Other:
- board size 40.6 x 31.8 mm -> 40.6 x 38.1 mm
- board text added: "0V SWD SWC 3.3 5V"
- board text added: "5V PB8 SWC SWD PA12 PA11 PC9 PC8 PC7 PC6 VDD GND"
- board text added: "PC14 PC15 VDD PA0 PA1 PA2 PA3 PA4 PA5 PA6 PA7 GND"
- board text removed: "GND PC15 VDD PA0 PA1 PA2 PA3 PA4 PA5 PA6 PA7 GND"
- board text removed: "PC14 PB8 SWC SWD PA12 PA11 PC9 PC8 PC7 PC6 VDD GND"

Commit message: Bump 208 board
Parts:
- A1: footprint RF_Antenna:Abracon_PRO-OB-440 -> RF_Antenna:Texas_SWRA117D_2.4GHz_Right
- C3, C8: value 1u -> 10u; footprint Capacitor_SMD:C_0402_1005Metric -> Capacitor_SMD:C_0603_1608Metric
- J3: footprint cnhardware:USB_C_MOD_Receptacle_HRO_TYPE-C-31-M-12 -> cnhardware:USB_C_TIGHT_IN_BOARD_161N-4BC21665
- moved C10 9.08 mm to (126.0, 85.4), turned to 0 degrees
- moved L1 5.36 mm to (124.2, 85.4), turned to 0 degrees
- moved A1 5.34 mm to (124.7, 86.4), turned to 180 degrees
- moved C8 3.13 mm to (127.6, 62.0)
- moved U3 2.02 mm to (124.0, 68.9)
- moved C7 1.90 mm to (126.2, 69.3)
- moved R2 1.51 mm to (117.7, 65.1)
- moved R3 1.31 mm to (122.0, 64.9)
- moved C9 1.29 mm to (122.3, 85.4), turned to 180 degrees
- moved C1 0.51 mm to (121.5, 67.8), turned to -90 degrees
- moved Y2 0.25 mm to (115.5, 69.0)
- moved C3 0.16 mm to (115.7, 72.0), turned to 150 degrees
- moved J3 0.09 mm to (120.0, 57.9)
Routing:
- net GND: track 74.9 -> 69.8 mm, vias 88 -> 89
- net +5V: track 43.2 -> 45.5 mm, vias 1 -> 3
- net CC2: track 0.00 -> 1.90 mm
- net VDD: track 64.7 -> 66.3 mm, vias 5 -> 6
- net D+: track 15.2 -> 13.8 mm, vias 0 -> 2
- net Net-(A1-Pad1): track 2.84 -> 1.88 mm
- net Net-(U1-ANT): track 17.9 -> 17.1 mm
- net Net-(J1-Pin_21): track 16.9 -> 16.2 mm
- net D-: track 14.7 -> 14.0 mm
- net Net-(J1-Pin_19): track 14.6 -> 14.1 mm
- net PA13/SWD: vias 4 -> 2
Other:
- board size 40.6 x 38.1 mm -> 40.6 x 35.6 mm

Commit message: Bump designs
Parts:
- added R4: 5.1k, Resistor_SMD:R_0402_1005Metric, F.Cu at (126.8, 65.0)
Connections:
- J4 pad 3: PA13/SWD -> Net-(J4-Pin_3)
- J4 pad 4: PA13/SWD -> Net-(J4-Pin_3)
- J4 pad 7: Net-(J4-Pin_7) -> PA13/SWD
- J4 pad 8: Net-(J4-Pin_7) -> PA13/SWD
- U1 pad 20: Net-(J4-Pin_7) -> PA13/SWD
- U1 pad 26: PA13/SWD -> Net-(J4-Pin_3)
Routing:
- net Net-(J4-Pin_3): track 0.00 -> 22.6 mm, vias 0 -> 2
- net Net-(J4-Pin_7): track 16.3 -> 0.00 mm
- net PA13/SWD: track 48.2 -> 39.1 mm
- net GND: vias 89 -> 91

Commit message: Bump funboards
Other:
- outline, holes or cut-outs redrawn
