File: ch570/lanterdongleaaa/lanterdongle123.kicad_pcb (KiCad board)
At the start: 2 copper layers, 37.2 x 61.5 mm, 39 parts, among them J1 PGM, Q1 2N7002, SW1 PWR, SW2 SW_SPST, SW3 SW_SPST, U2 TPS613221ADBV, U3 CH572Q, Y1 32M

Commit message: Update with new LED
Parts:
- added C11: 10nF, Capacitor_SMD:C_0805_2012Metric, F.Cu at (79.2, 158.9)
- moved R7 5.52 mm to (78.8, 150.5), turned to 0 degrees
- moved U2 4.21 mm to (77.6, 161.1), turned to 150 degrees
- moved C4 3.73 mm to (83.6, 161.2), turned to 140 degrees
- moved D6 2.40 mm to (73.8, 159.9), turned to -30 degrees
- moved D4 2.34 mm to (68.5, 149.2)
- moved R6 1.61 mm to (64.9, 152.9)
- moved D5 1.46 mm to (68.5, 156.0)
- moved L1 1.35 mm to (75.5, 165.0), turned to 60 degrees
- moved C1 0.79 mm to (76.0, 156.0)
- moved D3 0.71 mm to (63.1, 159.6)
- moved SW1 0.66 mm to (80.1, 165.8)
Connections:
- D1 pad 1: LED -> unconnected-(D1-DO-Pad1)
- D6 pad 4: unconnected-(D6-DI-Pad4) -> LED
Routing:
- net +3.3V: track 83.4 -> 73.6 mm, vias 6 -> 5
- net LED: track 41.5 -> 49.5 mm, vias 2 -> 4
- net Net-(SW2-A): track 7.91 -> 12.2 mm
- net Net-(D5-DI): track 4.18 -> 5.89 mm
- net Net-(SW3-A): track 24.3 -> 22.7 mm
- net GND: track 27.1 -> 25.6 mm, vias 66 -> 73
- net Net-(D3-DI): track 13.9 -> 12.5 mm
- net Net-(SW1-Pin_2): track 4.27 -> 5.31 mm
- net Net-(D2-DI): track 8.97 -> 8.29 mm
- net Net-(BT1-+): track 11.1 -> 10.5 mm
- net Net-(D1-DI): track 15.5 -> 16.1 mm
- net Net-(D4-DI): track 6.68 -> 6.10 mm
Other:
- board text added: "lanterdongleaaa2 revA"
- board text removed: "lanterdongleaaa2 rev-"

Commit message: Fixup overall
Parts:
- removed C11: 10nF, Capacitor_SMD:C_0805_2012Metric
- added C12: 33nF, Capacitor_SMD:C_0603_1608Metric, F.Cu at (69.8, 131.4)
- C10, C5, C6, C7: value 1uF -> 33nF; footprint Capacitor_SMD:C_1206_3216Metric -> Capacitor_SMD:C_0603_1608Metric
- C3, C4, C8, C9: value 10nF -> 33nF; footprint Capacitor_SMD:C_0805_2012Metric -> Capacitor_SMD:C_0603_1608Metric
- R1, R2, R3, R4, R6, R7: value 3.3k -> 2.2k; footprint Resistor_SMD:R_0805_2012Metric -> Resistor_SMD:R_0603_1608Metric
- R5: footprint Resistor_SMD:R_0805_2012Metric -> Resistor_SMD:R_0603_1608Metric
- moved C5 15.0 mm to (76.1, 158.1), turned to 0 degrees
- moved C6 11.2 mm to (75.6, 140.5), turned to -90 degrees
- moved C1 10.0 mm to (69.5, 163.7), turned to 180 degrees
- moved R4 8.17 mm to (76.0, 137.4), turned to 45 degrees
- moved R3 7.91 mm to (78.5, 135.1), turned to 60 degrees
- moved R1 5.61 mm to (74.0, 139.7), turned to 90 degrees
- moved U2 4.82 mm to (74.0, 164.3), turned to 180 degrees
- moved L1 3.99 mm to (74.7, 168.9), turned to 120 degrees
- moved C7 3.63 mm to (71.4, 152.7), turned to 150 degrees
- moved C10 2.02 mm to (74.6, 136.5), turned to 45 degrees
- moved C3 1.20 mm to (77.3, 134.3)
- moved D2 0.98 mm to (70.7, 167.2)
- moved R5 0.77 mm to (76.0, 133.6)
- moved R2 0.46 mm to (73.2, 135.3)
Routing:
- net GND: track 25.6 -> 46.3 mm, vias 73 -> 76
- net PA3: track 24.7 -> 16.8 mm
- net Net-(MK1-+): track 10.9 -> 6.05 mm
- net VDDA: track 27.9 -> 24.3 mm
- net Net-(SW1-Pin_2): track 5.31 -> 8.81 mm
- net PA2: track 4.99 -> 3.91 mm
- net Net-(D2-DI): track 8.29 -> 9.24 mm
- net +3.3V: track 73.6 -> 72.9 mm, vias 5 -> 6
- net Net-(D1-DI): track 16.1 -> 15.5 mm
